File: microcontroller.kicad_sch (KiCad schematic)
At the start: 65 parts, among them IC1 MIMXRT1062DVJ6B, J10 JTAG_SWD_10, J3 503182-1852, J4 USB_C_pycubed, J6 Conn_01x06, Q6 DMG2305UX-7, SW1 KMR231NG LFS, U6 TPS54226PWPR, U7 MR25H40MDF, U8 MKL02Z32VFG4, Y1 24.0mHz, Y2 32.768kHz

Commit message: hmm
Parts:
- renumbered J10 to J5, R38 to R15, R37 to R17, R37 to R25
Connections:
- net GPIO_EMC_14 renamed GPS_RX 
- net PROG: no longer names the net of SW1.A (P), SW1.A' (P1), U8.10 (PTB2)
- net VADCS_IN renamed ADCS_PWR_IN
Other:
- note added: "LPUART3_RXD"
- note added: "Should these be grounded or disconnected? Or, should I add PSRAM?"
- note removed: "Should these be grounded or disconnected?"
Changed lines of the file:
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@@
   (junction (at 222.9358 231.902) (diameter 0) (color 0 0 0 0)
   )
-  (junction (at 110.7948 250.063) (diameter 0) (color 0 0 0 0)
-  )
   (junction (at 238.9378 262.382) (diameter 0) (color 0 0 0 0)
   )
@@
     (stroke (width 0) (type default))
   )
-  (wire (pts (xy 110.7948 250.063) (xy 110.7948 248.412))
-    (stroke (width 0) (type default))
-  )
   (wire (pts (xy 144.1958 42.291) (xy 151.6888 42.291))
     (stroke (width 0) (type default))
@@
     (stroke (width 0) (type default))
   )
+  (wire (pts (xy 151.5872 334.3656) (xy 151.5364 334.3656))
+    (stroke (width 0) (type default))
+  )
   (wire (pts (xy 166.624 112.522) (xy 166.624 118.0084))
     (stroke (width 0) (type default))
@@
     (stroke (width 0) (type default))
   )
+  (wire (pts (xy 151.5364 334.3656) (xy 151.5364 333.502))
+    (stroke (width 0) (type default))
+  )
   (wire (pts (xy 73.0758 41.275) (xy 69.5198 41.275))
     (stroke (width 0) (type default))
@@
     (stroke (width 0) (type default))
   )
-  (wire (pts (xy 105.2068 250.063) (xy 110.7948 250.063))
-    (stroke (width 0) (type default))
-  )
   (wire (pts (xy 164.6428 261.112) (xy 164.6428 268.097))
     (stroke (width 0) (type default))
@@
     (stroke (width 0) (type default))
   )
+  (wire (pts (xy 151.5364 333.502) (xy 169.5958 333.502))
+    (stroke (width 0) (type default))
+  )
   (wire (pts (xy 152.4 130.302) (xy 160.401 130.302))
     (stroke (width 0) (type default))
@@
     (stroke (width 0) (type default))
   )
-  (wire (pts (xy 110.7948 250.063) (xy 110.7948 258.445))
+  (wire (pts (xy 110.7948 248.412) (xy 110.7948 258.445))
     (stroke (width 0) (type default))
   )
@@
     (effects (font (size 1.0668 1.0668)) (justify left bottom))
   )
+  (text "LPUART3_RXD" (at 124.3584 333.5528 0)
+    (effects (font (size 1.27 1.27)) (justify left bottom))
+  )
   (text "VADCS_IN is from the battery\n- after foot switches\n- after an ADCS board enable \nFET\n"
     (at 27.9908 124.7648 0)
@@
     (effects (font (size 1.27 1.27) (color 249 0 0 1)) (justify left bottom))
   )
-  (text "Should these be grounded \nor disconnected?\n" (at 142.5448 194.437 0)
+  (text "Should these be grounded \nor disconnected?\n\nOr, should I add PSRAM?\n"
+    (at 141.1224 196.7992 0)
     (effects (font (size 1.27 1.27) (color 255 0 0 1)) (justify left bottom))
   )
@@
     (effects (font (size 1.27 1.27)) (justify left bottom))
   )
+  (label "GPS_RX " (at 151.5872 334.3656 180) (fields_autoplaced)
+    (effects (font (size 1.27 1.27)) (justify right bottom))
+  )
   (label "FLASH.IO3" (at 154.8638 215.392 0) (fields_autoplaced)
     (effects (font (size 1.27 1.27)) (justify left bottom))
@@
     )
   )
-  (global_label "VADCS_IN" (shape bidirectional) (at 40.4368 100.457 270) (fields_autoplaced)
+  (global_label "ADCS_PWR_IN" (shape bidirectional) (at 40.4368 100.457 270) (fields_autoplaced)
     (effects (font (size 1.27 1.27)) (justify right))
-    (property "Intersheetrefs" "${INTERSHEET_REFS}" (at 40.4368 113.3831 90)
+    (property "Intersheetrefs" "${INTERSHEET_REFS}" (at 40.4368 117.2535 90)
       (effects (font (size 1.27 1.27)) (justify right) hide)
     )
@@
     )
   )
+  (global_label "ADCS_PWR_IN" (shape bidirectional) (at 52.6288 46.228 180) (fields_autoplaced)
+    (effects (font (size 1.27 1.27)) (justify right))
+    (property "Intersheetrefs" "${INTERSHEET_REFS}" (at 35.8323 46.228 0)
+      (effects (font (size 1.27 1.27)) (justify right) hide)
+    )
+  )
   (global_label "GPIO_B1_15" (shape bidirectional) (at 222.9358 202.692 0) (fields_autoplaced)
     (effects (font (size 1.27 1.27)) (justify left))
@@
     )
   )
-  (global_label "PROG" (shape bidirectional) (at 105.2068 250.063 180) (fields_autoplaced)
-    (effects (font (size 1.27 1.27)) (justify right))
-    (property "Intersheetrefs" "${INTERSHEET_REFS}" (at 95.9698 250.063 0)
-      (effects (font (size 1.27 1.27)) (justify right) hide)
-    )
-  )
-  (global_label "VADCS_IN" (shape bidirectional) (at 52.6288 46.228 180) (fields_autoplaced)
-    (effects (font (size 1.27 1.27)) (justify right))
-    (property "Intersheetrefs" "${INTERSHEET_REFS}" (at 39.7027 46.228 0)
-      (effects (font (size 1.27 1.27)) (justify right) hide)
-    )
-  )
   (global_label "PMIC_STBY_REQ" (shape bidirectional) (at 244.094 212.852 0) (fields_autoplaced)
     (effects (font (size 1.27 1.27)) (justify left))
@@
     )
   )
-  (global_label "GPIO_EMC_14" (shape bidirectional) (at 169.5958 333.502 180) (fields_autoplaced)
-    (effects (font (size 1.27 1.27)) (justify right))
-    (property "Intersheetrefs" "${INTERSHEET_REFS}" (at 152.7994 333.502 0)
-      (effects (font (size 1.27 1.27)) (justify right) hide)
-    )
-  )
   (global_label "GPIO_EMC_33" (shape bidirectional) (at 169.5958 343.662 180) (fields_autoplaced)
     (effects (font (size 1.27 1.27)) (justify right))
@@
   (symbol (lib_id "Device:R_US") (at 151.6888 268.859 0) (mirror x) (unit 1)
     (in_bom yes) (on_board yes) (dnp no)
-    (property "Reference" "R37" (at 147.6248 267.97 0)
+    (property "Reference" "R17" (at 147.6248 267.97 0)
       (effects (font (size 1.27 1.27)))
     )
@@
   (symbol (lib_id "Connector:Conn_ARM_JTAG_SWD_10") (at 61.6204 256.0828 0) (unit 1)
     (in_bom yes) (on_board yes) (dnp no)
-    (property "Reference" "J10" (at 53.5432 241.9604 0)
+    (property "Reference" "J5" (at 53.5432 241.9604 0)
       (effects (font (size 1.27 1.27)) (justify right))
     )
@@
   (symbol (lib_id "mainboard:GND") (at 123.1138 200.152 0) (unit 1)
     (in_bom yes) (on_board yes) (dnp no)
-    (property "Reference" "#GND023" (at 123.1138 200.152 0)
+    (property "Reference" "#GND04" (at 123.1138 200.152 0)
       (effects (font (size 1.27 1.27)) hide)
     )
@@
   (symbol (lib_id "mainboard:GND") (at 117.7798 230.378 0) (unit 1)
     (in_bom yes) (on_board yes) (dnp no)
-    (property "Reference" "#GND022" (at 117.7798 230.378 0)
+    (property "Reference" "#GND015" (at 117.7798 230.378 0)
       (effects (font (size 1.27 1.27)) hide)
     )
@@
   (symbol (lib_id "Device:R_US") (at 123.1138 159.512 0) (mirror x) (unit 1)
     (in_bom yes) (on_board yes) (dnp no)
-    (property "Reference" "R38" (at 119.3038 156.972 0)
+    (property "Reference" "R15" (at 119.3038 156.972 0)
       (effects (font (size 1.27 1.27)))
     )
@@
   (symbol (lib_name "+3V3_1") (lib_id "power:+3V3") (at 61.6204 239.8268 0) (unit 1)
     (in_bom yes) (on_board yes) (dnp no) (fields_autoplaced)
-    (property "Reference" "#PWR023" (at 61.6204 243.6368 0)
+    (property "Reference" "#PWR028" (at 61.6204 243.6368 0)
       (effects (font (size 1.27 1.27)) hide)
     )
@@
   (symbol (lib_id "mainboard:3.3V") (at 117.7798 215.138 0) (unit 1)
     (in_bom yes) (on_board yes) (dnp no)
-    (property "Reference" "#SUPPLY08" (at 117.7798 215.138 0)
+    (property "Reference" "#SUPPLY07" (at 117.7798 215.138 0)
       (effects (font (size 1.27 1.27)) hide)
     )
@@
   (symbol (lib_id "Device:R_US") (at 107.2388 245.872 270) (mirror x) (unit 1)
     (in_bom yes) (on_board yes) (dnp no)
-    (property "Reference" "R37" (at 105.3338 242.951 90)
+    (property "Reference" "R25" (at 105.3338 242.951 90)
       (effects (font (size 1.27 1.27)))
     )
@@
   (symbol (lib_id "mainboard:3.3V") (at 125.6538 154.432 0) (unit 1)
     (in_bom yes) (on_board yes) (dnp no)
-    (property "Reference" "#SUPPLY09" (at 125.6538 154.432 0)
+    (property "Reference" "#SUPPLY08" (at 125.6538 154.432 0)
       (effects (font (size 1.27 1.27)) hide)
     )

Commit message: organize
Connections:
- net GPS_RX  renamed GPIO_EMC_14

Commit message: ready for review
Parts:
- removed C31: 10nF, symbol pycubed_mainboard:10NF_10000PF-50V-10%(0603)
- added C32: 10nF, symbol pycubed_mainboard:10NF_10000PF-50V-10%(0603)
Connections:
- net +3V3: now also J6.6 (Pin_6)
- net GND: now also J6.3 (Pin_3), C32.2; no longer J6.5 (Pin_5)
- net GNDREF: now also J6.4 (Pin_4); no longer J6.6 (Pin_6)
- net at C50.1, C51.1, C52.1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: now also C32.1
- net ADCS_PWR_IN renamed ADCS_VBATT
- new net ENAB_ADCS: J6.5 (Pin_5)
Other:
- note added: ""ENAB""
- note added: "what dis?"
- note removed: ""XXX""

Commit message: pete feedback
Connections:
- net ENAB_ADCS renamed EN_ADCS
Other:
- note added: ""EN""
- note added: "Pete: "R42 turns on the regulator, but I can't imagine (similar to your note) why the microprocessor would want to turn of the power. If it's latched up, it won't be executing any code.""
- note added: "Should I put a pull-up on CS? - Pete votes no"
- note removed: ""ENAB""
- note removed: "Should I put a pull-up on CS?"
- note removed: "VBATT 4.5 to 18V"
Changed lines of the file:
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@@
     (effects (font (size 1.27 1.27) (color 253 0 0 1)) (justify left bottom))
-  )
-  (text "VBATT 4.5 to 18V" (at 37.3888 44.831 0)
-    (effects (font (size 1.0668 1.0668)) (justify left bottom))
   )
   (text "LPUART3_RXD" (at 139.2936 334.4672 0)
@@
     (effects (font (size 2.54 2.54)) (justify left bottom))
   )
-  (text "Should I put a\npull-up on CS?" (at 76.3524 219.5068 0)
+  (text "Should I put a\npull-up on CS?\n- Pete votes no" (at 76.3524 219.5068 0)
     (effects (font (size 1.27 1.27) (color 253 0 0 1)) (justify left bottom))
   )
   (text "pull up on CS?\n" (at 140.462 212.1408 0)
     (effects (font (size 1.27 1.27) (color 251 0 0 1)) (justify left bottom))
+  )
+  (text "Pete: \"R42 turns on the regulator, \nbut I can't imagine (similar to \nyour note) why the microprocessor\nwould want to turn of the power.  \nIf it's latched up, it won't be \nexecuting any code.\"\n"
+    (at 126.8222 31.0896 0)
+    (effects (font (size 1.27 1.27) (color 6 96 0 1)) (justify left bottom))
   )
   (text "Populate (and program) with either \nMKL02 from PJRC pre-programmed \nwith the Teensy Bootloader;\nor with JTAG/SWD connector"
@@
     (effects (font (size 1.27 1.27) (color 249 0 0 1)) (justify left bottom))
   )
-  (text "\"ENAB\"" (at 53.3654 85.09 0)
+  (text "\"EN\"" (at 52.2478 85.09 0)
     (effects (font (size 0.889 0.889)) (justify right bottom))
   )
@@
     (effects (font (size 1.27 1.27)) (justify left))
   )
-  (hierarchical_label "ENAB_ADCS" (shape input) (at 48.0568 99.2124 270) (fields_autoplaced)
-    (effects (font (size 1.27 1.27)) (justify right))
-  )
+  (hierarchical_label "EN_ADCS" (shape input) (at 48.0568 99.2124 270) (fields_autoplaced)
+    (effects (font (size 1.27 1.27)) (justify right))
+  )

Commit message: save
Parts:
- renumbered C32 to C7, R40 to R37, R39 to R38, R29 to R42
Changed lines of the file:
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@@
   (symbol (lib_id "power:+3V3") (at 118.0338 29.083 0) (unit 1)
     (in_bom yes) (on_board yes) (dnp no) (fields_autoplaced)
-    (property "Reference" "#PWR030" (at 118.0338 32.893 0)
+    (property "Reference" "#PWR07" (at 118.0338 32.893 0)
       (effects (font (size 1.27 1.27)) hide)
     )
@@
   (symbol (lib_id "mainboard:GND") (at 72.9488 56.388 0) (unit 1)
     (in_bom yes) (on_board yes) (dnp no)
-    (property "Reference" "#GND018" (at 72.9488 56.388 0)
+    (property "Reference" "#GND017" (at 72.9488 56.388 0)
       (effects (font (size 1.27 1.27)) hide)
     )
@@
   (symbol (lib_id "mainboard:R-US_R0603") (at 109.5248 29.083 0) (unit 1)
     (in_bom yes) (on_board yes) (dnp no)
-    (property "Reference" "R29" (at 106.8578 24.638 0)
+    (property "Reference" "R42" (at 106.8578 24.638 0)
       (effects (font (size 1.4986 1.4986)) (justify left bottom))
     )
@@
   (symbol (lib_id "Device:R_US") (at 117.1448 104.648 270) (mirror x) (unit 1)
     (in_bom yes) (on_board yes) (dnp no)
-    (property "Reference" "R40" (at 115.2398 102.489 90)
+    (property "Reference" "R37" (at 115.2398 102.489 90)
       (effects (font (size 1.27 1.27)))
     )
@@
   (symbol (lib_id "power:+3V3") (at 35.6108 37.973 0) (unit 1)
     (in_bom yes) (on_board yes) (dnp no) (fields_autoplaced)
-    (property "Reference" "#PWR030" (at 35.6108 41.783 0)
+    (property "Reference" "#PWR08" (at 35.6108 41.783 0)
       (effects (font (size 1.27 1.27)) hide)
     )
@@
   (symbol (lib_id "Device:C_Small") (at 80.4418 91.948 90) (unit 1)
     (in_bom yes) (on_board yes) (dnp no)
-    (property "Reference" "C32" (at 82.4738 86.614 90)
+    (property "Reference" "C7" (at 82.4738 86.614 90)
       (effects (font (size 1.27 1.27)) (justify left))
     )
@@
   (symbol (lib_id "power:GNDREF") (at 125.1458 107.188 0) (unit 1)
     (in_bom yes) (on_board yes) (dnp no)
-    (property "Reference" "#PWR016" (at 125.1458 113.538 0)
+    (property "Reference" "#PWR012" (at 125.1458 113.538 0)
       (effects (font (size 1.27 1.27)) hide)
     )
@@
   (symbol (lib_id "mainboard:GND") (at 126.4158 57.023 0) (unit 1)
     (in_bom yes) (on_board yes) (dnp no)
-    (property "Reference" "#GND021" (at 126.4158 57.023 0)
+    (property "Reference" "#GND018" (at 126.4158 57.023 0)
       (effects (font (size 1.27 1.27)) hide)
     )
@@
   (symbol (lib_id "power:GNDREF") (at 68.2498 137.541 0) (unit 1)
     (in_bom yes) (on_board yes) (dnp no)
-    (property "Reference" "#PWR017" (at 68.2498 143.891 0)
+    (property "Reference" "#PWR02" (at 68.2498 143.891 0)
       (effects (font (size 1.27 1.27)) hide)
     )
@@
   (symbol (lib_id "power:+3V3") (at 57.2262 103.505 0) (unit 1)
     (in_bom yes) (on_board yes) (dnp no) (fields_autoplaced)
-    (property "Reference" "#PWR030" (at 57.2262 107.315 0)
+    (property "Reference" "#PWR031" (at 57.2262 107.315 0)
       (effects (font (size 1.27 1.27)) hide)
     )
@@
   (symbol (lib_id "power:+3V3") (at 106.6038 61.976 0) (unit 1)
     (in_bom yes) (on_board yes) (dnp no)
-    (property "Reference" "#PWR030" (at 106.6038 65.786 0)
+    (property "Reference" "#PWR010" (at 106.6038 65.786 0)
       (effects (font (size 1.27 1.27)) hide)
     )
@@
   (symbol (lib_id "mainboard:GND") (at 60.3758 28.575 0) (unit 1)
     (in_bom yes) (on_board yes) (dnp no)
-    (property "Reference" "#GND017" (at 60.3758 28.575 0)
+    (property "Reference" "#GND016" (at 60.3758 28.575 0)
       (effects (font (size 1.27 1.27)) hide)
     )
@@
   (symbol (lib_id "Device:R_US") (at 117.1448 107.188 270) (mirror x) (unit 1)
     (in_bom yes) (on_board yes) (dnp no)
-    (property "Reference" "R39" (at 115.2398 109.474 90)
+    (property "Reference" "R38" (at 115.2398 109.474 90)
       (effects (font (size 1.27 1.27)))
     )
