File: sqrt_of_g/sensors.kicad_sch (KiCad schematic)
At the start: 22 parts, among them J1 Amphenol_901-144, J2 Amphenol_901-144, Q8 IRLML2803, Q9 NDS8434, U2 BMM150, U3 BMI270, U4 S1216V8, U5 EP2W+

Commit message: more schematic work... I was supposed to finish this a long time ago
Parts:
- removed C1, C2, C3, C4: 0.1uF, Capacitor_SMD:C_0603_1608Metric, symbol mainboard:C_Small
- removed C32: 10nF, symbol pycubed_mainboard:10NF_10000PF-50V-10%(0603)
- removed C50: 10uF, symbol pycubed_mainboard:10NF_10000PF-50V-10%(0603)
- removed C51: 4.7uF, symbol pycubed_mainboard:10NF_10000PF-50V-10%(0603)
- removed C52: 0.22uF, symbol pycubed_mainboard:10NF_10000PF-50V-10%(0603)
- removed J1, J2: Amphenol_901-144, mainboard:SMA_901-144-horizontal, symbol Connector:Conn_Coaxial
- removed Q8: IRLML2803, mainboard:SOT-23, symbol mainboard:IRLML2803TRPBF
- removed Q9: NDS8434, mainboard:NDS8434, symbol mainboard:NDS8434
- removed R1, R2: 10k, Resistor_SMD:R_0603_1608Metric, symbol mainboard:R-US_R0603
- removed R3: 10K, Resistor_SMD:R_0603_1608Metric, symbol mainboard:10KOHM-1_10W-1%(0603)0603
- removed R31: 10K, Resistor_SMD:R_0603_1608Metric, symbol mainboard:R-US_R0603
- removed R32: 4.7K, Resistor_SMD:R_0603_1608Metric, symbol mainboard:R-US_R0603
- removed R33: 3.3K, Resistor_SMD:R_0603_1608Metric, symbol mainboard:R-US_R0603
- removed U2: BMM150, Sensor_Motion:XDCR_BMM150, symbol mainboard:BMM150
- removed U3: BMI270, Sensor_Motion:XDCR_BMI270, symbol mainboard:BMI270
- removed U4: S1216V8, mainboard:S1216_24PIN_PACKAGE, symbol mainboard:S1216V8
- removed U5: EP2W+, mainboard:QFN32-5X5MM, symbol mainboard:EP2W+
Connections:
- no-connect marks 22 -> 0
Other:
- added sheet IMU1_and_MAG1 (imu_and_magnetometer.kicad_sch)
- added sheet IMU1_and_MAG2 (imu_and_magnetometer.kicad_sch)
- note removed: "6DOF SDO: bit 0 | SDO | ADDR | |-----|------| | GND | 0x68 | | 3V3 | 0x69 |"
- note removed: "Consider using the secondary I2C interface on the BMI270 Pros: - coherent data Cons: - if one device fails, they both fail? Or could we put isolation circuitry on the secondary interface?"
- note removed: "GPS Module"
- note removed: "GPS Power"
- note removed: "Magnetometer CSB: bit 0 SDO: bit 1 00100 | CSB | SDO | ADDR | |-----|-----|------| | GND | GND | 0x10 |"
- note removed: "Per Orion B16 datasheet, V_BCKP current draw is 15 μA"
- note removed: "RF Splitter (2 Way, 0deg DC-Pass)"
