File: sqrt_of_g/motors.kicad_sch (KiCad schematic)
At the start: 25 parts, among them U9 DRV8332DKDR

Commit message: ready for 2nd round of reviews
Connections:
- net Motor1.Fault renamed Fault
- net Motor1.M1 renamed M1
- net Motor1.OTW renamed OTW
- net Motor1.PWM_A renamed PWM_A
- net Motor1.PWM_B renamed PWM_B
- net Motor1.PWM_C renamed PWM_C
- net Motor1.RESET_A renamed RESET_A
- net Motor1.RESET_B renamed RESET_B
- net Motor1.RESET_C renamed RESET_C
