File: sqrt_of_g/photodiode_enable.kicad_sch (KiCad schematic)
At the start: 18 parts, among them Q10 IRLML2803, Q11 NDS8434, Q5 IRLML2803, Q7 NDS8434

Commit message: ready for 2nd round of reviews
Parts:
- removed C50: 10uF, symbol pycubed_mainboard:10NF_10000PF-50V-10%(0603)
- removed C52: 0.22uF, symbol pycubed_mainboard:10NF_10000PF-50V-10%(0603)
Connections:
- net 3V3_PHOTODIODE1: no longer C32.1, C51.1, Q7.5 (Drain), Q7.6 (Drain), Q7.7 (Drain), Q7.8 (Drain)
- new net: C32.1, C51.1, Q7.5 (Drain), Q7.6 (Drain), Q7.7 (Drain), Q7.8 (Drain)
Other:
- note added: "Photodiode Enable 1"
- note added: "Photodiode Enable 2"
- note removed: "Photodiode Power 1"
- note removed: "Photodiode Power 2"
Changed lines of the file:
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@@
   (junction (at 167.64 119.38) (diameter 0) (color 0 0 0 0)
   )
-  (junction (at 180.34 73.66) (diameter 0) (color 0 0 0 0)
-  )
   (junction (at 142.24 63.5) (diameter 0) (color 0 0 0 0)
   )
   (junction (at 180.34 137.16) (diameter 0) (color 0 0 0 0)
   )
-  (junction (at 180.34 81.28) (diameter 0) (color 0 0 0 0)
-  )
   (junction (at 187.96 129.54) (diameter 0) (color 0 0 0 0)
   )
@@
   (junction (at 137.16 73.66) (diameter 0) (color 0 0 0 0)
   )
-  (junction (at 187.96 73.66) (diameter 0) (color 0 0 0 0)
-  )
   (junction (at 172.72 73.66) (diameter 0) (color 0 0 0 0)
   )
@@
   (junction (at 167.64 63.5) (diameter 0) (color 0 0 0 0)
   )
-  (junction (at 187.96 81.28) (diameter 0) (color 0 0 0 0)
-  )
   (junction (at 137.16 119.38) (diameter 0) (color 0 0 0 0)
   )
@@
     (stroke (width 0) (type default))
   )
-  (wire (pts (xy 180.34 73.66) (xy 187.96 73.66))
-    (stroke (width 0) (type default))
-  )
   (wire (pts (xy 167.64 129.54) (xy 172.72 129.54))
     (stroke (width 0) (type default))
@@
     (stroke (width 0) (type default))
   )
-  (wire (pts (xy 187.96 73.66) (xy 193.04 73.66))
+  (wire (pts (xy 197.3326 73.6346) (xy 197.2564 73.6346))
     (stroke (width 0) (type default))
   )
@@
     (stroke (width 0) (type default))
   )
-  (wire (pts (xy 187.96 81.28) (xy 193.04 81.28))
+  (wire (pts (xy 197.3326 73.6346) (xy 197.3326 73.66))
     (stroke (width 0) (type default))
   )
@@
     (stroke (width 0) (type default))
   )
-  (wire (pts (xy 180.34 81.28) (xy 187.96 81.28))
-    (stroke (width 0) (type default))
-  )
   (wire (pts (xy 132.08 137.16) (xy 132.08 129.54))
     (stroke (width 0) (type default))
@@
     (stroke (width 0) (type default))
   )
-  (text "Photodiode Power 1" (at 139.065 50.292 0)
+  (text "Photodiode Enable 1" (at 139.065 50.292 0)
     (effects (font (size 2.159 2.159)) (justify left bottom))
   )
@@
     (effects (font (size 1.27 1.27)) (justify left bottom))
   )
-  (text "Photodiode Power 2" (at 140.4874 106.7308 0)
+  (text "Photodiode Enable 2" (at 140.4874 106.7308 0)
     (effects (font (size 2.159 2.159)) (justify left bottom))
   )
@@
     (effects (font (size 1.27 1.27)) (justify right))
   )
-  (hierarchical_label "3V3_PHOTODIODE1" (shape input) (at 193.04 73.66 0) (fields_autoplaced)
+  (hierarchical_label "3V3_PHOTODIODE1" (shape input) (at 180.34 73.6854 0) (fields_autoplaced)
     (effects (font (size 1.27 1.27)) (justify left))
   )
@@
     )
   )
-  (symbol (lib_id "pycubed_mainboard:10NF_10000PF-50V-10%(0603)") (at 187.96 78.74 0) (unit 1)
-    (in_bom yes) (on_board yes) (dnp no)
-    (property "Reference" "C52" (at 182.499 75.057 0)
-      (effects (font (size 1.4986 1.4986)) (justify left))
-    )
-    (property "Value" "0.22uF" (at 180.086 79.883 0)
-      (effects (font (size 1.4986 1.4986)) (justify left))
-    )
-    (property "Footprint" "" (at 187.96 78.74 0)
-      (effects (font (size 1.27 1.27)) hide)
-    )
-    (property "Datasheet" "" (at 187.96 78.74 0)
-      (effects (font (size 1.27 1.27)) hide)
-    )
-    (pin "1")
-    (pin "2")
-    (instances
-      (project "adcs-hardware"
-        (path "/2bf29f96-8e90-4c56-8856-49bc3b5fab50/3472706a-4f86-4fa0-acec-6a7dc1abcee9"
-          (reference "C52") (unit 1)
-        )
-        (path "/2bf29f96-8e90-4c56-8856-49bc3b5fab50/858df03b-f3fa-405c-9f19-26f8c483a3cb"
-          (reference "C41") (unit 1)
-        )
-      )
-    )
-  )
   (symbol (lib_id "pycubed_mainboard:10NF_10000PF-50V-10%(0603)") (at 180.34 78.74 0) (unit 1)
     (in_bom yes) (on_board yes) (dnp no)
@@
         )
       )
-    )
-  )
-  (symbol (lib_id "pycubed_mainboard:10NF_10000PF-50V-10%(0603)") (at 193.04 78.74 0) (unit 1)
-    (in_bom yes) (on_board yes) (dnp no)
-    (property "Reference" "C50" (at 187.579 75.057 0)
-      (effects (font (size 1.4986 1.4986)) (justify left))
-    )
-    (property "Value" "10uF" (at 187.071 79.883 0)
-      (effects (font (size 1.4986 1.4986)) (justify left))
-    )
-    (property "Footprint" "" (at 193.04 78.74 0)
-      (effects (font (size 1.27 1.27)) hide)
-    )
-    (property "Datasheet" "" (at 193.04 78.74 0)
-      (effects (font (size 1.27 1.27)) hide)
-    )
-    (pin "1")
-    (pin "2")
-    (instances
-      (project "adcs-hardware"
-        (path "/2bf29f96-8e90-4c56-8856-49bc3b5fab50/3472706a-4f86-4fa0-acec-6a7dc1abcee9"
-          (reference "C50") (unit 1)
-        )
-        (path "/2bf29f96-8e90-4c56-8856-49bc3b5fab50/858df03b-f3fa-405c-9f19-26f8c483a3cb"
-          (reference "C42") (unit 1)
-        )
-      )
