File: sqrt_of_g/adcs-hardware.kicad_pcb (KiCad board)
At the start: 2 copper layers, 36.2 x 47.6 mm, 45 parts, among them J5 JTAG_SWD_10, J6 Conn_01x06, Y1 24.0mHz, Y2 32.768kHz

Commit message: ready for 2nd round of reviews
Parts:
- added C37: 0.1uF, Capacitor_SMD:C_0603_1608Metric, F.Cu at (37.7, 40.1)
- added C38: 0.1uF, Capacitor_SMD:C_0603_1608Metric, F.Cu at (37.7, 42.6)
- added C57: 0.1uF, Capacitor_SMD:C_0603_1608Metric, F.Cu at (47.7, 40.1)
- added C58: 0.1uF, Capacitor_SMD:C_0603_1608Metric, F.Cu at (47.7, 42.6)
- added J19: 353621050, adcs:CON_353621050, F.Cu at (57.7, 23.3)
- added J20: 353621050, adcs:CON_353621050, F.Cu at (57.7, 32.5)
- added R1: 10K, Resistor_SMD:R_0603_1608Metric, F.Cu at (37.7, 45.1)
- added R10: 10k, Resistor_SMD:R_0603_1608Metric, F.Cu at (41.7, 45.1)
- added R11: 10k, Resistor_SMD:R_0603_1608Metric, F.Cu at (41.7, 47.7)
- added R12: 10k, Resistor_SMD:R_0603_1608Metric, F.Cu at (41.7, 50.2)
- added R13: 4.7K, Resistor_SMD:R_0603_1608Metric, F.Cu at (57.7, 42.6)
- added R14: 3.3K, Resistor_SMD:R_0603_1608Metric, F.Cu at (57.7, 45.1)
- added R18: 10K, Resistor_SMD:R_0603_1608Metric, F.Cu at (57.7, 47.7)
- added R19: 10K, Resistor_SMD:R_0603_1608Metric, F.Cu at (66.2, 19.8)
- added R2: 4.7K, Resistor_SMD:R_0603_1608Metric, F.Cu at (37.7, 47.7)
- added R21: 4.7K, Resistor_SMD:R_0603_1608Metric, F.Cu at (66.2, 22.3)
- added R22: 3.3K, Resistor_SMD:R_0603_1608Metric, F.Cu at (66.2, 24.8)
- added R23: 10K, Resistor_SMD:R_0603_1608Metric, F.Cu at (66.2, 27.3)
- added R24: 4.7K, Resistor_SMD:R_0603_1608Metric, F.Cu at (66.2, 29.8)
- added R26: 3.3K, Resistor_SMD:R_0603_1608Metric, F.Cu at (66.2, 32.4)
- added R3: 10K, Resistor_SMD:R_0603_1608Metric, F.Cu at (57.7, 40.1)
- added R30: 10K, Resistor_SMD:R_0603_1608Metric, F.Cu at (47.7, 45.1)
- added R31: 4.7K, Resistor_SMD:R_0603_1608Metric, F.Cu at (47.7, 47.7)
- added R32: 3.3K, Resistor_SMD:R_0603_1608Metric, F.Cu at (47.7, 50.2)
- added R33: 10k, Resistor_SMD:R_0603_1608Metric, F.Cu at (51.7, 40.1)
- added R34: 10k, Resistor_SMD:R_0603_1608Metric, F.Cu at (51.7, 42.6)
- added R35: 10k, Resistor_SMD:R_0603_1608Metric, F.Cu at (51.7, 45.1)
- added R36: 10k, Resistor_SMD:R_0603_1608Metric, F.Cu at (51.7, 47.7)
- added R40: 10k, Resistor_SMD:R_0603_1608Metric, F.Cu at (51.7, 50.2)
- added R7: 3.3K, Resistor_SMD:R_0603_1608Metric, F.Cu at (37.7, 50.2)
- added R8: 10k, Resistor_SMD:R_0603_1608Metric, F.Cu at (41.7, 40.1)
- added R9: 10k, Resistor_SMD:R_0603_1608Metric, F.Cu at (41.7, 42.6)

Commit message: pete feedback
Parts:
- added IC1: MIMXRT1062DVJ6B, adcs:BGA196C80P14X14_1200X1200X152N, F.Cu at (70.5, 103.2)
- added J14: 353621050, adcs:CON_353621050, F.Cu at (56.5, 100.4)
- added J6: Conn_01x06, Connector_PinHeader_2.54mm:PinHeader_1x06_P2.54mm_Vertical, F.Cu at (36.9, 107.1)
- added R1: 10K, Resistor_SMD:R_0603_1608Metric, F.Cu at (71.0, 114.0)
- added R13: 4.7K, Resistor_SMD:R_0603_1608Metric, F.Cu at (65.0, 116.5)
- added R14: 3.3k, Resistor_SMD:R_0603_1608Metric, F.Cu at (65.0, 119.0)
- added R19: 10K, Resistor_SMD:R_0603_1608Metric, F.Cu at (48.6, 125.4)
- added R2: 4.7K, Resistor_SMD:R_0603_1608Metric, F.Cu at (71.0, 116.5)
- added R21: 4.7K, Resistor_SMD:R_0603_1608Metric, F.Cu at (48.6, 127.9)
- added R22: 3.3k, Resistor_SMD:R_0603_1608Metric, F.Cu at (48.6, 130.4)
- added R3: 3.3k, Resistor_SMD:R_0603_1608Metric, F.Cu at (71.0, 119.0)
- added R41: 10K, Resistor_SMD:R_0603_1608Metric, F.Cu at (42.5, 125.4)
- added R43: 4.7K, Resistor_SMD:R_0603_1608Metric, F.Cu at (42.5, 127.9)
- added R44: 3.3k, Resistor_SMD:R_0603_1608Metric, F.Cu at (42.5, 130.4)
- added R45: 100k, Resistor_SMD:R_0603_1608Metric, F.Cu at (71.0, 128.5)
- added R46: 0, Resistor_SMD:R_0603_1608Metric, F.Cu at (41.2, 106.1)
- added R47: 0, Resistor_SMD:R_0603_1608Metric, F.Cu at (41.2, 108.6)
- added R48: 0, Resistor_SMD:R_0603_1608Metric, F.Cu at (41.2, 111.1)
- added R49: 0, Resistor_SMD:R_0603_1608Metric, F.Cu at (41.2, 113.6)
- added R5: 10K, Resistor_SMD:R_0603_1608Metric, F.Cu at (71.0, 123.5)
- added R50: 0, Resistor_SMD:R_0603_1608Metric, F.Cu at (41.2, 116.1)
- added R51: 0, Resistor_SMD:R_0603_1608Metric, F.Cu at (41.2, 118.6)
- added R52: 10K, Resistor_SMD:R_0603_1608Metric, F.Cu at (65.0, 123.5)
- added R53: 4.7K, Resistor_SMD:R_0603_1608Metric, F.Cu at (65.0, 126.0)
- added R54: 3.3k, Resistor_SMD:R_0603_1608Metric, F.Cu at (65.0, 128.5)
- added R55: 10K, Resistor_SMD:R_0603_1608Metric, F.Cu at (36.5, 125.4)
- added R56: 4.7K, Resistor_SMD:R_0603_1608Metric, F.Cu at (36.5, 127.9)
- added R57: 3.3k, Resistor_SMD:R_0603_1608Metric, F.Cu at (36.5, 130.4)
- added R6: 4.7K, Resistor_SMD:R_0603_1608Metric, F.Cu at (71.0, 126.0)
- added R7: 10K, Resistor_SMD:R_0603_1608Metric, F.Cu at (65.0, 114.0)
Connections:
- net /3V3_PHOTODIODE1 renamed /3V3_PD1
- net /3V3_PHOTODIODE2 renamed /3V3_PD2
- C10 pad 2: 3V3 -> +3V3
- C11 pad 2: 3V3 -> +3V3
- C12 pad 1: ADCS_VBATT -> /VBATT
- C13 pad 1: ADCS_VBATT -> /VBATT
- C37 pad 1: /IMU1_and_MAG1/3V3_SENSOR -> /IMU1_and_MAG1/3V3_SENSORS
- C38 pad 1: /IMU1_and_MAG1/3V3_SENSOR -> /IMU1_and_MAG1/3V3_SENSORS
- C57 pad 1: /IMU2_and_MAG2/3V3_SENSOR -> /IMU2_and_MAG2/3V3_SENSORS
- C58 pad 1: /IMU2_and_MAG2/3V3_SENSOR -> /IMU2_and_MAG2/3V3_SENSORS
- D2 pad 2: 3V3 -> +3V3
- J5 pad 1: 3V3 -> +3V3
- R11 pad 2: /IMU1_and_MAG1/SCL_SENSE -> /SCL2
- R12 pad 2: /IMU1_and_MAG1/SDA_SENSE -> /SDA2
- R27 pad 2: 3V3 -> +3V3
- R36 pad 2: /IMU2_and_MAG2/SCL_SENSE -> /SCL4
- R40 pad 2: /IMU2_and_MAG2/SDA_SENSE -> /SDA4
- R42 pad 2: 3V3 -> +3V3

Commit message: update board
Parts:
- removed the J6 at (70.2, 46.3)
- removed the J6 at (36.9, 107.1)
- added C1: 10nF, Capacitor_SMD:C_0603_1608Metric, F.Cu at (-25.7, 12.5)
- added C17: 4.7uF, Capacitor_SMD:C_0603_1608Metric, F.Cu at (-31.7, -4.58)
- added C18: 0.22uF, Capacitor_SMD:C_0603_1608Metric, F.Cu at (-31.7, -2.07)
- added C19: 10uF, Capacitor_SMD:C_0603_1608Metric, F.Cu at (-31.7, 0.44)
- added C2: 4.7uF, Capacitor_SMD:C_0603_1608Metric, F.Cu at (-25.7, 15.0)
- added C20: 4.7uF, Capacitor_SMD:C_0603_1608Metric, F.Cu at (-31.7, 2.95)
- added C21: 0.22uF, Capacitor_SMD:C_0603_1608Metric, F.Cu at (-31.7, 5.46)
- added C22: 10uF, Capacitor_SMD:C_0603_1608Metric, F.Cu at (-31.7, 7.97)
- added C23: 0.22uF, Capacitor_SMD:C_0603_1608Metric, F.Cu at (-27.7, -4.58)
- added C24: 2.2uF, Capacitor_SMD:C_0603_1608Metric, F.Cu at (-27.7, -2.07)
- added C25: 4.7uF, Capacitor_SMD:C_0603_1608Metric, F.Cu at (-31.6, -22.5)
- added C26: 0.22uF, Capacitor_SMD:C_0603_1608Metric, F.Cu at (-31.6, -20.0)
- added C27: 4.7uF, Capacitor_SMD:C_0603_1608Metric, F.Cu at (-31.6, -17.4)
- added C28: 0.22uF, Capacitor_SMD:C_0603_1608Metric, F.Cu at (-31.6, -14.9)
- added C29: 0.22uF, Capacitor_SMD:C_0603_1608Metric, F.Cu at (-31.6, -12.4)
- added C3: 10nF, Capacitor_SMD:C_0603_1608Metric, F.Cu at (-31.7, 12.5)
- added C30: 0.22uF, Capacitor_SMD:C_0603_1608Metric, F.Cu at (-27.7, 0.44)
- added C31: 10uF, Capacitor_SMD:C_0603_1608Metric, F.Cu at (-27.7, 2.95)
- added C32: 10nF, Capacitor_SMD:C_0603_1608Metric, F.Cu at (-27.7, 5.46)
- added C33: 10nF, Capacitor_SMD:C_0603_1608Metric, F.Cu at (-17.6, 9.46)
- added C34: 4.7uF, Capacitor_SMD:C_0603_1608Metric, F.Cu at (-17.6, 12.0)
- added C4: 4.7uF, Capacitor_SMD:C_0603_1608Metric, F.Cu at (-31.7, 15.0)
- added C41: 10nF, Capacitor_SMD:C_0603_1608Metric, F.Cu at (-17.6, -4.58)
- added C42: 4.7uF, Capacitor_SMD:C_0603_1608Metric, F.Cu at (-17.6, -2.07)
- added C5: 10nF, Capacitor_SMD:C_0603_1608Metric, F.Cu at (-11.6, -4.58)
- added C50: 10uF, Capacitor_SMD:C_0603_1608Metric, F.Cu at (-27.7, 7.97)
- added C51: 4.7uF, Capacitor_SMD:C_0603_1608Metric, F.Cu at (-23.6, -4.58)
- added C52: 0.22uF, Capacitor_SMD:C_0603_1608Metric, F.Cu at (-23.6, -2.07)
- added C59: 0.22uF, Capacitor_SMD:C_0603_1608Metric, F.Cu at (-23.6, 0.44)
- added C6: 4.7uF, Capacitor_SMD:C_0603_1608Metric, F.Cu at (-11.6, -2.07)
- added C60: 10nF, Capacitor_SMD:C_0603_1608Metric, F.Cu at (-11.6, 2.44)
- added C61: 4.7uF, Capacitor_SMD:C_0603_1608Metric, F.Cu at (-11.6, 4.95)
- added C62: 10nF, Capacitor_SMD:C_0603_1608Metric, F.Cu at (-17.6, 2.44)
- added C63: 4.7uF, Capacitor_SMD:C_0603_1608Metric, F.Cu at (-17.6, 4.95)
- added J1: Amphenol_901-144, mainboard:SMA_901-144-horizontal, F.Cu at (118.2, 83.8)
- added J10: 35362-0650, mainboard:MOLEX_35362-0650, F.Cu at (32.0, 62.1)
- added J11: Conn_01x10, Connector_PinHeader_1.27mm:PinHeader_1x10_P1.27mm_Vertical, F.Cu at (107.8, 72.2)
- added J13: 35362-0650, mainboard:MOLEX_35362-0650, F.Cu at (41.9, 62.1)
- added J15: Conn_01x10, Connector_PinHeader_1.27mm:PinHeader_1x10_P1.27mm_Vertical, F.Cu at (107.8, 68.1)
- added J16: 35362-0650, mainboard:MOLEX_35362-0650, F.Cu at (51.5, 62.0)
- added J17: Conn_01x10, Connector_PinHeader_1.27mm:PinHeader_1x10_P1.27mm_Vertical, F.Cu at (107.8, 63.9)
- added J18: 35362-0650, mainboard:MOLEX_35362-0650, F.Cu at (51.4, 46.3)
- added J2: Amphenol_901-144, mainboard:SMA_901-144-horizontal, F.Cu at (118.0, 102.5)
- added J21: Conn_01x06, mainboard:MOLEX_35362-0650, F.Cu at (32.8, 112.6)
- added J22: Conn_01x06, mainboard:MOLEX_35362-0650, F.Cu at (39.8, 112.6)
- added J23: Conn_01x06, mainboard:MOLEX_35362-0650, F.Cu at (46.9, 112.6)
- added J24: Conn_01x06, mainboard:MOLEX_35362-0650, F.Cu at (32.8, 96.8)
- added J25: Conn_01x06, mainboard:MOLEX_35362-0650, F.Cu at (39.9, 96.8)
- added J26: Conn_01x06, mainboard:MOLEX_35362-0650, F.Cu at (46.9, 96.8)
- added J27: Conn_01x10, Connector_PinHeader_1.27mm:PinHeader_1x10_P1.27mm_Vertical, F.Cu at (107.9, 60.1)
- added J28: 35362-0650, mainboard:MOLEX_35362-0650, F.Cu at (57.2, 30.4)
- added J3: 503182-1852, mainboard:MOLEX_503182-1852, B.Cu at (74.9, 116.5)
- added J4: USB_C_pycubed, mainboard:USB_C_Receptacle_XKB_U262-161N-4BVC11, F.Cu at (71.2, 31.6)
- added J6: Conn_01x06, Connector_PinHeader_2.54mm:PinHeader_1x06_P2.54mm_Vertical, F.Cu at (51.3, 36.6)
- added J7: Conn_01x08, Connector_PinHeader_2.54mm:PinHeader_1x08_P2.54mm_Vertical, F.Cu at (92.7, 42.0)
- added J8: Conn_01x10, Connector_PinHeader_1.27mm:PinHeader_1x10_P1.27mm_Vertical, F.Cu at (107.8, 76.4)
- added J9: 35362-0650, mainboard:MOLEX_35362-0650, F.Cu at (116.9, 43.5)
- added L1: 3.3uH, mainboard:L_2141, F.Cu at (-19.8, 63.9)
- added Q1: IRLML2803, mainboard:SOT-23, F.Cu at (-62.3, 68.0)
- added Q10: NDS8434, mainboard:NDS8434, F.Cu at (-15.7, 74.1)
- added Q11: NDS8434, mainboard:NDS8434, F.Cu at (-28.1, 74.1)
- added Q12: NDS8434, mainboard:NDS8434, F.Cu at (-54.8, 70.2)
- added Q13: NDS8434, mainboard:NDS8434, F.Cu at (69.3, 46.1)
- added Q14: IRLML2803, mainboard:SOT-23, F.Cu at (-37.4, 57.6)
- added Q16: IRLML2803, mainboard:SOT-23, F.Cu at (-62.3, 57.6)
- added Q18: IRLML2803, mainboard:SOT-23, F.Cu at (-49.9, 57.6)
- added Q2: NDS8434, mainboard:NDS8434, F.Cu at (-67.2, 70.2)
- added Q3: IRLML2803, mainboard:SOT-23, F.Cu at (-10.8, 71.9)
- added Q4: NDS8434, mainboard:NDS8434, F.Cu at (-42.3, 59.8)
- added Q5: IRLML2803, mainboard:SOT-23, F.Cu at (-23.2, 71.9)
- added Q7: NDS8434, mainboard:NDS8434, F.Cu at (-67.2, 59.8)
- added Q8: IRLML2803, mainboard:SOT-23, F.Cu at (-49.9, 68.0)
- added Q9: NDS8434, mainboard:NDS8434, F.Cu at (-54.8, 59.8)
- added R16: 10k, Resistor_SMD:R_0603_1608Metric, F.Cu at (-13.2, 25.1)
- added R20: 1k, Resistor_SMD:R_0603_1608Metric, F.Cu at (-13.2, 27.6)
- added R39: 10k, Resistor_SMD:R_0603_1608Metric, F.Cu at (-13.2, 30.1)
- added SW1: KMR231NG LFS, mainboard:BTN_KMR2_4.6X2.8, F.Cu at (-11.4, 65.5)
- added U1: ~, adcs:RM3100, B.Cu at (74.7, 108.7)
- added U2: BMI270, adcs:XDCR_BMI270, F.Cu at (57.2, 78.2)
- added U3: S1216V8, mainboard:S1216_24PIN_PACKAGE, F.Cu at (105.6, 105.4)
- added U4: EP2W+, mainboard:QFN32-5X5MM, F.Cu at (116.2, 100.8)
- added U5: ~, adcs:RM3100, F.Cu at (125.2, -28.5)
- added U6: TPS54226PWPR, mainboard:PWP14_2P31X2P46-L, F.Cu at (-27.3, 64.6)
- added U7: MR25H40MDF, mainboard:SON127P600X500X90-9N, F.Cu at (-10.2, 60.1)
- added U8: MKL02Z32VFG4, adcs:QFN50P300X300X65-17N, F.Cu at (86.0, 71.5)
- added U9: BMI270, adcs:XDCR_BMI270, F.Cu at (57.2, 84.2)
- J14: value 353621050 -> Thruster
- R44: value 3.3k -> 100k
- moved R1 149.7 mm to (28.4, -29.5)
- moved R13 149.7 mm to (22.4, -27.0)
- moved R14 149.7 mm to (22.4, -24.5)
- moved R19 149.7 mm to (5.92, -18.1)
- moved R2 149.7 mm to (28.4, -27.0)
- moved R21 149.7 mm to (5.92, -15.6)
- moved R22 149.7 mm to (5.92, -13.0)
- moved R3 149.7 mm to (28.4, -24.5)
- moved R41 149.7 mm to (-0.09, -18.1)
- moved R43 149.7 mm to (-0.09, -15.6)
- moved R44 149.7 mm to (-0.09, -13.0)
- moved R45 149.7 mm to (28.4, -15.0)
- moved R46 149.7 mm to (-1.45, -37.4)
- moved R47 149.7 mm to (-1.45, -34.9)
- moved R48 149.7 mm to (-1.45, -32.4)
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Connections:
- IC1 pad A11: /GPS/RX_GPS -> /TX_TO_GPS
- IC1 pad B11: /GPS/TX_GPS -> /RX_FROM_GPS
- IC1 pad L11: /RX_ADCS -> /RX_FROM_PYCUBED
- IC1 pad M12: /TX_ADCS -> /TX_TO_PYCUBED
Other:
- board size 36.2 x 47.6 mm -> 99 x 99 mm

Commit message: update main board
Parts:
- removed the C1 at (-25.7, 12.5)
- removed the C1 at (82.4, 40.6)
- removed the C2 at (82.4, 43.1)
- removed the C2 at (-25.7, 15.0)
- removed the C3 at (82.4, 45.6)
- removed the C3 at (-31.7, 12.5)
- removed the C30 at (-27.7, 0.44)
- removed the C31 at (-27.7, 2.95)
- removed the C4 at (-31.7, 15.0)
- removed the C4 at (82.4, 48.1)
- removed the C5 at (-11.6, -4.58)
- removed the C5 at (76.4, 40.6)
- removed C52, C59: 0.22uF, Capacitor_SMD:C_0603_1608Metric
- removed C57, C58: 0.1uF, Capacitor_SMD:C_0603_1608Metric
- removed the C6 at (-11.6, -2.07)
- removed the C6 at (76.4, 43.1)
- removed C60, C62: 10nF, Capacitor_SMD:C_0603_1608Metric
- removed C61, C63: 4.7uF, Capacitor_SMD:C_0603_1608Metric
- removed D5: BAT54C, Package_TO_SOT_SMD:SOT-23
- removed the J10 at (32.0, 62.1)
- removed J21, J24: Conn_01x06, mainboard:MOLEX_35362-0650
- removed the J22 at (39.8, 112.6)
- removed the J23 at (46.9, 112.6)
- removed the J25 at (39.9, 96.8)
- removed the J8 at (107.8, 76.4)
- removed Q16, Q18: IRLML2803, mainboard:SOT-23
- removed the R1 at (44.2, 14.2)
- removed the R1 at (82.4, 50.6)
- removed the R1 at (28.4, -29.5)
- removed the R13 at (64.2, 11.7)
- removed the R13 at (22.4, -27.0)
- removed the R14 at (22.4, -24.5)
- removed the R14 at (64.2, 14.2)
- removed the R19 at (72.7, -11.2)
- removed the R19 at (5.92, -18.1)
- removed the R2 at (86.4, 40.6)
- removed the R2 at (28.4, -27.0)
- removed the R2 at (44.2, 16.7)
- removed the R21 at (5.92, -15.6)
- removed the R21 at (72.7, -8.66)
- removed the R22 at (5.92, -13.0)
- removed the R22 at (72.7, -6.15)
- removed the R3 at (28.4, -24.5)
- removed the R3 at (86.4, 43.1)
- removed the R3 at (64.2, 9.16)
- removed the R31 at (54.2, 16.7)
- removed the R31 at (86.4, 45.6)
- removed the R32 at (54.2, 19.2)
- removed the R32 at (86.4, 48.1)
- removed the R33 at (58.2, 9.16)
- removed the R33 at (86.4, 50.6)
- removed the R5 at (28.4, -20.0)
- removed the R5 at (76.4, 48.1)
- removed R51: 0, Resistor_SMD:R_0603_1608Metric
- removed R52, R55: 10K, Resistor_SMD:R_0603_1608Metric
- removed R53, R56: 4.7K, Resistor_SMD:R_0603_1608Metric
- removed R54, R57: 3.3k, Resistor_SMD:R_0603_1608Metric
- removed the R6 at (76.4, 50.6)
- removed the R6 at (28.4, -17.5)
- removed the R7 at (44.2, 19.2)
- removed the R7 at (22.4, -29.5)
- removed the U5 at (125.2, -28.5)
- removed the U7 at (-10.2, 60.1)
- removed the Y1 at (97.0, 18.8)
- added C1: 22uF, Capacitor_SMD:C_0603_1608Metric, F.Cu at (152.1, 31.9)
- added C2: 22uF, Capacitor_SMD:C_0603_1608Metric, F.Cu at (152.1, 34.4)
- added C3: 100uF, Capacitor_SMD:C_1210_3225Metric, F.Cu at (175.5, 50.4)
- added C35: 4.7uF, Capacitor_SMD:C_0603_1608Metric, F.Cu at (182.6, 49.1)
- added C36: 0.1uF, Capacitor_SMD:C_0603_1608Metric, F.Cu at (152.1, 64.3)
- added C39: 0.1uF, Capacitor_SMD:C_0603_1608Metric, F.Cu at (158.1, 66.8)
- added C4: 100uF, Capacitor_SMD:C_1210_3225Metric, F.Cu at (175.5, 54.6)
- added C40: 10nF, Capacitor_SMD:C_0603_1608Metric, F.Cu at (182.6, 61.2)
- added C43: 4.7uF, Capacitor_SMD:C_0603_1608Metric, F.Cu at (194.7, 34.4)
- added C44: 10nF, Capacitor_SMD:C_0603_1608Metric, F.Cu at (194.7, 46.6)
- added C45: 4.7uF, Capacitor_SMD:C_0603_1608Metric, F.Cu at (194.7, 49.1)
- added C46: 10nF, Capacitor_SMD:C_0603_1608Metric, F.Cu at (182.6, 31.9)
- added C47: 4.7uF, Capacitor_SMD:C_0603_1608Metric, F.Cu at (182.6, 34.4)
- added C48: 10nF, Capacitor_SMD:C_0603_1608Metric, F.Cu at (170.2, 64.3)
- added C5: 0.1uF, Capacitor_SMD:C_0603_1608Metric, F.Cu at (152.1, 37.0)
- added C6: 4.7uF, Capacitor_SMD:C_0603_1608Metric, F.Cu at (152.1, 39.5)
- added D4: LED, LED_SMD:LED_0402_1005Metric, F.Cu at (156.7, 58.2)
- added F1: Fuse, Resistor_SMD:R_0805_2012Metric, F.Cu at (176.4, 32.2)
- added FB1: FerriteBead, Resistor_SMD:R_0805_2012Metric, F.Cu at (176.4, 35.1)
- added FB2: FerriteBead, Resistor_SMD:R_0805_2012Metric, F.Cu at (176.4, 38.1)
- added H1: MountingHole_Pad, MountingHole:MountingHole_3.2mm_M3_DIN965_Pad, F.Cu at (29.3, 29.2)
- added H2: MountingHole_Pad, MountingHole:MountingHole_3.2mm_M3_DIN965_Pad, F.Cu at (120.1, 29.6)
- added H3: MountingHole_Pad, MountingHole:MountingHole_3.2mm_M3_DIN965_Pad, F.Cu at (29.2, 119.6)
- added H4: MountingHole_Pad, MountingHole:MountingHole_3.2mm_M3_DIN965_Pad, F.Cu at (120.0, 119.2)
- added J12: Conn_01x10, Connector_PinHeader_1.27mm:PinHeader_1x10_P1.27mm_Vertical, F.Cu at (37.9, 33.9)
- added J14: Conn_01x10, Connector_PinHeader_1.27mm:PinHeader_1x10_P1.27mm_Vertical, F.Cu at (37.7, 50.7)
- added J3: 353620850, adcs:SHDR8W50P0X200_1X8_1830X550X850P, F.Cu at (49.4, 47.5)
- added J4: 353620850, adcs:SHDR8W50P0X200_1X8_1830X550X850P, F.Cu at (49.4, 69.3)
- added J6: 353620650, mainboard:MOLEX_35362-0650, F.Cu at (118.1, 47.0)
- added L2: 3.3uH, mainboard:L_2141, F.Cu at (161.8, 58.0)
- added L3: 4.7uH, Capacitor_SMD:C_0805_2012Metric, F.Cu at (174.9, 58.3)
- added Q15: NDS8434, mainboard:NDS8434, F.Cu at (200.0, 64.2)
- added Q6: IRLML2803, mainboard:SOT-23, F.Cu at (198.9, 41.2)
- added R1: 0, Resistor_SMD:R_0603_1608Metric, F.Cu at (164.2, 64.3)
- added R13: 10k, Resistor_SMD:R_0603_1608Metric, F.Cu at (172.2, 31.9)
- added R14: 100K, Resistor_SMD:R_0603_1608Metric, F.Cu at (172.2, 34.4)
- added R19: 10K, Resistor_SMD:R_0603_1608Metric, F.Cu at (182.6, 51.6)
- added R2: 0, Resistor_SMD:R_0603_1608Metric, F.Cu at (164.2, 66.8)
- added R21: 100k, Resistor_SMD:R_0603_1608Metric, F.Cu at (182.6, 56.6)
- added R22: 10k, Resistor_SMD:R_0603_1608Metric, F.Cu at (152.1, 69.3)
- added R3: 0, Resistor_SMD:R_0603_1608Metric, F.Cu at (164.2, 69.3)
- added R31: 10k, Resistor_SMD:R_0603_1608Metric, F.Cu at (158.1, 79.3)
- added R32: 10K, Resistor_SMD:R_0603_1608Metric, F.Cu at (194.7, 75.9)
- added R33: 10K, Resistor_SMD:R_0603_1608Metric, F.Cu at (182.6, 66.2)
- added R5: 0, Resistor_SMD:R_0603_1608Metric, F.Cu at (164.2, 74.3)
- added R6: 0, Resistor_SMD:R_0603_1608Metric, F.Cu at (164.2, 76.8)
- added R7: 73.2K, Resistor_SMD:R_0603_1608Metric, F.Cu at (168.2, 34.4)
- added U2: MR25H40MDF, mainboard:SON127P600X500X90-9N, F.Cu at (162.5, 51.6)
- added U4: RM3100 Dev Board, adcs:RM3100, F.Cu at (94.0, 109.0)
- added Y2: 24.0mHz, Crystal:Crystal_SMD_2016-4Pin_2.0x1.6mm, F.Cu at (176.1, 45.8)
- C10: value 22uF -> 3.3nF
- C11: value 22uF -> 1uF
- C12: value 100uF -> 4.7uF; footprint Capacitor_SMD:C_1210_3225Metric -> Capacitor_SMD:C_0603_1608Metric
- C13: value 100uF -> 0.22uF; footprint Capacitor_SMD:C_1210_3225Metric -> Capacitor_SMD:C_0603_1608Metric
- C14: value 0.1uF -> 10uF
- C15: value 3.3nF -> 0.22uF
- C16: value 1uF -> 4.7uF
- C18: value 0.22uF -> 10nF
- C19, C22: value 10uF -> 0.22uF
- C20, C25: value 4.7uF -> 0.22uF
- C23: value 0.22uF -> 4.7uF
- C24: value 2.2uF -> 0.22uF
- C26: value 0.22uF -> 2.2uF
- C27: value 4.7uF -> 10uF
- C28, C29: value 0.22uF -> 10uF
- C32, C33: value 10nF -> 10pF
- C34, C42: value 4.7uF -> 10nF
- C41: value 10nF -> 4.7uF
- C49: value 0.1uF -> 4.7uF
- C50: value 10uF -> 10nF
- C8: value 10pF -> 0.22uF
- C9: value 10pF -> 0.1uF
- D2: value LED -> TVS Diode; footprint LED_SMD:LED_0402_1005Metric -> Package_TO_SOT_SMD:SOT-143
- D3: value SP0503BAHT -> BAT54C; footprint Package_TO_SOT_SMD:SOT-143 -> Package_TO_SOT_SMD:SOT-23
- J1, J2: value Amphenol_901-144 -> 353620650; footprint mainboard:SMA_901-144-horizontal -> mainboard:MOLEX_35362-0650
- J10: renamed from J14; value Thruster -> Thruster Connector
- J13: value 35362-0650 -> Conn_01x10; footprint mainboard:MOLEX_35362-0650 -> Connector_PinHeader_1.27mm:PinHeader_1x10_P1.27mm_Vertical
- J15, J17: value Conn_01x10 -> 353620650; footprint Connector_PinHeader_1.27mm:PinHeader_1x10_P1.27mm_Vertical -> mainboard:MOLEX_35362-0650
- J16, J18: value 35362-0650 -> 353620650
- J19, J20: value 353621050 -> 353620650; footprint adcs:CON_353621050 -> mainboard:MOLEX_35362-0650
- J26: value Conn_01x06 -> SMA-J-P-H-ST-EM1; footprint mainboard:MOLEX_35362-0650 -> adcs:SAMTEC_SMA-J-P-H-ST-EM1
- J27: value Conn_01x10 -> SMA-J-P-H-ST-EM1; footprint Connector_PinHeader_1.27mm:PinHeader_1x10_P1.27mm_Vertical -> adcs:SAMTEC_SMA-J-P-H-ST-EM1
- J5: renamed from J28; value 35362-0650 -> 353620650
- J8: renamed from J7; value Conn_01x08 -> Control Debug Header
- J9: value 35362-0650 -> 353620850; footprint mainboard:MOLEX_35362-0650 -> adcs:SHDR8W50P0X200_1X8_1830X550X850P
- L1: value 3.3uH -> 330uH; footprint mainboard:L_2141 -> adcs:IND_SRN6045TA-331K
- Q1, Q3, Q5: value IRLML2803 -> NDS8434; footprint mainboard:SOT-23 -> mainboard:NDS8434
- Q10, Q12, Q2, Q4: value NDS8434 -> IRLML2803; footprint mainboard:NDS8434 -> mainboard:SOT-23
- R10: value 10k -> 22.1K
- R11, R12: value 10k -> 5.1k
- R16, R35: value 10k -> 100k
- R17: value 100k -> 1k
- R18, R23, R30: value 10K -> 10k
- R20: value 1k -> 4.7K
- R24: value 4.7K -> 10k
- R25: value 1k -> 10k
- R26: value 3.3K -> 10k
- R27: value 73.2K -> 10k
- R28: value 22.1K -> 10k
- R29: value 100K -> 10k
- R34, R40: value 10k -> 4.7K
- R36, R39: value 10k -> 10K
- R37: value 5.1k -> 4.7K
- R38: value 5.1k -> 3.3k
- R4: value 10K -> 0
- R41: value 10K -> 3.3k
- R42: value 100K -> 10K
- R44: value 100k -> 3.3k
- R45: value 100k -> 10K
- R46, R49: value 0 -> 4.7K
- R47, R50: value 0 -> 3.3k
- R48: value 0 -> 10K
- R8: value 10k -> 1k
- R9: value 10k -> 100K
- U1: value ~ -> TPS54226PWPR; footprint adcs:RM3100 -> mainboard:PWP14_2P31X2P46-L; moved to F.Cu
- U6: value TPS54226PWPR -> RM3100 Dev Board; footprint mainboard:PWP14_2P31X2P46-L -> adcs:RM3100
- U8: renamed from U3; value S1216V8 -> Orion B16; moved to B.Cu
- U9: renamed from U4; moved to B.Cu
- moved Q7 268.4 mm to (200.0, 34.9)
- moved Q9 255.0 mm to (200.0, 49.5)
- moved Q2 254.4 mm to (186.8, 55.8)
- moved Q8 249.0 mm to (198.9, 55.8)
- moved Q14 236.6 mm to (198.9, 70.4)
- moved Q1 232.8 mm to (169.9, 52.5)
- moved Q4 229.4 mm to (186.8, 70.4)
- moved Q12 229.2 mm to (174.4, 73.5)
- moved C51 228.7 mm to (194.7, 63.7)
- moved C50 228.6 mm to (194.7, 61.2)
- moved Q11 219.6 mm to (187.9, 34.9)
- moved R48 219.5 mm to (194.7, 66.2)
- moved R49 219.5 mm to (194.7, 68.7)
- moved R50 219.5 mm to (194.7, 71.3)
- moved C42 215.0 mm to (194.7, 31.9)
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- renumbered C48 to C30, C47 to C31, J5 to J22, J4 to J23, J3 to J25, J6 to J7, U8 to U3, U2 to U5, U9 to U7, Y2 to Y1
Connections:
- C10 pad 1: GND -> Net-(U1-SS)
- C10 pad 2: +3V3 -> GND
- C11 pad 1: GND -> Net-(U1-VREG5)
- C11 pad 2: +3V3 -> GND
- C12 pad 1: /VBATT -> Net-(IC1-NVCC_PLL)
- C13 pad 1: /VBATT -> Net-(IC1-NVCC_PLL)
- C14 pad 1: Net-(U6-SW1) -> Net-(IC1-VDD_USB_CAP)
- C14 pad 2: Net-(U6-VBST) -> GND
- C15 pad 1: Net-(U6-SS) -> Net-(IC1-DCDC__IN_Q)
- C16 pad 1: Net-(U6-VREG5) -> Net-(IC1-DCDC__IN_Q)
- C18 pad 1: Net-(IC1-DCDC_IN_1) -> Net-(IC1-DCDC_SENSE)
- C19 pad 1: Net-(IC1-DCDC_IN_1) -> Net-(IC1-VDD_SNVS_CAP)
- C20 pad 1: Net-(IC1-DCDC__IN_Q) -> Net-(IC1-VDD_USB_CAP)
- C23 pad 1: Net-(IC1-DCDC__IN_Q) -> Net-(IC1-DCDC_SENSE)
- C24 pad 1: Net-(IC1-DCDC__IN_Q) -> Net-(IC1-DCDC_IN_1)
- C25 pad 1: Net-(IC1-VDD_HIGH_CAP) -> Net-(IC1-DCDC_SENSE)
- C26 pad 1: Net-(IC1-VDD_HIGH_CAP) -> Net-(IC1-DCDC__IN_Q)
- C27 pad 1: Net-(IC1-NVCC_PLL) -> Net-(IC1-DCDC__IN_Q)
- C28 pad 1: Net-(IC1-NVCC_PLL) -> Net-(IC1-DCDC_IN_1)
- C29 pad 1: Net-(IC1-VDD_SNVS_CAP) -> Net-(IC1-DCDC_SENSE)
- C32 pad 1: Net-(IC1-DCDC_SENSE) -> Net-(IC1-RTC_XTALO)
- C33 pad 1: /3V3_PD2 -> Net-(IC1-RTC_XTALI)
- C33 pad 2: Net-(C33-Pad2) -> GND
- C34 pad 1: /3V3_PD2 -> /Coil Power Enable/VBUS_OUT
- C34 pad 2: Net-(C33-Pad2) -> Net-(C34-Pad2)
- C38 pad 1: /IMU1_and_MAG1/3V3_SENSORS -> /IMU2_and_MAG2/3V3_SENSORS
- C41 pad 1: /IMU1_and_MAG1/3V3_SENSORS -> /VBATT
- C41 pad 2: Net-(C41-Pad2) -> Net-(C40-Pad2)
- C42 pad 2: Net-(C41-Pad2) -> Net-(C42-Pad2)
- C49 pad 1: 3.3V -> /3V3_PD1
- C49 pad 2: GND -> Net-(C48-Pad2)
- C50 pad 1: Net-(IC1-DCDC_SENSE) -> /3V3_PD2
- C50 pad 2: GND -> Net-(C50-Pad2)
- C51 pad 1: Net-(IC1-DCDC_SENSE) -> /3V3_PD2
- C51 pad 2: GND -> Net-(C50-Pad2)
- C7 pad 1: GNDREF -> Net-(IC1-VDD_HIGH_CAP)
- C7 pad 2: +5VD -> GND
- C8 pad 1: Net-(IC1-RTC_XTALI) -> Net-(IC1-VDD_HIGH_CAP)
- C9 pad 1: Net-(IC1-RTC_XTALO) -> 3.3V
- D1 pad 1: GND -> Net-(D1-K)
- D1 pad 2: Net-(D1-A) -> +3V3
- D2 pad 1: Net-(D2-K) -> GNDREF
- D2 pad 2: +3V3 -> +5VD
- D3 pad 1: GNDREF -> Net-(IC1-VDD_USB_CAP)
- D3 pad 2: +5VD -> 3.3V
- D3 pad 3: /MCU/USB1_D- -> Net-(IC1-VDD_SNVS_IN)
- J1 pad 1: Net-(J1-In) -> /3V3_PD2
- J11 pad 1: /MCU/GPIO_B1_02 -> /MCU/GPIO_B1_10
- J11 pad 2: /MCU/GPIO_B1_03 -> /MCU/GPIO_B1_11
- J11 pad 3: /MCU/GPIO_B1_04 -> /MCU/GPIO_B1_12
- J11 pad 4: /MCU/GPIO_B1_05 -> /MCU/GPIO_B1_13
- J11 pad 5: /MCU/GPIO_B1_07 -> /MCU/GPIO_B1_14
- J11 pad 6: /MCU/GPIO_B1_09 -> /MCU/GPIO_B1_15
- J11 pad 7: /MCU/GPIO_EMC_18 -> /MCU/GPIO_EMC_00
- J11 pad 8: /MCU/GPIO_EMC_19 -> /MCU/GPIO_EMC_03
- J11 pad 9: /MCU/GPIO_EMC_20 -> /MCU/GPIO_EMC_04
- J13 pad 1: /3V3_PD1 -> /MCU/GPIO_B0_08
- J13 pad 2: GND -> /MCU/GPIO_B0_09
- J13 pad 3: /MCU/GPIO_AD_B0_12 -> /MCU/GPIO_B0_10
- J13 pad 4: GND -> /MCU/GPIO_B0_11
- J13 pad 5: /MCU/GPIO_AD_B0_13 -> /MCU/GPIO_B0_12
- J13 pad 6: GND -> /MCU/GPIO_B0_14
- J15 pad 1: /MCU/GPIO_B0_08 -> /SCL2
- J15 pad 2: /MCU/GPIO_B0_09 -> /SDA2
- J15 pad 3: /MCU/GPIO_B0_10 -> GND
- J15 pad 4: /MCU/GPIO_B0_11 -> +3V3
- J15 pad 5: /MCU/GPIO_B0_12 -> /Coil Power Enable/VBUS_OUT
- J15 pad 6: /MCU/GPIO_B0_14 -> Net-(J15-Pin_6)
- J16 pad 1: /3V3_PD2 -> /SCL4
- J16 pad 2: GND -> /SDA4
- J16 pad 3: /MCU/GPIO_AD_B1_08 -> GND
- J16 pad 4: GND -> +3V3
- J16 pad 5: /MCU/GPIO_AD_B1_09 -> /Coil Power Enable/VBUS_OUT
- J16 pad 6: GND -> Net-(J16-Pin_6)
- J17 pad 1: /MCU/GPIO_SD_B1_00 -> /SCL4
- J17 pad 2: /MCU/GPIO_SD_B1_01 -> /SDA4
- J17 pad 3: /MCU/GPIO_SD_B1_02 -> GND
- J17 pad 4: /MCU/GPIO_SD_B1_03 -> +3V3
- J17 pad 5: /MCU/GPIO_AD_B1_14 -> /Coil Power Enable/VBUS_OUT
- J17 pad 6: /MCU/GPIO_AD_B1_15 -> Net-(J17-Pin_6)
- J18 pad 1: /3V3_PD1 -> /SCL2
- J18 pad 2: GND -> /SDA2
- J18 pad 3: /MCU/GPIO_AD_B0_14 -> GND
- J18 pad 4: GND -> +3V3
- J18 pad 5: /MCU/GPIO_AD_B0_15 -> /Coil Power Enable/VBUS_OUT
- J18 pad 6: GND -> Net-(J18-Pin_6)
- J19 pad 1: /3V3_PD2 -> /SCL4
- J19 pad 2: GND -> /SDA4
- J19 pad 3: /MCU/GPIO_AD_B1_10 -> GND
- J19 pad 4: GND -> +3V3
- J19 pad 5: /MCU/GPIO_AD_B1_11 -> /Coil Power Enable/VBUS_OUT
- J19 pad 6: GND -> Net-(J19-Pin_6)
- J2 pad 1: Net-(J2-In) -> /3V3_PD1
- J20 pad 1: /3V3_PD1 -> /SCL4
- J20 pad 2: GND -> /SDA4
- J20 pad 3: /MCU/GPIO_AD_B1_00 -> GND
- J20 pad 4: GND -> +3V3
- J20 pad 5: /MCU/GPIO_AD_B1_01 -> /Coil Power Enable/VBUS_OUT
- J20 pad 6: GND -> Net-(J20-Pin_6)
- J26 pad 1: /SCL4 -> Net-(U9-PORT2)
- J27 pad 1: +3V3 -> Net-(U9-PORT1)
- J9 pad 2: GND -> /MCU/ONOFF
- J9 pad 3: GND -> /MCU/WAKEUP
- J9 pad 4: GND -> /MCU/PMIC_STBY_REQ
- J9 pad 5: GND -> /MCU/POR_B
- J9 pad 6: GND -> /RX_FROM_PYCUBED
- L1 pad 1: Net-(U6-SW1) -> /VBATT_IN
- L1 pad 2: +3V3 -> /ADCS Power Enable/VBUS_IN
- Q1 pad 1: Net-(Q1-G) -> +5V
- Q1 pad 2: GND -> +5V
- Q1 pad 3: Net-(Q1-D) -> +5V
- Q10 pad 1: +3V3 -> Net-(Q10-G)
- Q10 pad 2: +3V3 -> GND
- Q10 pad 3: +3V3 -> Net-(Q10-D)
- Q11 pad 4: Net-(Q11-Gate) -> Net-(Q10-D)
- Q11 pad 5: /3V3_PD1 -> /GPS/3V3_GPS
- Q11 pad 6: /3V3_PD1 -> /GPS/3V3_GPS
- Q11 pad 7: /3V3_PD1 -> /GPS/3V3_GPS
- Q11 pad 8: /3V3_PD1 -> /GPS/3V3_GPS
- Q12 pad 1: +3V3 -> Net-(Q12-G)
- Q12 pad 2: +3V3 -> GND
- Q12 pad 3: +3V3 -> Net-(Q12-D)
- Q13 pad 1: +5V -> +3V3
- Q13 pad 2: +5V -> +3V3
- Q13 pad 3: +5V -> +3V3
- Q13 pad 4: GND -> Net-(Q12-D)
- Q13 pad 5: Net-(FB1-Pad2) -> /3V3_PD1
- Q13 pad 6: Net-(FB1-Pad2) -> /3V3_PD1
- Q13 pad 7: Net-(FB1-Pad2) -> /3V3_PD1
- Q13 pad 8: Net-(FB1-Pad2) -> /3V3_PD1
- Q2 pad 1: /VBATT -> Net-(Q2-G)
- Q2 pad 2: /VBATT -> GND
- Q2 pad 3: /VBATT -> Net-(Q2-D)
- Q3 pad 1: Net-(Q3-G) -> /VBATT
- Q3 pad 2: GND -> /VBATT
- Q3 pad 3: Net-(Q10-Gate) -> /VBATT
- Q4 pad 1: GND -> Net-(Q4-G)
- Q4 pad 3: GND -> Net-(Q4-D)
- Q5 pad 1: Net-(Q5-G) -> /ADCS Power Enable/VBUS_IN
- Q5 pad 2: GND -> /ADCS Power Enable/VBUS_IN
- Q5 pad 3: Net-(Q11-Gate) -> /ADCS Power Enable/VBUS_IN
- Q7 pad 4: Net-(Q16-D) -> Net-(Q6-D)
- Q8 pad 3: Net-(Q12-Gate) -> Net-(Q8-D)
- Q9 pad 4: Net-(Q18-D) -> Net-(Q8-D)
- R10 pad 1: Net-(U1-I2CEN) -> GND
- R10 pad 2: /IMU1_and_MAG1/3V3_SENSORS -> Net-(U1-VFB)
- R11 pad 1: /IMU1_and_MAG1/3V3_SENSORS -> GNDREF
- R11 pad 2: /SCL2 -> /MCU/USB1_CC1
- R12 pad 1: /IMU1_and_MAG1/3V3_SENSORS -> GNDREF
- R12 pad 2: /SDA2 -> /MCU/USB1_CC2
- R15 pad 1: /MCU/SD.DAT3 -> /MCU/FLASH.IO3
- R16 pad 1: /MCU/FLASH.IO3 -> GND
- R16 pad 2: 3.3V -> /MCU/JTAG.MUX.TRSTB
- R17 pad 1: GND -> Net-(IC1-GPIO_B0_03)
- R17 pad 2: /MCU/JTAG.MUX.TRSTB -> Net-(D4-A)
- R18 pad 1: Net-(U3-RSTN) -> GND
- R18 pad 2: /GPS/3V3_GPS -> /MCU/PMIC_STBY_REQ
- R20 pad 1: Net-(IC1-GPIO_B0_03) -> /EN_COILS
- R20 pad 2: Net-(D1-A) -> Net-(Q2-G)
- R23 pad 1: /MCU/GPIO_B0_07 -> GND
- R23 pad 2: GND -> Net-(U4-SSN/ADDR0)
- R24 pad 1: /MCU/GPIO_B0_07 -> Net-(U4-I2CEN)
- R24 pad 2: Net-(Q10-G) -> /IMU1_and_MAG1/3V3_SENSORS
- R25 pad 1: Net-(U8-PTB3) -> /IMU1_and_MAG1/3V3_SENSORS
- R25 pad 2: Net-(D2-K) -> /SCL2
- R26 pad 1: 3V3 -> /IMU1_and_MAG1/3V3_SENSORS
- R26 pad 2: Net-(Q10-D) -> /SDA2
- R27 pad 1: Net-(U6-VFB) -> GND
- R27 pad 2: +3V3 -> Net-(U6-SO/ADDR1)
- R28 pad 2: Net-(U6-VFB) -> Net-(U6-SSN/ADDR0)
- R29 pad 1: Net-(U6-PG) -> Net-(U6-I2CEN)
- R29 pad 2: Net-(U6-VREG5) -> /IMU2_and_MAG2/3V3_SENSORS
- R30 pad 1: /IMU2_and_MAG2/EN_SENSOR -> /IMU2_and_MAG2/3V3_SENSORS
- R30 pad 2: GND -> /SCL4
- R34 pad 2: Net-(U5-SSN/ADDR0) -> Net-(Q4-G)
- R35 pad 1: Net-(U5-I2CEN) -> /ADCS Power Enable/VBUS_IN
- R35 pad 2: /IMU2_and_MAG2/3V3_SENSORS -> Net-(Q4-D)
- R36 pad 1: /IMU2_and_MAG2/3V3_SENSORS -> /IMU1_and_MAG1/EN_SENSORS
- R36 pad 2: /SCL4 -> GND
- R37 pad 1: GNDREF -> /IMU1_and_MAG1/EN_SENSORS
- R37 pad 2: /MCU/USB1_CC1 -> Net-(Q6-G)
- R38 pad 1: GNDREF -> +3V3
- R38 pad 2: /MCU/USB1_CC2 -> Net-(Q6-D)
- R39 pad 1: GND -> /IMU2_and_MAG2/EN_SENSORS
- R39 pad 2: /MCU/PMIC_STBY_REQ -> GND
- R4 pad 1: /EN_ADCS -> /MCU/GPIO_EMC_39
- R4 pad 2: GND -> Net-(J18-Pin_6)
- R40 pad 1: /IMU2_and_MAG2/3V3_SENSORS -> /IMU2_and_MAG2/EN_SENSORS
- R40 pad 2: /SDA4 -> Net-(Q8-G)
- R41 pad 1: GND -> +3V3
- R41 pad 2: GND -> Net-(Q8-D)
- R42 pad 1: Net-(IC1-PMIC_ON_REQ) -> /GPS/EN_GPS
- R42 pad 2: +3V3 -> GND
- R43 pad 1: GND -> /GPS/EN_GPS
- R43 pad 2: Net-(Q14-G) -> Net-(Q10-G)
- R44 pad 1: GND -> +3V3
- R44 pad 2: Net-(Q14-D) -> Net-(Q10-D)
- R45 pad 1: /VBATT -> /MCU/GPIO_B0_07
- R45 pad 2: Net-(Q1-D) -> GND
- R46 pad 1: /MCU/GPIO_EMC_05 -> /MCU/GPIO_B0_07
- R46 pad 2: Net-(J23-Pin_6) -> Net-(Q12-G)
- R47 pad 1: /MCU/GPIO_EMC_06 -> +3V3
- R47 pad 2: Net-(J24-Pin_6) -> Net-(Q12-D)
- R48 pad 1: /MCU/GPIO_EMC_34 -> /MCU/GPIO_B0_06
- R48 pad 2: Net-(J21-Pin_6) -> GND
- R49 pad 1: /MCU/GPIO_EMC_39 -> /MCU/GPIO_B0_06
- R49 pad 2: Net-(J22-Pin_6) -> Net-(Q14-G)
- R50 pad 1: /MCU/GPIO_AD_B0_01 -> +3V3
- R50 pad 2: Net-(J25-Pin_6) -> Net-(Q14-D)
- R8 pad 1: GND -> Net-(U3-PTB3)
- R8 pad 2: Net-(U1-SO/ADDR1) -> Net-(D1-K)
- R9 pad 1: GND -> Net-(IC1-PMIC_ON_REQ)
- R9 pad 2: Net-(U1-SSN/ADDR0) -> +3V3
- U1 pad 1: /SCL2 -> +3V3
- U1 pad 2: Net-(U1-SO/ADDR1) -> Net-(U1-VFB)
- U1 pad 3: /SDA2 -> Net-(U1-VREG5)
- U1 pad 4: Net-(U1-SSN/ADDR0) -> Net-(U1-SS)
- U1 pad 5: /IMU1_and_MAG1/DRDY_MAG -> GND
- U1 pad 6: unconnected-(U1-NC-Pad6) -> Net-(U1-PG)
- U1 pad 7: GND -> Net-(IC1-PMIC_ON_REQ)
- U3 pad 11: Net-(U8-PTB3) -> Net-(U3-PTB3)
- U6 pad 1: +3V3 -> /SCL4
- U6 pad 10: Net-(U6-SW1) -> Net-(U6-I2CEN)
- U6 pad 11: Net-(U6-SW1) -> unconnected-(U6-NC-Pad11)
- U6 pad 12: Net-(U6-VBST) -> /IMU2_and_MAG2/3V3_SENSORS
- U6 pad 13: /VBATT -> /IMU2_and_MAG2/3V3_SENSORS
- U6 pad 14: /VBATT -> GND
- U6 pad 2: Net-(U6-VFB) -> Net-(U6-SO/ADDR1)
- U6 pad 3: Net-(U6-VREG5) -> /SDA4
- U6 pad 4: Net-(U6-SS) -> Net-(U6-SSN/ADDR0)
- U6 pad 5: GND -> /IMU2_and_MAG2/DRDY_MAG
- U6 pad 6: Net-(U6-PG) -> unconnected-(U6-NC-Pad6)
- U6 pad 7: Net-(IC1-PMIC_ON_REQ) -> GND
- U6 pad 8: GND -> unconnected-(U6-NC-Pad8)
- U6 pad 9: GND -> unconnected-(U6-NC-Pad9)
- U8 pad 8: Net-(U3-RSTN) -> Net-(U8-RSTN)
- U9 pad 15: Net-(J1-In) -> Net-(U9-PORT1)
- U9 pad 26: Net-(J2-In) -> Net-(U9-PORT2)
