File: sqrt_of_g/imu_and_magnetometer.kicad_sch (KiCad schematic)
At the start: 18 parts, among them Q12 IRLML2803, Q13 NDS8434, U9 BMI270

Commit message: ready for 2nd round of reviews
Parts:
- removed C32: 10nF, symbol pycubed_mainboard:10NF_10000PF-50V-10%(0603)
- removed C50: 10uF, symbol pycubed_mainboard:10NF_10000PF-50V-10%(0603)
- removed C51: 4.7uF, symbol pycubed_mainboard:10NF_10000PF-50V-10%(0603)
- removed C52: 0.22uF, symbol pycubed_mainboard:10NF_10000PF-50V-10%(0603)
- removed Q12: IRLML2803, mainboard:SOT-23, symbol mainboard:IRLML2803TRPBF
- removed Q13: NDS8434, mainboard:NDS8434, symbol mainboard:NDS8434
- removed R30: 10K, Resistor_SMD:R_0603_1608Metric, symbol mainboard:R-US_R0603
- removed R31: 4.7K, Resistor_SMD:R_0603_1608Metric, symbol mainboard:R-US_R0603
- removed R32: 3.3K, Resistor_SMD:R_0603_1608Metric, symbol mainboard:R-US_R0603
Connections:
- net 3V3_SENSOR is gone; now on net 3V3_SENSORS: C57.1, C58.1, U9.5 (VDDIO), U9.8 (VDD)
- net 3V3_SENSORS: now also U9.10 (OSCB)
- net 3.3V: no longer names the net of U9.12 (CSB)
Other:
- added sheet Enable (power_enable.kicad_sch)
- note added: "Symbol/footprint for this is the Dev board, which has shipped. The components themselves has a 10-week lead time"
- note removed: "IMU+Mag Power"
- moved on the sheet: C57, C58, R33, R34, R35, R36, R40, U5

Commit message: pete feedback
Other:
- company: (none) -> Stanford Student Space Initiative
- moved on the sheet: C57, C58, R33, R34, R35, R36, R40, U5, U9

Commit message: update board
Parts:
- U5: footprint (none) -> adcs:RM3100
- U9: footprint Sensor_Motion:XDCR_BMI270 -> adcs:XDCR_BMI270
Changed lines of the file:
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@@
       (effects (font (size 1.27 1.27)))
     )
-    (property "Footprint" "Sensor_Motion:XDCR_BMI270" (at 212.09 95.5802 0)
+    (property "Footprint" "adcs:XDCR_BMI270" (at 212.09 95.5802 0)
       (effects (font (size 1.27 1.27)) (justify bottom) hide)
     )
@@
       (effects (font (size 1.27 1.27)))
     )
-    (property "Footprint" "" (at 69.85 103.2002 0)
-      (effects (font (size 1.27 1.27)) hide)
-    )
+    (property "Footprint" "adcs:RM3100" (at 69.85 103.2002 0)
+      (effects (font (size 1.27 1.27)) hide)
+    )

Commit message: update main board
Parts:
- R27: renamed from R33; DNI (none) -> Mixed Values
- R28: renamed from R34; DNI (none) -> Mixed Values
- R29: renamed from R35; DNI (none) -> Mixed Values
- R30: renamed from R36; DNI (none) -> Mixed Values
- R31: renamed from R40; DNI (none) -> Mixed Values
- U6: renamed from U5; value ~ -> RM3100 Dev Board; Flight (none) -> RM3100; Manufacturer_Name (none) -> PNI Technologies; Unit Price (none) -> 25.0
- U7: renamed from U9; Flight (none) -> BMI270; MANUFACTURER Bosch Sensortec -> (none); MAXIMUM_PACKAGE_HEIGHT 0.87mm -> (none); Manufacturer_Name (none) -> Bosch Sensortec; PATREV 1.0 -> (none); STANDARD Manufacturer Recommendations -> (none); Unit Price (none) -> 5.88
- renumbered C57 to C38, C58 to C39
Other:
- note removed: "Symbol/footprint for this is the Dev board, which has shipped. The components themselves has a 10-week lead time"
