File: sqrt_of_g/microcontroller.kicad_sch (KiCad schematic)
At the start: 65 parts, among them IC1 MIMXRT1062DVJ6B, J3 503182-1852, J4 USB_C_pycubed, J5 JTAG_SWD_10, J6 Conn_01x06, Q6 DMG2305UX-7, SW1 KMR231NG LFS, U6 TPS54226PWPR, U7 MR25H40MDF, U8 MKL02Z32VFG4, Y1 24.0mHz, Y2 32.768kHz

Commit message: move mainboard to subdirectory
Parts:
- IC1: symbol adcs:MIMXRT1062DVJ6B -> adcs:MIMXRT1062DVJ6B_2
Changed lines of the file:
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@@
     )
   )
-  (symbol (lib_name "MIMXRT1062DVJ6B_2") (lib_id "adcs:MIMXRT1062DVJ6B") (at 196.2658 165.862 0) (unit 1)
+  (symbol (lib_id "adcs:MIMXRT1062DVJ6B_2") (at 196.2658 165.862 0) (unit 1)
     (in_bom yes) (on_board yes) (dnp no)
     (property "Reference" "IC1" (at 176.0728 41.6052 0)

Commit message: more schematic work... I was supposed to finish this a long time ago
Parts:
- added R16: 10k, symbol pycubed_mainboard:RESISTOR0603
- added TP1, TP2, TP3, TP4, TP5, TP6: TestPoint, symbol Connector:TestPoint
Connections:
- net 3.3V: now also R16.2
- net FLASH.IO3: now also R16.1
- net SD.CLK: now also TP4.1
- net SD.CMD: now also TP3.1
- net SD.DAT0: now also TP5.1
- net SD.DAT1: now also TP6.1
- net SD.DAT2: now also TP1.1
- net SD.DAT3: now also TP2.1
Other:
- note added: "4.5-18V"
- note added: "Double check component choice for space (BAT54C)"
- note removed: "Double check component choice for space"
- note removed: "Should I add a 1M resistor between shield and GNDREF?"
- note removed: "Should I put a pull-up on CS? - Pete votes no"
- note removed: "Should these be grounded or disconnected? Or, should I add PSRAM?"
- note removed: "pull up on CS?"

Commit message: ready for 2nd round of reviews
Parts:
- removed J6: Conn_01x06, Connector_PinHeader_2.54mm:PinHeader_1x06_P2.54mm_Vertical, symbol Connector_Generic:Conn_01x06
- removed U6: TPS54226PWPR, mainboard:PWP14_2P31X2P46-L, symbol mainboard:TPS54226PWPRPWP14_2P31X2P46-L
- added U6: TPS54226PWPR, mainboard:PWP14_2P31X2P46-L, symbol adcs:TPS54226PWPRPWP14_2P31X2P46-L
Connections:
- net +3V3: now also U6.1 (VO)
- net GND: now also U6.15 (EPAD), U6.5 (GND), U6.8 (PGND1), U6.9 (PGND2)
- net GPIO_AD_B0_03: no longer IC1.J14 (GPIO_AD_B1_15)
- net GPIO_AD_B1_04: no longer IC1.P2 (GPIO_SD_B1_04)
- net GPIO_AD_B1_05: no longer IC1.N3 (GPIO_SD_B1_05)
- net at C14.1, L1.1: now also U6.10 (SW1), U6.11 (SW2)
- net at C14.2: now also U6.12 (VBST)
- net at R27.1, R28.2: now also U6.2 (VFB)
- net at C16.1, R29.2: now also U6.3 (VREG5)
- net at C15.1: now also U6.4 (SS)
- net at R29.1: now also U6.6 (PG)
- net at IC1.K7 (PMIC_ON_REQ), R42.1: now also U6.7 (EN)
- net ADCS_VBATT renamed VBATT
- net VBATT: now also U6.13 (VIN), U6.14 (VCC)
- new net GPIO_AD_B1_15: IC1.J14 (GPIO_AD_B1_15)
- new net GPIO_SD_B1_04: IC1.P2 (GPIO_SD_B1_04)
- new net GPIO_SD_B1_05: IC1.N3 (GPIO_SD_B1_05)
Other:
- note added: "TODO: add inductor here"
- note added: "TODO: decide whether to break these out or put PSRAM"
- note added: "TODO: figure out what to do with these"
- note removed: ""EN""
- note removed: ""GND""
- note removed: ""VUSB""
- note removed: "Add jumper to allow USB battery charging (even inside deployer)."
- note removed: "RBF Jumpers"
- note removed: "Remove both jumpers before flight"
- note removed: "VADCS_IN is from the battery - after foot switches - after an ADCS board enable FET"
- note removed: "what do for these?"

Commit message: pete feedback
Parts:
- IC1: footprint BGA196C80P14X14_1200X1200X152 -> adcs:BGA196C80P14X14_1200X1200X152N
- R15: DNP (none) -> DNP
Other:
- company: (none) -> Stanford Student Space Initiative
- title: (none) -> RT1062_Careful_COTS
Changed lines of the file:
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@@
 (kicad_sch (version 20230121) (generator eeschema)
   (paper "B" portrait)
+  (title_block
+    (title "RT1062_Careful_COTS")
+    (date "2023-11-01")
+    (rev "1.0")
+    (company "Stanford Student Space Initiative")
+    (comment 1 "RE: Flynn Dreilinger")
+    (comment 2 "Reviewer 1: Pete Mahowald")
+    (comment 3 "Reviewer 2: Tim Vrakas")
+    (comment 4 "Reviewer 3: Grant Regen")
+  )
   (bus_alias "3V3_RAIL" (members "3V3" "GND"))
   (bus_alias "I2C" (members "SDA" "SCL"))
@@
     (stroke (width 0) (type default))
   )
-  (wire (pts (xy 253.3904 17.8054) (xy 256.5908 17.8054))
-    (stroke (width 0) (type default))
-  )
   (wire (pts (xy 169.5958 94.742) (xy 169.5958 92.202))
     (stroke (width 0) (type default))
@@
     (effects (font (size 1.27 1.27)) (justify right bottom))
   )
-  (global_label "GND" (shape input) (at 256.5908 17.8054 0) (fields_autoplaced)
-    (effects (font (size 1.27 1.27)) (justify left))
-    (property "Intersheetrefs" "${INTERSHEET_REFS}" (at 263.4465 17.8054 0)
-      (effects (font (size 1.27 1.27)) (justify left) hide)
-    )
-  )
   (hierarchical_label "GPIO_B1_15" (shape bidirectional) (at 222.9358 197.612 0) (fields_autoplaced)
     (effects (font (size 1.27 1.27)) (justify left))
@@
     )
   )
-  (symbol (lib_name "GND_2") (lib_id "power:GND") (at 253.3904 17.8054 0) (unit 1)
-    (in_bom yes) (on_board yes) (dnp no) (fields_autoplaced)
-    (property "Reference" "#PWR033" (at 253.3904 24.1554 0)
-      (effects (font (size 1.27 1.27)) hide)
-    )
-    (property "Value" "GND" (at 253.3904 22.3774 0)
-      (effects (font (size 1.27 1.27)))
-    )
-    (property "Footprint" "" (at 253.3904 17.8054 0)
-      (effects (font (size 1.27 1.27)) hide)
-    )
-    (property "Datasheet" "" (at 253.3904 17.8054 0)
-      (effects (font (size 1.27 1.27)) hide)
-    )
-    (pin "1")
-    (instances
-      (project "adcs-hardware"
-        (path "/2bf29f96-8e90-4c56-8856-49bc3b5fab50/3472706a-4f86-4fa0-acec-6a7dc1abcee9"
-          (reference "#PWR033") (unit 1)
-        )
-      )
-    )
-  )
   (symbol (lib_id "mainboard:C_Small") (at 246.5578 262.382 90) (mirror x) (unit 1)
     (in_bom yes) (on_board yes) (dnp no)
@@
       (effects (font (size 1.27 1.27)) hide)
     )
+    (property "DigiKey Part Number" "" (at 123.1138 159.512 0)
+      (effects (font (size 1.27 1.27)) hide)
+    )
+    (property "Tolerance" "" (at 123.1138 159.512 0)
+      (effects (font (size 1.27 1.27)))
+    )
+    (property "Power Rating" "" (at 123.1138 159.512 0)
+      (effects (font (size 1.27 1.27)))
+    )
+    (property "DNP" "DNP" (at 115.2144 158.3436 0)
+      (effects (font (size 1.27 1.27)))
+    )
     (pin "1")
     (pin "2")
@@
       (effects (font (size 1.27 1.27)))
     )
-    (property "Footprint" "BGA196C80P14X14_1200X1200X152" (at 238.1758 109.982 0)
+    (property "Footprint" "adcs:BGA196C80P14X14_1200X1200X152N" (at 238.1758 109.982 0)
       (effects (font (size 1.27 1.27)) (justify left) hide)
     )

Commit message: update board
Parts:
- removed Q6: DMG2305UX-7, DMG2305UX-7:SOT91P240X110-3N_DMG2305UX-7, symbol adcs:DMG2305UX-7
- added Q2: NDS8434, mainboard:NDS8434, symbol adcs:NDS8434
- C17, C18, C19, C20, C21, C22, C23, C24, C25, C26, C27, C28, C29, C30, C31, C32, C50, C51, C52, C59: footprint (none) -> Capacitor_SMD:C_0603_1608Metric
- R16, R20, R39: footprint (none) -> Resistor_SMD:R_0603_1608Metric
- U8: footprint Package_DFN_QFN:QFN-16-1EP_3x3mm_P0.5mm_EP1.8x1.8mm -> adcs:QFN50P300X300X65-17N
Connections:
- net +5V: now also Q2.1 (Source), Q2.2 (Source), Q2.3 (Source)
- net GND: now also Q2.4 (Gate)
- net at FB1.2: now also Q2.5 (Drain), Q2.6 (Drain), Q2.7 (Drain), Q2.8 (Drain)
Other:
- note added: "A latch up does not necessarily cause the CPU has crashed. In fact it generally does not, and a software protection that detects increased current and power cycles the chip is totally valid. If you want to actually do this, you should do some analysis of the timing. A common way to do this is to have a capacitor on the enable pin, with a weak pull-up, and then an N-FET to ground. When you turn on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"
- note added: "Now I am thinking TCXO might be good here."

Commit message: update main board
Parts:
- removed TP1, TP2, TP3, TP4, TP5, TP6: TestPoint, symbol Connector:TestPoint
- added J24: SD Card Debug Header, Connector_PinHeader_2.54mm:PinHeader_1x08_P2.54mm_Vertical, symbol Connector_Generic:Conn_01x08
- D1: renamed from D2; footprint LED_SMD:LED_0402_1005Metric -> LED_SMD:LED_0603_1608Metric
- D2: renamed from D3; value SP0503BAHT -> TVS Diode; Flight (none) -> SP0503BAHTG; Manufacturer_Name (none) -> Littlefuse
- D3: renamed from D5; Flight (none) -> BAT54C; Manufacturer_Name (none) -> [Many]; Unit Price (none) -> 0.15
- D4: renamed from D1; footprint LED_SMD:LED_0402_1005Metric -> LED_SMD:LED_0603_1608Metric
- F1: footprint (none) -> Resistor_SMD:R_0805_2012Metric; Flight (none) -> 0ZCK0050FF2E; Manufacturer_Name (none) -> Bel Fuse
- FB1, FB2: footprint (none) -> Resistor_SMD:R_0805_2012Metric; Flight (none) -> MPZ2012S101ATD25; Manufacturer_Name (none) -> TDK Corporation
- IC1: Flight (none) -> MIMXRT1062DVJ6B; Height 1.52 -> (none); Manufacturer_Part_Number MIMXRT1062DVJ6B -> (none); Mouser Part Number 771-MIMXRT1062DVJ6B -> (none); Mouser Price/Stock https://www.mouser.co.uk/ProductDetail/NXP-Semiconductors/M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 -> (none); Unit Price (none) -> 15.93
- J22: renamed from J5; Flight (none) -> BD125-10-A-0305-0580-L-B; Manufacturer_Name (none) -> GCT
- J23: renamed from J4; Flight (none) -> U262-161N-4BVC11; Manufacturer_Name (none) -> XKB Connectivity; Supplier 1 (none) -> LCSC
- J25: renamed from J3; Manufacturer_Part_Number 5031821852 -> (none)
- L2: renamed from L1; Manufacturer_Part_Number HPC5040NF-3R3MTH -> (none)
- L3: footprint (none) -> Capacitor_SMD:C_0805_2012Metric; Flight (none) -> LQM21PN4R7MGRD; Manufacturer_Name (none) -> Murata Electronics
- Q?: renamed from Q2; Manufacturer_Part_Number NDS8434 -> (none)
- R13: renamed from R15; DNI (none) -> Mixed Values; DNP DNP -> (none)
- R15: renamed from R16; DNI (none) -> Mixed Values
- R18: renamed from R39; DNI (none) -> Mixed Values
- SW1: Manufacturer_Part_Number KMR231NG LFS -> (none)
- U1: renamed from U6; Manufacturer_Part_Number TPS54226PWPR -> (none); Proto TPS54226PWPR -> PS54226PWPR
- U2: renamed from U7; Manufacturer_Part_Number W25Q80DVSNIG -> (none); Unit Price (none) -> 35.95; Unit Price (Proto) (none) -> 0.50
- U3: renamed from U8; DNI (none) -> DNI; Flight (none) -> MKL02Z32VFG4; MFGR Supplied by PJRC -> (none); MPN Custom firmware part -> (none); Manufacturer_Name (none) -> PJRC
- Y1: renamed from Y2; Manufacturer_Part_Number SC-32S32.768kHz20PPM7pF -> (none); Proto SC-32S32.768kHz20PPM7pF -> (none)
- Y2: renamed from Y1; Manufacturer_Part_Number XRCGB24M000F1SBDR0 -> (none)
- renumbered C10 to C1, C15 to C10, C16 to C11, C27 to C12, C28 to C13, C31 to C14, C30 to C15, C20 to C16, C32 to C18, C29 to C19, C11 to C2, C59 to C20, C23 to C22, C51 to C23, C18 to C24, C52 to C25, C24 to C26, C22 to C27, C19 to C28, C50 to C29, C12 to C3, C48 to C30, C47 to C31, C9 to C32, C8 to C33, C13 to C4, C14 to C5, C7 to C6, C25 to C7, C26 to C8, C49 to C9, R28 to R10, R37 to R11, R38 to R12, R29 to R14, R17 to R16, R20 to R17, R27 to R7, R25 to R8, R42 to R9
Connections:
- net 3.3V: now also J24.1 (Pin_1)
- net GND: now also J24.8 (Pin_8)
- net SD.CLK: now also J24.5 (Pin_5)
- net SD.CMD: now also J24.4 (Pin_4)
- net SD.DAT0: now also J24.6 (Pin_6)
- net SD.DAT1: now also J24.7 (Pin_7)
- net SD.DAT2: now also J24.2 (Pin_2)
- net SD.DAT3: now also J24.3 (Pin_3)
