File: sqrt_of_g/power_enable.kicad_sch (KiCad schematic)
At the start: 7 parts, among them Q12 IRLML2803, Q13 NDS8434

Commit message: pete feedback
Parts:
- removed Q13: NDS8434, mainboard:NDS8434, symbol mainboard:NDS8434
- added Q2: NDS8434, mainboard:NDS8434, symbol adcs:NDS8434
- R32: value 3.3K -> ${source_resistor}
Connections:
- net VBUS_IN: now also Q2.1 (Source), Q2.2 (Source), Q2.3 (Source)
- net VBUS_OUT: now also Q2.5 (Drain), Q2.6 (Drain), Q2.7 (Drain), Q2.8 (Drain)
- net at Q12.3 (D), R32.2: now also Q2.4 (Gate)
Other:
- company: (none) -> Stanford Student Space Initiative
- moved on the sheet: C32, C51, Q12, R30, R31, R32

Commit message: update board
Parts:
- C32, C51: footprint (none) -> Capacitor_SMD:C_0603_1608Metric
Changed lines of the file:
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@@
       (effects (font (size 1.4986 1.4986)) (justify left))
     )
-    (property "Footprint" "" (at 171.7294 114.3762 0)
+    (property "Footprint" "Capacitor_SMD:C_0603_1608Metric" (at 171.7294 114.3762 0)
       (effects (font (size 1.27 1.27)) hide)
     )
     (property "Datasheet" "" (at 171.7294 114.3762 0)
       (effects (font (size 1.27 1.27)) hide)
+    )
+    (property "DigiKey Part Number" "" (at 171.7294 114.3762 0)
+      (effects (font (size 1.27 1.27)) hide)
+    )
+    (property "Tolerance" "" (at 171.7294 114.3762 0)
+      (effects (font (size 1.27 1.27)))
+    )
+    (property "Power Rating" "" (at 171.7294 114.3762 0)
+      (effects (font (size 1.27 1.27)))
     )
     (pin "1")
@@
       (effects (font (size 1.4986 1.4986)) (justify left))
     )
-    (property "Footprint" "" (at 164.1094 114.3762 0)
+    (property "Footprint" "Capacitor_SMD:C_0603_1608Metric" (at 164.1094 114.3762 0)
       (effects (font (size 1.27 1.27)) hide)
     )
@@
       (effects (font (size 1.27 1.27)) hide)
     )
-    (pin "1")
+    (property "DigiKey Part Number" "" (at 164.1094 114.3762 0)
+      (effects (font (size 1.27 1.27)) hide)
+    )
+    (property "Tolerance" "" (at 164.1094 114.3762 0)
+      (effects (font (size 1.27 1.27)))
+    )
+    (property "Power Rating" "" (at 164.1094 114.3762 0)
+      (effects (font (size 1.27 1.27)))
+    )
+    (pin "1")

Commit message: update main board
Parts:
- Q3: renamed from Q2; Manufacturer_Part_Number NDS8434 -> (none)
- Q?: renamed from Q12; Manufacturer_Part_Number IRLML2803TRPbF -> (none)
- renumbered C51 to C?, C32 to C?, R31 to R?, R32 to R?, R30 to R?
