File: sfh2430_breakout/sfh2430_breakout.kicad_pcb (KiCad board)
At the start: 2 copper layers, 37.8 x 65.6 mm, 18 parts, among them J2 Conn_01x10, U1 LTC2052IS_PBF

Commit message: work on sun pyramid
Parts:
- added H1: MountingHole_Pad, MountingHole:MountingHole_2.2mm_M2, F.Cu at (128.7, 116.3)
- added H2: MountingHole_Pad, MountingHole:MountingHole_2.2mm_M2, F.Cu at (139.3, 127.0)
- added H3: MountingHole_Pad, MountingHole:MountingHole_2.2mm_M2, F.Cu at (129.0, 137.0)
- added H4: MountingHole_Pad, MountingHole:MountingHole_2.2mm_M2, F.Cu at (118.0, 127.0)
Other:
- board size 37.8 x 65.6 mm -> 76.5 x 65.6 mm
Changed lines of the file:
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@@
     )
+  )
+  (footprint "MountingHole:MountingHole_2.2mm_M2" (layer "F.Cu")
+    (at 128.7 116.3)
+    (descr "Mounting Hole 2.2mm, no annular, M2")
+    (tags "mounting hole 2.2mm no annular m2")
+    (property "DigiKey Part Number" "")
+    (property "Power Rating" "")
+    (property "Sheetfile" "sfh2430_breakout.kicad_sch")
+    (property "Sheetname" "")
+    (property "Tolerance" "")
+    (property "exclude_from_bom" "")
+    (property "ki_description" "Mounting Hole with connection")
+    (property "ki_keywords" "mounting hole")
+    (attr exclude_from_pos_files exclude_from_bom)
+    (fp_text reference "H1" (at 0 -3.2) (layer "F.SilkS")
+        (effects (font (size 1 1) (thickness 0.15)))
+    )
+    (fp_text value "MountingHole_Pad" (at 0 3.2) (layer "F.Fab")
+        (effects (font (size 1 1) (thickness 0.15)))
+    )
+    (fp_text user "${REFERENCE}" (at 0 0) (layer "F.Fab")
+        (effects (font (size 1 1) (thickness 0.15)))
+    )
+    (fp_circle (center 0 0) (end 2.2 0)
+      (stroke (width 0.15) (type solid)) (fill none) (layer "Cmts.User"))
+    (fp_circle (center 0 0) (end 2.45 0)
+      (stroke (width 0.05) (type solid)) (fill none) (layer "F.CrtYd"))
+    (pad "" np_thru_hole circle (at 0 0) (size 2.2 2.2) (drill 2.2) (layers "*.Cu" "*.Mask"))
   )
   (footprint "Capacitor_SMD:C_0603_1608Metric" (layer "F.Cu")
@@
       (rotate (xyz 0 0 0))
     )
+  )
+  (footprint "MountingHole:MountingHole_2.2mm_M2" (layer "F.Cu")
+    (at 118 127)
+    (descr "Mounting Hole 2.2mm, no annular, M2")
+    (tags "mounting hole 2.2mm no annular m2")
+    (property "DigiKey Part Number" "")
+    (property "Power Rating" "")
+    (property "Sheetfile" "sfh2430_breakout.kicad_sch")
+    (property "Sheetname" "")
+    (property "Tolerance" "")
+    (property "exclude_from_bom" "")
+    (property "ki_description" "Mounting Hole with connection")
+    (property "ki_keywords" "mounting hole")
+    (attr exclude_from_pos_files exclude_from_bom)
+    (fp_text reference "H4" (at 0 -3.2) (layer "F.SilkS")
+        (effects (font (size 1 1) (thickness 0.15)))
+    )
+    (fp_text value "MountingHole_Pad" (at 0 3.2) (layer "F.Fab")
+        (effects (font (size 1 1) (thickness 0.15)))
+    )
+    (fp_text user "${REFERENCE}" (at 0 0) (layer "F.Fab")
+        (effects (font (size 1 1) (thickness 0.15)))
+    )
+    (fp_circle (center 0 0) (end 2.2 0)
+      (stroke (width 0.15) (type solid)) (fill none) (layer "Cmts.User"))
+    (fp_circle (center 0 0) (end 2.45 0)
+      (stroke (width 0.05) (type solid)) (fill none) (layer "F.CrtYd"))
+    (pad "" np_thru_hole circle (at 0 0) (size 2.2 2.2) (drill 2.2) (layers "*.Cu" "*.Mask"))
   )
   (footprint "Capacitor_SMD:C_0603_1608Metric" (layer "F.Cu")
@@
     )
   )
+  (footprint "MountingHole:MountingHole_2.2mm_M2" (layer "F.Cu")
+    (at 129 137)
+    (descr "Mounting Hole 2.2mm, no annular, M2")
+    (tags "mounting hole 2.2mm no annular m2")
+    (property "DigiKey Part Number" "")
+    (property "Power Rating" "")
+    (property "Sheetfile" "sfh2430_breakout.kicad_sch")
+    (property "Sheetname" "")
+    (property "Tolerance" "")
+    (property "exclude_from_bom" "")
+    (property "ki_description" "Mounting Hole with connection")
+    (property "ki_keywords" "mounting hole")
+    (attr exclude_from_pos_files exclude_from_bom)
+    (fp_text reference "H3" (at 0 -3.2) (layer "F.SilkS")
+        (effects (font (size 1 1) (thickness 0.15)))
+    )
+    (fp_text value "MountingHole_Pad" (at 0 3.2) (layer "F.Fab")
+        (effects (font (size 1 1) (thickness 0.15)))
+    )
+    (fp_text user "${REFERENCE}" (at 0 0) (layer "F.Fab")
+        (effects (font (size 1 1) (thickness 0.15)))
+    )
+    (fp_circle (center 0 0) (end 2.2 0)
+      (stroke (width 0.15) (type solid)) (fill none) (layer "Cmts.User"))
+    (fp_circle (center 0 0) (end 2.45 0)
+      (stroke (width 0.05) (type solid)) (fill none) (layer "F.CrtYd"))
+    (pad "" np_thru_hole circle (at 0 0) (size 2.2 2.2) (drill 2.2) (layers "*.Cu" "*.Mask"))
+  )
   (footprint "Capacitor_SMD:C_0603_1608Metric" (layer "F.Cu")
     (at 79.257903 115.790805)
@@
       (rotate (xyz 0 0 0))
     )
+  )
+  (footprint "MountingHole:MountingHole_2.2mm_M2" (layer "F.Cu")
+    (at 139.3 127)
+    (descr "Mounting Hole 2.2mm, no annular, M2")
+    (tags "mounting hole 2.2mm no annular m2")
+    (property "DigiKey Part Number" "")
+    (property "Power Rating" "")
+    (property "Sheetfile" "sfh2430_breakout.kicad_sch")
+    (property "Sheetname" "")
+    (property "Tolerance" "")
+    (property "exclude_from_bom" "")
+    (property "ki_description" "Mounting Hole with connection")
+    (property "ki_keywords" "mounting hole")
+    (attr exclude_from_pos_files exclude_from_bom)
+    (fp_text reference "H2" (at 0 -3.2) (layer "F.SilkS")
+        (effects (font (size 1 1) (thickness 0.15)))
+    )
+    (fp_text value "MountingHole_Pad" (at 0 3.2) (layer "F.Fab")
+        (effects (font (size 1 1) (thickness 0.15)))
+    )
+    (fp_text user "${REFERENCE}" (at 0 0) (layer "F.Fab")
+        (effects (font (size 1 1) (thickness 0.15)))
+    )
+    (fp_circle (center 0 0) (end 2.2 0)
+      (stroke (width 0.15) (type solid)) (fill none) (layer "Cmts.User"))
+    (fp_circle (center 0 0) (end 2.45 0)
+      (stroke (width 0.05) (type solid)) (fill none) (layer "F.CrtYd"))
+    (pad "" np_thru_hole circle (at 0 0) (size 2.2 2.2) (drill 2.2) (layers "*.Cu" "*.Mask"))
   )
   (footprint "Capacitor_SMD:C_0603_1608Metric" (layer "F.Cu")
@@
   (gr_line (start 79.9 121.183541) (end 79.9 161.525)
     (stroke (width 0.1) (type default)) (layer "Edge.Cuts"))
+  (gr_rect (start 120.16 118.5) (end 137.16 135.5)
+    (stroke (width 0.2) (type default)) (fill none) (layer "Edge.Cuts"))
   (gr_line (start 76.3 98.8) (end 73.471573 95.971573)
     (stroke (width 0.1) (type default)) (layer "Edge.Cuts"))
@@
   (gr_line (start 70.119886 104.980114) (end 74.35 104.980114)
     (stroke (width 0.1) (type default)) (layer "Edge.Cuts"))
+  (gr_poly
+    (pts
+      (xy 70.8 113.8)
+      (xy 84.942136 99.657864)
+      (xy 99.084271 113.8)
+      (xy 84.942136 127.942136)
+    )
+    (stroke (width 0.1) (type default)) (fill none) (layer "Edge.Cuts"))
   (gr_line (start 76.782411 107.3) (end 74.35 104.980114)
     (stroke (width 0.1) (type default)) (layer "Edge.Cuts"))
@@
   (gr_line (start 75.298105 127.717208) (end 75.298105 124.648364)
     (stroke (width 0.1) (type default)) (layer "Edge.Cuts"))
+  (gr_poly
+    (pts
+      (xy 114.515047 127.004365)
+      (xy 128.657183 112.862229)
+      (xy 142.799318 127.004365)
+      (xy 128.657183 141.146501)
+    )
+    (stroke (width 0.1) (type default)) (fill none) (layer "Edge.Cuts"))
   (gr_line (start 96.264823 104.885177) (end 99.333667 104.885177)
     (stroke (width 0.1) (type default)) (layer "Edge.Cuts"))
