File: cpu_board/cpu_board.kicad_pcb (KiCad board)
At the start: 6 copper layers, 60 x 60 mm, 198 parts, among them J1 USB_C_pycubed, J2 353620650, J3 JTAG_SWD_10, J4 353620650, J5 353620650, J6 DF40C-100DP-0.4V(51), J7 DF40C-100DP-0.4V(51), Q1 IRLML2803, Q2 NDS8434, SW1 SWITCH_SMT4.6X2.8, SW2 SW_DIP_x10, SW3 SW_DIP_x04, U1 TPS7A4501DCQT, U2 MIMXRT1176, U3 EM064LXQADG13IS1T, U4 MT29F1G01ABBFDWB, U5 USBLC6-2SC6, U6 MT48H32M16LFB4-6, U7 TPS54226PWPRPWP14_2P31X2P46-L, U8 TPS54226PWPRPWP14_2P31X2P46-L, Y2 24.0mHz, Y3 32.768kHz

Commit message: floorplan complete
Parts:
- removed C11: 4.7uF, Capacitor_SMD:C_0402_1005Metric
- removed C16: 0.22uF, Capacitor_SMD:C_0402_1005Metric
- removed C24, C28, C30, C37, C39, C7: 0.1uF, Capacitor_SMD:C_0402_1005Metric
- removed C27, C29: 2.2uF, Capacitor_SMD:C_0402_1005Metric
- removed C32, C33: 10uF, Capacitor_SMD:C_0402_1005Metric
- removed C35, C36: 22uF, Capacitor_SMD:C_0402_1005Metric
- removed C55: 10pF, Capacitor_SMD:C_0402_1005Metric
- removed C57: 1uF, Capacitor_SMD:C_0402_1005Metric
- removed L1: 4.7uH, adcs:IND-SMD_L5.8-W5.2_PIO54
- removed R11, R12, R13, R14, R15, R6: 0Ω, Resistor_SMD:R_0402_1005Metric
- removed R4, R9: DNP, Resistor_SMD:R_0402_1005Metric
- removed R5: 4.7kΩ, Resistor_SMD:R_0402_1005Metric
- removed TP3, TP4, TP5, TP6, TP7: TestPoint, TestPoint:TestPoint_Pad_1.0x1.0mm
- C10, C12, C13, C14, C15, C17, C22, C23, C25, C26, C3, C34, C38, C4, C40, C41, C42, C43, C44, C45, C46, C47, C48, C49, C50, C51, C52, C53, C54, C56, C58, C59, C6, C60, C61, C67, C68, C69, C70, C71, C72, C73, C74, C75, C8, C9, R10, R24, R26, R8, TP1, TP2: moved to B.Cu
- C5: value 22uF -> 10pF; moved to B.Cu
- FB1, FB2, FB3, FB4, FB5: footprint adcs:L0402_H0.55MM -> Inductor_SMD:L_0402_1005Metric; moved to B.Cu
- FB6: footprint adcs:L0402_H0.55MM -> Inductor_SMD:L_0402_1005Metric
- J5: value 353620650 -> Conn_01x06; footprint mainboard:MOLEX_35362-0650 -> Connector_PinHeader_2.54mm:PinHeader_1x06_P2.54mm_Vertical
- R3: value 30kΩ -> 10kΩ; moved to B.Cu
- R31: moved to F.Cu
- moved C31 131.1 mm to (55.4, 51.5)
- moved R7 128.1 mm to (55.5, 50.3)
- moved C3 125.4 mm to (50.0, 42.3), turned to 90 degrees
- moved C10 119.6 mm to (46.1, 34.7), turned to 180 degrees
- moved C14 119.4 mm to (51.5, 40.4), turned to 90 degrees
- moved C38 118.7 mm to (52.3, 36.5), turned to -90 degrees
- moved C12 117.6 mm to (47.5, 36.0), turned to -90 degrees
- moved C23 117.2 mm to (49.0, 40.0), turned to -90 degrees
- moved C8 116.8 mm to (51.5, 42.2), turned to -90 degrees
- moved C45 116.7 mm to (45.9, 39.7), turned to -90 degrees
- moved R8 116.4 mm to (47.5, 42.2), turned to -90 degrees
- moved C44 115.9 mm to (51.0, 37.3)
- moved C25 115.6 mm to (49.0, 42.3), turned to -90 degrees
- moved C15 115.5 mm to (50.0, 38.7), turned to 90 degrees
- moved C13 115.5 mm to (48.9, 35.2)
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Connections:
- net /USB-C/USB_DN_CON renamed /USB-C/USB_CON_DN
- net /USB-C/USB_DP_CON renamed /USB-C/USB_CON_DP
- net Net-(U2B-VDDA_ADC_3P3) renamed /RT1176 #1/VDDA_ADC_3P3
- net Net-(U2E-CLK1_N) renamed /RT1176 #1/CLK1_N
- net Net-(U2E-CLK1_P) renamed /RT1176 #1/CLK1_P
- net Net-(U2L-VDD_USB_1P8) renamed /RT1176 #3/VDD_USB_1P8
- net Net-(U2L-VDD_USB_3P3) renamed /RT1176 #3/VDD_USB_3P3
- C10 pad 1: Net-(U2B-VDD_SOC_IN_1) -> VDD_SOC_IN
- C12 pad 1: Net-(U2B-VDD_SOC_IN_1) -> VDD_SOC_IN
- C13 pad 1: Net-(U2B-VDD_SOC_IN_1) -> VDD_SOC_IN
- C17 pad 1: Net-(U2B-VDD_SOC_IN_1) -> VDD_SOC_IN
- C22 pad 1: Net-(U2B-VDD_SOC_IN_1) -> VDD_SOC_IN
- C34 pad 1: ADC_1V8_IN -> Net-(U2B-VDDA_1P8_IN)
- C4 pad 1: Net-(U2B-VDD_SOC_IN_1) -> VDD_SOC_IN
- C47 pad 1: Net-(U2I-NVCC_DISP1) -> VDD_1V8
- C48 pad 1: Net-(U2I-NVCC_DISP2) -> VDD_3V3
- C49 pad 1: Net-(U2G-NVCC_SD1) -> VDD_1V8
- C5 pad 1: VDD_3V3 -> /RT1176 #3/SEMC_DQS
- C50 pad 1: Net-(U2G-NVCC_SD2) -> VDD_1V8
- C6 pad 1: Net-(U2B-VDD_SOC_IN_1) -> VDD_SOC_IN
- C60 pad 1: /RT1176 #3/VUSB -> VUSB
- FB2 pad 1: DCDC_1V8_OUT -> VDD_1V8
- J4 pad 1: /Interface/POR_B -> POR_B
- J5 pad 6: /Interface/VUSB -> VUSB
- R3 pad 1: VDD_3V3 -> GND
- R3 pad 2: Net-(U2C-DCDC_PSWITCH) -> /RT1176 #3/VDD_MIPI_1P0
- U2 pad D12: Net-(U2I-NVCC_DISP1) -> VDD_1V8
- U2 pad D14: Net-(U2G-NVCC_SD1) -> VDD_1V8
- U2 pad D17: /RT1176 #3/VUSB -> VUSB
- U2 pad E7: Net-(U2I-NVCC_DISP2) -> VDD_3V3
- U2 pad F10: Net-(U2K-VDD_MIPI_1P0) -> /RT1176 #3/VDD_MIPI_1P0
- U2 pad G13: Net-(U2G-NVCC_SD2) -> VDD_1V8
- U2 pad H10: Net-(U2B-VDD_SOC_IN_1) -> VDD_SOC_IN
- U2 pad H8: Net-(U2B-VDD_SOC_IN_1) -> VDD_SOC_IN
- U2 pad H9: Net-(U2B-VDD_SOC_IN_1) -> VDD_SOC_IN
- U2 pad J10: Net-(U2B-VDD_SOC_IN_1) -> VDD_SOC_IN
- U2 pad J2: GPIO_EMC_B1_40 -> /RT1176 #3/SEMC_DQS
- U2 pad J8: Net-(U2B-VDD_SOC_IN_1) -> VDD_SOC_IN
- U2 pad J9: Net-(U2B-VDD_SOC_IN_1) -> VDD_SOC_IN
- U2 pad K10: Net-(U2B-VDD_SOC_IN_1) -> VDD_SOC_IN
- U2 pad K8: VDD_SOC_IN -> unconnected-(U2C-DCDC_DIG_1-PadK8)
- U2 pad K9: VDD_SOC_IN -> unconnected-(U2C-DCDC_DIG_2-PadK9)
- U2 pad L5: VDD_3V3 -> unconnected-(U2C-DCDC_IN_Q-PadL5)
- U2 pad L7: VDD_SOC_IN -> unconnected-(U2C-DCDC_DIG_SENSE-PadL7)
- U2 pad L8: VDD_SOC_IN -> unconnected-(U2C-DCDC_DIG_3-PadL8)
- U2 pad M11: ADC_1V8_IN -> Net-(U2B-VDDA_1P8_IN)
- U2 pad M5: VDD_3V3 -> unconnected-(U2C-DCDC_IN_1-PadM5)
- U2 pad M6: DCDC_1V8_OUT -> unconnected-(U2C-DCDC_ANA_SENSE-PadM6)
- U2 pad M7: DCDC_1V8_OUT -> unconnected-(U2C-DCDC_ANA_1-PadM7)
- U2 pad M8: DCDC_1V8_OUT -> unconnected-(U2C-DCDC_ANA_2-PadM8)
- U2 pad N4: Net-(U2C-DCDC_MODE) -> GND
- U2 pad N5: VDD_3V3 -> unconnected-(U2C-DCDC_IN_2-PadN5)
- U2 pad P3: Net-(U2C-DCDC_PSWITCH) -> GND
- U2 pad T11: Net-(U2A-TEST_MODE) -> GND
- U2 pad T3: Net-(U2C-DCDC_LP_1) -> unconnected-(U2C-DCDC_LP_1-PadT3)
- U2 pad T4: Net-(U2C-DCDC_LN_1) -> unconnected-(U2C-DCDC_LN_1-PadT4)
- U2 pad U3: Net-(U2C-DCDC_LP_1) -> unconnected-(U2C-DCDC_LP_2-PadU3)
- U2 pad U4: Net-(U2C-DCDC_LN_1) -> unconnected-(U2C-DCDC_LN_2-PadU4)
Routing:
- net /Interface/EN_RT1176: track 1.01 -> 89.1 mm, vias 0 -> 2
- net GND: track 15.6 -> 71.7 mm, vias 13 -> 63
- net VUSB: track 2.78 -> 24.0 mm, vias 2 -> 4
- net /SDRAM/SDRAM_1V8: track 2.77 -> 22.8 mm, vias 6 -> 15
- net SEMC_A10: track 1.60 -> 20.9 mm
- net VDD_SNVS_ANA: track 0.00 -> 18.9 mm, vias 0 -> 4
- net POR_B: track 0.00 -> 17.1 mm
- net VDD_3V3: track 6.62 -> 23.4 mm, vias 20 -> 17
- net SEMC_A2: track 37.0 -> 20.3 mm
- net VDD_SNVS_3V3: track 0.00 -> 16.4 mm, vias 0 -> 2
- net OTG1_D_N: track 0.00 -> 15.1 mm
- net OTG1_D_P: track 0.00 -> 14.9 mm
- net VDD_SOC_IN: track 0.00 -> 14.1 mm, vias 0 -> 8
- net VSYS: track 18.6 -> 30.6 mm, vias 18 -> 17
- net SWD_RESET: track 0.00 -> 11.6 mm
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- added copper zone on In3.Cu, net /SDRAM/SDRAM_1V8
- added copper zone on B.Cu, net GNDREF
- added copper zone on In3.Cu, net VBATT_IN
- added copper zone on In3.Cu, net VUSB
- removed copper zone on In3.Cu, net GND

Commit message: add models and power diagram
Parts:
- U2: footprint adcs:BGA289C80P17X17_1400X14000X152 -> adcs:U_MIMXRT1176DVMAA_NXP
- U6: footprint adcs:BGA54C80P6X9_800X800X100 -> adcs:VFBGA54_8X8_MRN
- moved C40 0.23 mm to (52.9, 33.9)
Routing:
- net FlexSPI_A_D2: track 0.00 -> 25.0 mm, vias 0 -> 3
- net FlexSPI_A_SS1: track 0.00 -> 23.1 mm, vias 0 -> 4
- net FlexSPI_A_D1: track 0.00 -> 21.3 mm, vias 0 -> 2
- net FlexSPI_A_SS0: track 0.00 -> 14.9 mm, vias 0 -> 2
- net FlexSPI_A_CLK: track 0.00 -> 14.8 mm, vias 0 -> 3
- net FlexSPI_A_D0: track 0.00 -> 14.4 mm, vias 0 -> 4
- net FlexSPI_A_D3: track 0.00 -> 14.4 mm, vias 0 -> 3
- net VDD_1V8: track 41.6 -> 44.7 mm, vias 21 -> 22
- net GND: track 71.7 -> 69.3 mm, vias 63 -> 56
- net /SDRAM/SDRAM_1V8: track 22.8 -> 23.8 mm, vias 15 -> 17
- net SEMC_BA0: track 19.5 -> 20.0 mm, vias 2 -> 3
- net SEMC_A6: track 20.9 -> 21.4 mm, vias 0 -> 1
- net SEMC_CKE: track 23.4 -> 23.8 mm, vias 2 -> 3
- net SEMC_A3: vias 2 -> 3
- net /RT1176 #1/VDDA_ADC_3P3: vias 1 -> 2

Commit message: continue work on fanout
Parts:
- removed D1: CDBQR00340-HF, adcs:D0402_H0.55MM
- removed FB4, FB5: 190mΩ, Inductor_SMD:L_0402_1005Metric
- removed R1: 6.9k, Resistor_SMD:R_0402_1005Metric
- removed R2: 4k, Resistor_SMD:R_0402_1005Metric
- removed U1: TPS7A4501DCQT, mainboard:TPS7A4501DCQT
- added R5: 2.2MΩ, adcs:Perfect_0402, F.Cu at (97.5, 50.6)
- added R6: 1.27MΩ, adcs:Perfect_0402, F.Cu at (97.5, 52.6)
- added U9: LT3014IS5-TRMPBF, adcs:S_5_ADI, F.Cu at (91.9, 51.9)
- C1, C10, C12, C13, C14, C15, C17, C2, C22, C23, C25, C26, C3, C31, C34, C38, C40, C41, C42, C43, C44, C45, C46, C47, C48, C49, C5, C50, C51, C52, C53, C54, C56, C58, C59, C6, C61, C69, C70, C71, C72, C73, C74, C75, C8, C9, C90: footprint Capacitor_SMD:C_0402_1005Metric -> adcs:Perfect_0201
- C18, C19, C20, C21, C4, C60, C62, C63, C66, C67, C68, C76, C77, C78, C80, C84, C85, C86, C87, C88, C89, C91: footprint Capacitor_SMD:C_0402_1005Metric -> adcs:Perfect_0402
- C79, C81, C82, C83: footprint Capacitor_SMD:C_1210_3225Metric -> adcs:Perfect_0402
- FB1, FB2, FB3, FB6: footprint Inductor_SMD:L_0402_1005Metric -> adcs:Perfect_0402
- R10, R16, R17, R18, R20, R22, R23, R24, R25, R26, R27, R28, R29, R30, R31, R32, R33, R34, R35, R36, R37, R38, R39, R40, R41, R42, R43, R44, R45, R46, R47, R48, R49, R50, R51, R52, R53, R54, R55, R56, R57, R58, R59, R60, R61, R62, R63, R64, R7, R8: footprint Resistor_SMD:R_0402_1005Metric -> adcs:Perfect_0402
- R3: footprint Resistor_SMD:R_0402_1005Metric -> adcs:Perfect_0201
- moved C2 76.3 mm to (13.9, -6.90), turned to 0 degrees
- moved FB3 7.71 mm to (55.3, 32.6), turned to 180 degrees
- moved R3 7.39 mm to (48.3, 33.3), turned to 90 degrees
- moved C50 3.74 mm to (50.7, 33.3), turned to 90 degrees
- moved C58 3.05 mm to (49.5, 34.5), turned to 180 degrees
- moved C56 2.35 mm to (47.5, 33.1), turned to -90 degrees
- moved TP1 1.87 mm to (57.0, 42.7)
- moved TP2 1.87 mm to (57.0, 40.7)
- moved C59 1.68 mm to (49.9, 33.3)
- moved C52 1.51 mm to (45.1, 35.8)
- moved C42 1.33 mm to (50.5, 35.5), turned to -135 degrees
- moved C15 0.88 mm to (49.6, 39.5), turned to -135 degrees
- moved C61 0.81 mm to (53.1, 31.6), turned to -90 degrees
- moved R24 0.80 mm to (39.9, 39.2)
- moved C54 0.78 mm to (45.5, 34.9), turned to 0 degrees
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Connections:
- C2 pad 2: Net-(D1-A) -> VDD_SNVS_3V3
- C58 pad 1: /RT1176 #3/VDD_USB_1P8 -> VDD_1V8
- C59 pad 1: /RT1176 #3/VDD_USB_3P3 -> VDD_3V3
- U2 pad A11: MIPI_CSI_D0_N -> unconnected-(U2K-MIPI_CSI_DN0-PadA11)
- U2 pad A12: MIPI_CSI_CK_N -> unconnected-(U2K-MIPI_CSI_CKN-PadA12)
- U2 pad A13: MIPI_CSI_D1_N -> unconnected-(U2K-MIPI_CSI_DN1-PadA13)
- U2 pad B11: MIPI_CSI_D0_P -> unconnected-(U2K-MIPI_CSI_DP0-PadB11)
- U2 pad B12: MIPI_CSI_CK_P -> unconnected-(U2K-MIPI_CSI_CKP-PadB12)
- U2 pad B13: MIPI_CSI_D1_P -> unconnected-(U2K-MIPI_CSI_DP1-PadB13)
- U2 pad C16: USB2_TPU_N -> unconnected-(U2L-USB2_DN-PadC16)
- U2 pad C17: USB2_TPU_P -> unconnected-(U2L-USB2_DP-PadC17)
- U2 pad G12: /RT1176 #3/VDD_USB_3P3 -> VDD_3V3
- U2 pad H12: /RT1176 #3/VDD_USB_1P8 -> VDD_1V8
- U7 pad 7: VSYS -> PMIC_ON_REQ
- U8 pad 7: VSYS -> PMIC_ON_REQ
Routing:
- net ENET_RGMII_TXD1_BT: track 0.00 -> 37.9 mm, vias 0 -> 2
- net ENET_RGMII_TXD3_BT: track 0.00 -> 36.4 mm, vias 0 -> 2
- net ENET_RGMII_TXD2_BT: track 0.00 -> 36.2 mm, vias 0 -> 2
- net ENET_RGMII_TXD0_BT: track 0.00 -> 32.1 mm, vias 0 -> 2
- net ENET_RGMII_TX_EN_BT: track 0.00 -> 29.6 mm, vias 0 -> 2
- net GPIO_AD_16: track 0.00 -> 29.3 mm, vias 0 -> 1
- net ENET_RGMII_TXC_BT: track 0.00 -> 29.2 mm, vias 0 -> 2
- net GPIO_DISP_B2_01: track 0.00 -> 27.3 mm, vias 0 -> 2
- net GPIO_AD_12: track 0.00 -> 27.1 mm, vias 0 -> 1
- net GPIO_AD_29: track 0.00 -> 26.5 mm, vias 0 -> 1
- net GPIO_DISP_B2_00: track 0.00 -> 25.7 mm, vias 0 -> 2
- net GPIO_DISP_B2_02: track 0.00 -> 25.3 mm, vias 0 -> 2
- net GPIO_AD_10: track 0.00 -> 25.0 mm, vias 0 -> 1
- net GPIO_AD_31: track 0.00 -> 23.9 mm, vias 0 -> 1
- net GPIO_AD_07: track 0.00 -> 23.1 mm, vias 0 -> 1
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- added copper zone on In3.Cu, net GND
- removed copper zone on In1.Cu, net GND
- removed copper zone on In2.Cu, net GND
- removed copper zone on In4.Cu, net GND
