File: cpu_board/rt1176_2.kicad_sch (KiCad schematic)
At the start: 9 parts, among them U2 MIMXRT1176

Commit message: clean up silkscreen
Parts:
- C? (x7): Footprint (for JLCPCB) 0402 -> 0201
Changed lines of the file:
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@@
       (effects (font (size 1.27 1.27)) hide)
     )
-    (property "Datasheet" "~" (at 217.805 79.375 0)
+    (property "Datasheet" "" (at 217.805 79.375 0)
       (effects (font (size 1.27 1.27)) hide)
     )
@@
       (effects (font (size 1.27 1.27)) hide)
     )
-    (property "Footprint (for JLCPCB)" "0402" (at 217.805 79.375 0)
+    (property "Footprint (for JLCPCB)" "0201" (at 217.805 79.375 0)
       (effects (font (size 1.27 1.27)) hide)
     )
@@
       (effects (font (size 1.27 1.27)) hide)
     )
-    (property "Datasheet" "~" (at 217.805 104.775 0)
+    (property "Datasheet" "" (at 217.805 104.775 0)
       (effects (font (size 1.27 1.27)) hide)
     )
@@
       (effects (font (size 1.27 1.27)) hide)
     )
-    (property "Footprint (for JLCPCB)" "0402" (at 217.805 104.775 0)
+    (property "Footprint (for JLCPCB)" "0201" (at 217.805 104.775 0)
       (effects (font (size 1.27 1.27)) hide)
     )
@@
       (effects (font (size 1.27 1.27)) hide)
     )
-    (property "Footprint (for JLCPCB)" "0402" (at 62.23 170.815 0)
+    (property "Footprint (for JLCPCB)" "0201" (at 62.23 170.815 0)
       (effects (font (size 1.27 1.27)) hide)
     )
@@
       (effects (font (size 1.27 1.27)) hide)
     )
-    (property "Datasheet" "~" (at 69.215 90.805 0)
+    (property "Datasheet" "" (at 69.215 90.805 0)
       (effects (font (size 1.27 1.27)) hide)
     )
@@
       (effects (font (size 1.27 1.27)) hide)
     )
-    (property "Footprint (for JLCPCB)" "0402" (at 69.215 90.805 0)
+    (property "Footprint (for JLCPCB)" "0201" (at 69.215 90.805 0)
       (effects (font (size 1.27 1.27)) hide)
     )
@@
       (effects (font (size 1.27 1.27)) hide)
     )
-    (property "Datasheet" "~" (at 72.39 170.815 0)
+    (property "Datasheet" "" (at 72.39 170.815 0)
       (effects (font (size 1.27 1.27)) hide)
     )
@@
       (effects (font (size 1.27 1.27)) hide)
     )
-    (property "Footprint (for JLCPCB)" "0402" (at 72.39 170.815 0)
+    (property "Footprint (for JLCPCB)" "0201" (at 72.39 170.815 0)
       (effects (font (size 1.27 1.27)) hide)
     )
@@
       (effects (font (size 1.27 1.27)) hide)
     )
-    (property "Datasheet" "~" (at 215.265 172.72 0)
+    (property "Datasheet" "" (at 215.265 172.72 0)
       (effects (font (size 1.27 1.27)) hide)
     )
@@
       (effects (font (size 1.27 1.27)) hide)
     )
-    (property "Footprint (for JLCPCB)" "0402" (at 215.265 172.72 0)
+    (property "Footprint (for JLCPCB)" "0201" (at 215.265 172.72 0)
       (effects (font (size 1.27 1.27)) hide)
     )
@@
       (effects (font (size 1.27 1.27)) hide)
     )
-    (property "Datasheet" "~" (at 215.265 205.74 0)
+    (property "Datasheet" "" (at 215.265 205.74 0)
       (effects (font (size 1.27 1.27)) hide)
     )
@@
       (effects (font (size 1.27 1.27)) hide)
     )
-    (property "Footprint (for JLCPCB)" "0402" (at 215.265 205.74 0)
-      (effects (font (size 1.27 1.27)) hide)
-    )
+    (property "Footprint (for JLCPCB)" "0201" (at 215.265 205.74 0)
+      (effects (font (size 1.27 1.27)) hide)
+    )

Commit message: soldermander 1.0 ready for review
Parts:
- C? (x6): Voltage Rating (none) -> 10V
- C?: Voltage Rating (none) -> 6.3V
Changed lines of the file:
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@@
+      (effects (font (size 1.27 1.27)) hide)
+    )
+    (property "Voltage Rating" "10V" (at 217.805 79.375 0)
       (effects (font (size 1.27 1.27)) hide)
     )
@@
       (effects (font (size 1.27 1.27)) hide)
     )
+    (property "Voltage Rating" "10V" (at 217.805 104.775 0)
+      (effects (font (size 1.27 1.27)) hide)
+    )
     (pin "1")
     (pin "2")
@@
     (property "Power Rating" "" (at 62.23 170.815 0)
       (effects (font (size 1.27 1.27)))
+    )
+    (property "Voltage Rating" "6.3V" (at 62.23 170.815 0)
+      (effects (font (size 1.27 1.27)) hide)
     )
     (pin "1")
@@
       (effects (font (size 1.27 1.27)) hide)
     )
+    (property "Voltage Rating" "10V" (at 69.215 90.805 0)
+      (effects (font (size 1.27 1.27)) hide)
+    )
     (pin "1")
     (pin "2")
@@
       (effects (font (size 1.27 1.27)) hide)
     )
+    (property "Voltage Rating" "10V" (at 72.39 170.815 0)
+      (effects (font (size 1.27 1.27)) hide)
+    )
     (pin "1")
     (pin "2")
@@
       (effects (font (size 1.27 1.27)) hide)
     )
+    (property "Voltage Rating" "10V" (at 215.265 172.72 0)
+      (effects (font (size 1.27 1.27)) hide)
+    )
     (pin "1")
     (pin "2")
@@
       (effects (font (size 1.27 1.27)) hide)
     )
+    (property "Voltage Rating" "10V" (at 215.265 205.74 0)
+      (effects (font (size 1.27 1.27)) hide)
+    )
