File: cpu_board/cpu_board.kicad_sch (KiCad schematic)
At the start: 0 parts

Commit message: soldermander 1.0 ready for review
Other:
- note added: "TODOs - [x] Add VSYS connector - [ ] Might need to pick a new height - [ ] Route USB differentially and impedance match to 90ohms - [ ] Does this really matter? - [ ] Add 3D models of parts - [ ] Breakout board - [x] Spec passives - [ ] Clean up planes - [ ] beautify schematic - [x] decide on 0402 vs. 0603 for caps/resistors -- [x] 0402, some 0201, and a couple larger ones -- [x] make the RT1176 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"
- note removed: "TODOs - [ ] Spec passives - [x] decide on 0402 vs. 0603 for caps/resistors -- 0402, some 0201, and a couple larger ones - [ ] beautify schematic - - [x] make the RT1176 boxes wider - [x] Switch fixed regs to variable - [x] Make sure most components are on JLCPCB - [x] Double check GPIOs and GPIO voltages - [x] Fix the $source_resistor - [x] Double check D1/D2 - [x] add boot config switches - [x] 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"
Changed lines of the file:
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@@
     (effects (font (size 2.54 2.54) (color 132 0 0 1)) (justify left bottom))
   )
-  (text "TODOs\n- [ ] Spec passives\n- [x] decide on 0402 vs. 0603 for caps/resistors\n-- 0402, some 0201, and a couple larger ones\n- [ ] beautify schematic\n- - [x] make the RT1176 boxes wider\n- [x] Switch fixed regs to variable\n- [x] Make sure most components are on JLCPCB\n- [x] Double check GPIOs and GPIO voltages\n- [x] Fix the $source_resistor\n- [x] Double check D1/D2\n- [x] add boot config switches\n- [x] add boot circuitry\n- [x] double check xSPI MRAM\n- [x] clean up label sizing\n- [x] Finish putting caps on\n- [x] Route MRAM & Flash\n    - [x] Clean up MRAM and flash\n- [x] Route \n- [x] Try patching up ground\n- [x] Pick hole locations\n- [x] Add VSYS connector\n    - [ ] Might need to pick a new height\n- [x] Pick a UART for inter-board communications\n- [ ] Add JLC P/Ns\n- [ ] Double check passive specifications\n- [x] Double check paste layer (or just replace footprints)\n- [x] Put part outlines for things I copied from the coral\n- [ ] Clean up planes\n- [x] Route GPIO breakouts\n- [ ] Route USB differentially and impedance match to 90ohms\n    - [ ] Does this really matter?\n- [x] Tune SDRAM trace lengths (within 10mm)\n- [x] Tune Crystal trace lengths (within 0.02mm)\n- [x] Add power pins (Low priority)\n- [x] Clean up silkscreen\n- [ ] Add 3D models of parts\n- [ ] Breakout board"
-    (at 306.07 162.56 0)
+  (text "TODOs\n- [x] Add VSYS connector\n    - [ ] Might need to pick a new height\n- [ ] Route USB differentially and impedance match to 90ohms\n    - [ ] Does this really matter?\n- [ ] Add 3D models of parts\n- [ ] Breakout board\n- [x] Spec passives\n- [ ] Clean up planes\n- [ ] beautify schematic\n- [x] decide on 0402 vs. 0603 for caps/resistors\n-- [x] 0402, some 0201, and a couple larger ones\n-- [x] make the RT1176 boxes wider\n- [x] Switch fixed regs to variable\n- [x] Make sure most components are on JLCPCB\n- [x] Double check GPIOs and GPIO voltages\n- [x] Fix the $source_resistor\n- [x] Double check D1/D2\n- [x] add boot config switches\n- [x] add boot circuitry\n- [x] double check xSPI MRAM\n- [x] clean up label sizing\n- [x] Finish putting caps on\n- [x] Route MRAM & Flash\n    - [x] Clean up MRAM and flash\n- [x] Route \n- [x] Try patching up ground\n- [x] Pick hole locations\n- [x] Pick a UART for inter-board communications\n- [x] Add JLC P/Ns\n- [x] Double check passive specifications\n- [x] Double check paste layer (or just replace footprints)\n- [x] Put part outlines for things I copied from the coral\n- [x] Route GPIO breakouts\n- [x] Tune SDRAM trace lengths (within 10mm)\n- [x] Tune Crystal trace lengths (within 0.02mm)\n- [x] Add power pins (Low priority)\n- [x] Clean up silkscreen\n"
+    (at 306.705 168.275 0)
     (effects (font (size 2.54 2.54)) (justify left bottom))
   )

Commit message: update
Other:
- company: (none) -> Stanford Student Space Initiative
- title: (none) -> Soldermander
Changed lines of the file:
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@@
 (kicad_sch (version 20230121) (generator eeschema)
   (paper "A4")
+  (title_block
+    (title "Soldermander")
+    (date "2024-02-27")
+    (rev "1.0")
+    (company "Stanford Student Space Initiative")
+    (comment 1 "RE: Flynn Dreilinger")
+  )
   (text "Changes from Coral Schematic:\n- removed PMIC, added individual switching regs (TPS54) and LDOs (TPS7A)\n- added MRAM on FlexSPI A CS1 to test booting from it.\n- 24mhz crystal -> TCXO\n- changed NAND flash to be 2GB instead of 1GB (since that is what is available on JLCPCB)\n- changed USB-C component to use same P/N as PyCubed\n- changed some of the GPIO banks from 1.8V to 3.3V\n- added a few connectors for RBF + interface with a PyCubed\n-- removed USB-C controller (since we do not need OTG functionality)\n- changed most unused pin names to generic RT1176 names\n-- left: SD Card, Camera, TPU, ethernet (in order of likelihood that we add these things)"
     (at 93.98 60.96 0)
