File: PCBranch/PCBranch.kicad_pcb (KiCad board)
At the start: 4 copper layers, 90.2 x 95.9 mm, 15 parts, among them J1 CLP-105-02-X-D, J2 DF40HC_3.0_-100DS-0.4V_51_, J3 DF40HC_3.0_-100DS-0.4V_51_, J4 Conn_02x25_Odd_Even, J5 Conn_02x25_Odd_Even, J6 Conn_02x25_Odd_Even, J7 Conn_02x25_Odd_Even

Commit message: PCBranch ready for review
Parts:
- moved J6 93.7 mm to (81.1, 78.9), turned to 0 degrees
- moved J4 73.6 mm to (9.18, 17.8)
- moved J7 60.5 mm to (15.0, 84.0), turned to -90 degrees
- moved J5 0.31 mm to (75.7, 13.4)
Connections:
- J2 pad 10: WAKEUP -> GND
- J2 pad 12: PMIC_ON_REQ -> ONOFF
- J2 pad 14: DAC_OUT -> PMIC_STBY_REQ
- J2 pad 16: EN_ADCS -> WAKEUP
- J2 pad 18: GND -> PMIC_ON_REQ
- J2 pad 20: GPIO_SD_B1_00 -> DAC_OUT
- J2 pad 22: GPIO_SD_B1_01 -> EN_ADCS
- J2 pad 24: GPIO_SD_B1_03 -> GND
- J2 pad 26: GPIO_SD_B1_04 -> GPIO_SD_B1_00
- J2 pad 28: GPIO_SD_B1_05 -> GPIO_SD_B1_01
- J2 pad 30: GND -> GPIO_SD_B1_03
- J2 pad 32: USDHC2_DATA3 -> GPIO_SD_B1_04
- J2 pad 34: USDHC2_DATA2 -> GPIO_SD_B1_05
- J2 pad 36: USDHC2_DATA1 -> GND
- J2 pad 38: USDHC2_DATA0 -> USDHC2_DATA3
- J2 pad 4: GND -> VDD_3V3
- J2 pad 40: USDHC2_CLK -> USDHC2_DATA2
- J2 pad 42: USDHC2_CMD -> USDHC2_DATA1
- J2 pad 44: GND -> USDHC2_DATA0
- J2 pad 46: GPIO_EMC_B1_40 -> USDHC2_CLK
- J2 pad 48: GPIO_EMC_B1_41 -> USDHC2_CMD
- J2 pad 50: unconnected-(J2-Pad50) -> GND
- J2 pad 52: GND -> GPIO_EMC_B1_40
- J2 pad 54: VDD_3V3_LP -> GPIO_EMC_B1_41
- J2 pad 56: VDD_3V3_LP -> unconnected-(J2-Pad56)
- J2 pad 58: VDD_3V3_LP -> GND
- J2 pad 6: ONOFF -> VDD_3V3
- J2 pad 62: GND -> VDD_3V3_LP
- J2 pad 64: unconnected-(J2-Pad64) -> VDD_3V3_LP
- J2 pad 66: unconnected-(J2-Pad66) -> VDD_3V3_LP
- J2 pad 68: unconnected-(J2-Pad68) -> GND
- J2 pad 72: GND -> unconnected-(J2-Pad72)
- J2 pad 78: unconnected-(J2-Pad78) -> GND
- J2 pad 8: PMIC_STBY_REQ -> VDD_3V3
- J2 pad 82: GND -> unconnected-(J2-Pad82)
- J2 pad 84: GPIO_AD_31 -> unconnected-(J2-Pad84)
- J2 pad 86: GPIO_AD_32 -> unconnected-(J2-Pad86)
- J2 pad 88: GPIO_AD_33 -> GND
- J2 pad 90: GPIO_AD_34 -> GPIO_AD_31
- J2 pad 92: GPIO_AD_35 -> GPIO_AD_32
- J2 pad 94: GND -> GPIO_AD_33
- J2 pad 96: unconnected-(J2-Pad96) -> GPIO_AD_34
- J2 pad 98: GND -> GPIO_AD_35
- J4 pad 1: unconnected-(J4-Pin_1-Pad1) -> GND
- J4 pad 10: unconnected-(J4-Pin_10-Pad10) -> VSYS
- J4 pad 11: unconnected-(J4-Pin_11-Pad11) -> GND
- J4 pad 12: unconnected-(J4-Pin_12-Pad12) -> VSYS
- J4 pad 13: unconnected-(J4-Pin_13-Pad13) -> GPIO_AD_14
- J4 pad 14: unconnected-(J4-Pin_14-Pad14) -> GND
- J4 pad 15: unconnected-(J4-Pin_15-Pad15) -> GPIO_AD_15
- J4 pad 16: unconnected-(J4-Pin_16-Pad16) -> VSYS
- J4 pad 17: unconnected-(J4-Pin_17-Pad17) -> GPIO_AD_16
- J4 pad 18: unconnected-(J4-Pin_18-Pad18) -> VSYS
- J4 pad 19: unconnected-(J4-Pin_19-Pad19) -> GPIO_AD_17
- J4 pad 2: unconnected-(J4-Pin_2-Pad2) -> GND
- J4 pad 20: unconnected-(J4-Pin_20-Pad20) -> VSYS
- J4 pad 21: unconnected-(J4-Pin_21-Pad21) -> GND
- J4 pad 22: unconnected-(J4-Pin_22-Pad22) -> VSYS
- J4 pad 23: unconnected-(J4-Pin_23-Pad23) -> GPIO_AD_18
- J4 pad 24: unconnected-(J4-Pin_24-Pad24) -> VSYS
- J4 pad 25: unconnected-(J4-Pin_25-Pad25) -> GPIO_AD_19
- J4 pad 26: unconnected-(J4-Pin_26-Pad26) -> VSYS
- J4 pad 27: unconnected-(J4-Pin_27-Pad27) -> GPIO_AD_20
- J4 pad 28: unconnected-(J4-Pin_28-Pad28) -> GND
- J4 pad 29: unconnected-(J4-Pin_29-Pad29) -> GPIO_AD_21
- J4 pad 3: unconnected-(J4-Pin_3-Pad3) -> GPIO_AD_10
- J4 pad 30: unconnected-(J4-Pin_30-Pad30) -> GND
- J4 pad 31: unconnected-(J4-Pin_31-Pad31) -> GND
- J4 pad 32: unconnected-(J4-Pin_32-Pad32) -> GPIO_AD_31
- J4 pad 33: unconnected-(J4-Pin_33-Pad33) -> GPIO_AD_30
- J4 pad 34: unconnected-(J4-Pin_34-Pad34) -> GPIO_AD_32
- J4 pad 35: unconnected-(J4-Pin_35-Pad35) -> GPIO_AD_29
- J4 pad 36: unconnected-(J4-Pin_36-Pad36) -> GPIO_AD_33
- J4 pad 37: unconnected-(J4-Pin_37-Pad37) -> GPIO_AD_28
- J4 pad 38: unconnected-(J4-Pin_38-Pad38) -> GPIO_AD_34
- J4 pad 39: unconnected-(J4-Pin_39-Pad39) -> GPIO_AD_27
- J4 pad 4: unconnected-(J4-Pin_4-Pad4) -> GND
- J4 pad 40: unconnected-(J4-Pin_40-Pad40) -> GPIO_AD_35
- J4 pad 41: unconnected-(J4-Pin_41-Pad41) -> GND
- J4 pad 42: unconnected-(J4-Pin_42-Pad42) -> GND
- J4 pad 43: unconnected-(J4-Pin_43-Pad43) -> VDD_3V3_LP
- J4 pad 44: unconnected-(J4-Pin_44-Pad44) -> GPIO_AD_26
- J4 pad 45: unconnected-(J4-Pin_45-Pad45) -> VDD_3V3_LP
- J4 pad 46: unconnected-(J4-Pin_46-Pad46) -> LPUART1_RX_BOOT
- J4 pad 47: unconnected-(J4-Pin_47-Pad47) -> VDD_3V3_LP
- J4 pad 48: unconnected-(J4-Pin_48-Pad48) -> GPIO_AD_22
- J4 pad 49: unconnected-(J4-Pin_49-Pad49) -> VDD_3V3_LP
- J4 pad 5: unconnected-(J4-Pin_5-Pad5) -> GPIO_AD_11
- J4 pad 50: unconnected-(J4-Pin_50-Pad50) -> GPIO_AD_23
- J4 pad 6: unconnected-(J4-Pin_6-Pad6) -> VSYS
- J4 pad 7: unconnected-(J4-Pin_7-Pad7) -> GPIO_AD_12
- J4 pad 8: unconnected-(J4-Pin_8-Pad8) -> VSYS
- J4 pad 9: unconnected-(J4-Pin_9-Pad9) -> GPIO_AD_13
- J5 pad 1: unconnected-(J5-Pin_1-Pad1) -> GPIO_LPSR_00
- J5 pad 10: unconnected-(J5-Pin_10-Pad10) -> GPIO_EMC_B2_08
- J5 pad 11: unconnected-(J5-Pin_11-Pad11) -> GPIO_LPSR_04
- J5 pad 12: unconnected-(J5-Pin_12-Pad12) -> GPIO_EMC_B2_09
- J5 pad 13: unconnected-(J5-Pin_13-Pad13) -> GPIO_LPSR_05
- J5 pad 14: unconnected-(J5-Pin_14-Pad14) -> GND
- J5 pad 15: unconnected-(J5-Pin_15-Pad15) -> GPIO_LPSR_06
- J5 pad 16: unconnected-(J5-Pin_16-Pad16) -> GPIO_EMC_B2_10
- J5 pad 17: unconnected-(J5-Pin_17-Pad17) -> GPIO_LPSR_07
- J5 pad 18: unconnected-(J5-Pin_18-Pad18) -> GPIO_EMC_B2_11
- J5 pad 19: unconnected-(J5-Pin_19-Pad19) -> GND
- J5 pad 2: unconnected-(J5-Pin_2-Pad2) -> GND
- J5 pad 20: unconnected-(J5-Pin_20-Pad20) -> GPIO_EMC_B2_12
- J5 pad 21: unconnected-(J5-Pin_21-Pad21) -> GPIO_LPSR_08
- J5 pad 22: unconnected-(J5-Pin_22-Pad22) -> GPIO_EMC_B2_13
- J5 pad 23: unconnected-(J5-Pin_23-Pad23) -> GPIO_LPSR_09
- J5 pad 24: unconnected-(J5-Pin_24-Pad24) -> GPIO_EMC_B2_14
- J5 pad 25: unconnected-(J5-Pin_25-Pad25) -> GPIO_AD_00
- J5 pad 26: unconnected-(J5-Pin_26-Pad26) -> GND
- J5 pad 27: unconnected-(J5-Pin_27-Pad27) -> GPIO_AD_01
- J5 pad 28: unconnected-(J5-Pin_28-Pad28) -> GPIO_EMC_B2_15
- J5 pad 29: unconnected-(J5-Pin_29-Pad29) -> GND
- J5 pad 3: unconnected-(J5-Pin_3-Pad3) -> GPIO_LPSR_01
- J5 pad 30: unconnected-(J5-Pin_30-Pad30) -> GPIO_EMC_B2_16
- J5 pad 31: unconnected-(J5-Pin_31-Pad31) -> GPIO_AD_02
- J5 pad 32: unconnected-(J5-Pin_32-Pad32) -> GPIO_EMC_B2_17
- J5 pad 33: unconnected-(J5-Pin_33-Pad33) -> GPIO_AD_03
- J5 pad 34: unconnected-(J5-Pin_34-Pad34) -> GPIO_EMC_B2_18
- J5 pad 35: unconnected-(J5-Pin_35-Pad35) -> GPIO_AD_04
- J5 pad 36: unconnected-(J5-Pin_36-Pad36) -> GPIO_EMC_B2_19
- J5 pad 37: unconnected-(J5-Pin_37-Pad37) -> BT_CFG_IO_EN
- J5 pad 38: unconnected-(J5-Pin_38-Pad38) -> GPIO_EMC_B2_20
- J5 pad 39: unconnected-(J5-Pin_39-Pad39) -> GND
- J5 pad 4: unconnected-(J5-Pin_4-Pad4) -> GPIO_EMC_B2_05
- J5 pad 40: unconnected-(J5-Pin_40-Pad40) -> VSYS
- J5 pad 41: unconnected-(J5-Pin_41-Pad41) -> GPIO_AD_06
- J5 pad 42: unconnected-(J5-Pin_42-Pad42) -> VSYS
- J5 pad 43: unconnected-(J5-Pin_43-Pad43) -> GPIO_AD_07
- J5 pad 44: unconnected-(J5-Pin_44-Pad44) -> VSYS
- J5 pad 45: unconnected-(J5-Pin_45-Pad45) -> GPIO_AD_08
- J5 pad 46: unconnected-(J5-Pin_46-Pad46) -> VSYS
- J5 pad 47: unconnected-(J5-Pin_47-Pad47) -> GPIO_AD_09
- J5 pad 48: unconnected-(J5-Pin_48-Pad48) -> VSYS
- J5 pad 49: unconnected-(J5-Pin_49-Pad49) -> GND
- J5 pad 5: unconnected-(J5-Pin_5-Pad5) -> GPIO_LPSR_02
- J5 pad 50: unconnected-(J5-Pin_50-Pad50) -> VSYS
- J5 pad 6: unconnected-(J5-Pin_6-Pad6) -> GPIO_EMC_B2_06
- J5 pad 7: unconnected-(J5-Pin_7-Pad7) -> GPIO_LPSR_03
- J5 pad 8: unconnected-(J5-Pin_8-Pad8) -> GPIO_EMC_B2_07
- J5 pad 9: unconnected-(J5-Pin_9-Pad9) -> GND
- J6 pad 1: unconnected-(J6-Pin_1-Pad1) -> VDD_1V8
- J6 pad 10: unconnected-(J6-Pin_10-Pad10) -> VDD_3V3
- J6 pad 11: unconnected-(J6-Pin_11-Pad11) -> VDD_3V3
- J6 pad 12: unconnected-(J6-Pin_12-Pad12) -> VDD_3V3
- J6 pad 13: unconnected-(J6-Pin_13-Pad13) -> VDD_3V3
- J6 pad 14: unconnected-(J6-Pin_14-Pad14) -> VDD_3V3
- J6 pad 15: unconnected-(J6-Pin_15-Pad15) -> VDD_3V3
- J6 pad 16: unconnected-(J6-Pin_16-Pad16) -> VDD_3V3
- J6 pad 17: unconnected-(J6-Pin_17-Pad17) -> GPIO_SNVS_00
- J6 pad 18: unconnected-(J6-Pin_18-Pad18) -> GND
- J6 pad 19: unconnected-(J6-Pin_19-Pad19) -> GPIO_SNVS_01
- J6 pad 2: unconnected-(J6-Pin_2-Pad2) -> VDD_1V8
- J6 pad 20: unconnected-(J6-Pin_20-Pad20) -> GPIO_DISP_B1_00
- J6 pad 21: unconnected-(J6-Pin_21-Pad21) -> GPIO_SNVS_02
- J6 pad 22: unconnected-(J6-Pin_22-Pad22) -> GPIO_DISP_B1_01
- J6 pad 23: unconnected-(J6-Pin_23-Pad23) -> GPIO_SNVS_03
- J6 pad 24: unconnected-(J6-Pin_24-Pad24) -> GPIO_DISP_B1_02
- J6 pad 25: unconnected-(J6-Pin_25-Pad25) -> GPIO_SNVS_04
- J6 pad 26: unconnected-(J6-Pin_26-Pad26) -> GPIO_DISP_B1_03
- J6 pad 27: unconnected-(J6-Pin_27-Pad27) -> GND
- J6 pad 28: unconnected-(J6-Pin_28-Pad28) -> GPIO_DISP_B1_04
- J6 pad 29: unconnected-(J6-Pin_29-Pad29) -> GPIO_SNVS_05
- J6 pad 3: unconnected-(J6-Pin_3-Pad3) -> VDD_1V8
- J6 pad 30: unconnected-(J6-Pin_30-Pad30) -> GPIO_DISP_B1_05
- J6 pad 31: unconnected-(J6-Pin_31-Pad31) -> GPIO_SNVS_06
- J6 pad 32: unconnected-(J6-Pin_32-Pad32) -> GND
- J6 pad 33: unconnected-(J6-Pin_33-Pad33) -> GPIO_SNVS_07
- J6 pad 34: unconnected-(J6-Pin_34-Pad34) -> GPIO_DISP_B1_06
- J6 pad 35: unconnected-(J6-Pin_35-Pad35) -> GPIO_SNVS_08
- J6 pad 36: unconnected-(J6-Pin_36-Pad36) -> GPIO_DISP_B1_07
- J6 pad 37: unconnected-(J6-Pin_37-Pad37) -> GPIO_SNVS_09
- J6 pad 38: unconnected-(J6-Pin_38-Pad38) -> GPIO_DISP_B1_08
- J6 pad 39: unconnected-(J6-Pin_39-Pad39) -> GND
- J6 pad 4: unconnected-(J6-Pin_4-Pad4) -> VDD_1V8
- J6 pad 40: unconnected-(J6-Pin_40-Pad40) -> GPIO_DISP_B1_09
- J6 pad 41: unconnected-(J6-Pin_41-Pad41) -> GPIO_EMC_B2_00
- J6 pad 42: unconnected-(J6-Pin_42-Pad42) -> GPIO_DISP_B1_10
- J6 pad 43: unconnected-(J6-Pin_43-Pad43) -> GPIO_EMC_B2_01
- J6 pad 44: unconnected-(J6-Pin_44-Pad44) -> GPIO_DISP_B1_11
- J6 pad 45: unconnected-(J6-Pin_45-Pad45) -> GPIO_EMC_B2_02
- J6 pad 46: unconnected-(J6-Pin_46-Pad46) -> GND
- J6 pad 47: unconnected-(J6-Pin_47-Pad47) -> GPIO_EMC_B2_03
- J6 pad 48: unconnected-(J6-Pin_48-Pad48) -> GPIO_DISP_B2_00
- J6 pad 49: unconnected-(J6-Pin_49-Pad49) -> GPIO_EMC_B2_04
- J6 pad 5: unconnected-(J6-Pin_5-Pad5) -> VDD_1V8
- J6 pad 50: unconnected-(J6-Pin_50-Pad50) -> GPIO_DISP_B2_01
- J6 pad 6: unconnected-(J6-Pin_6-Pad6) -> VDD_1V8
- J6 pad 7: unconnected-(J6-Pin_7-Pad7) -> VDD_1V8
- J6 pad 8: unconnected-(J6-Pin_8-Pad8) -> VDD_1V8
- J6 pad 9: unconnected-(J6-Pin_9-Pad9) -> VDD_3V3
- J7 pad 10: unconnected-(J7-Pin_10-Pad10) -> USDHC2_CMD
- J7 pad 11: unconnected-(J7-Pin_11-Pad11) -> GND
- J7 pad 12: unconnected-(J7-Pin_12-Pad12) -> USDHC2_CLK
- J7 pad 14: unconnected-(J7-Pin_14-Pad14) -> USDHC2_DATA0
- J7 pad 16: unconnected-(J7-Pin_16-Pad16) -> USDHC2_DATA1
- J7 pad 17: unconnected-(J7-Pin_17-Pad17) -> GND
- J7 pad 18: unconnected-(J7-Pin_18-Pad18) -> USDHC2_DATA2
- J7 pad 19: unconnected-(J7-Pin_19-Pad19) -> GPIO_DISP_B2_15
- J7 pad 2: unconnected-(J7-Pin_2-Pad2) -> Net-(J7-Pin_2)
- J7 pad 20: unconnected-(J7-Pin_20-Pad20) -> USDHC2_DATA3
- J7 pad 21: unconnected-(J7-Pin_21-Pad21) -> GPIO_DISP_B2_14
- J7 pad 22: unconnected-(J7-Pin_22-Pad22) -> Net-(J7-Pin_2)
- J7 pad 23: unconnected-(J7-Pin_23-Pad23) -> GPIO_DISP_B2_13
- J7 pad 24: unconnected-(J7-Pin_24-Pad24) -> GPIO_SD_B1_05
- J7 pad 25: unconnected-(J7-Pin_25-Pad25) -> GPIO_DISP_B2_12
- J7 pad 26: unconnected-(J7-Pin_26-Pad26) -> GPIO_SD_B1_04
- J7 pad 27: unconnected-(J7-Pin_27-Pad27) -> GPIO_DISP_B2_11
- J7 pad 28: unconnected-(J7-Pin_28-Pad28) -> GPIO_SD_B1_03
- J7 pad 29: unconnected-(J7-Pin_29-Pad29) -> GND
- J7 pad 30: unconnected-(J7-Pin_30-Pad30) -> GPIO_SD_B1_01
- J7 pad 31: unconnected-(J7-Pin_31-Pad31) -> GPIO_DISP_B2_10
- J7 pad 32: unconnected-(J7-Pin_32-Pad32) -> GPIO_SD_B1_00
- J7 pad 33: unconnected-(J7-Pin_33-Pad33) -> GPIO_DISP_B2_09
- J7 pad 34: unconnected-(J7-Pin_34-Pad34) -> Net-(J7-Pin_2)
- J7 pad 35: unconnected-(J7-Pin_35-Pad35) -> GPIO_DISP_B2_08
- J7 pad 36: unconnected-(J7-Pin_36-Pad36) -> EN_ADCS
- J7 pad 37: unconnected-(J7-Pin_37-Pad37) -> GPIO_DISP_B2_07
- J7 pad 38: unconnected-(J7-Pin_38-Pad38) -> DAC_OUT
- J7 pad 39: unconnected-(J7-Pin_39-Pad39) -> GPIO_DISP_B2_06
- J7 pad 4: unconnected-(J7-Pin_4-Pad4) -> GPIO_EMC_B1_41
- J7 pad 40: unconnected-(J7-Pin_40-Pad40) -> PMIC_ON_REQ
- J7 pad 41: unconnected-(J7-Pin_41-Pad41) -> GND
- J7 pad 42: unconnected-(J7-Pin_42-Pad42) -> WAKEUP
- J7 pad 43: unconnected-(J7-Pin_43-Pad43) -> GPIO_DISP_B2_05
- J7 pad 44: unconnected-(J7-Pin_44-Pad44) -> PMIC_STBY_REQ
- J7 pad 45: unconnected-(J7-Pin_45-Pad45) -> GPIO_DISP_B2_04
- J7 pad 46: unconnected-(J7-Pin_46-Pad46) -> ONOFF
- J7 pad 47: unconnected-(J7-Pin_47-Pad47) -> GPIO_DISP_B2_03
- J7 pad 48: unconnected-(J7-Pin_48-Pad48) -> Net-(J7-Pin_2)
- J7 pad 49: unconnected-(J7-Pin_49-Pad49) -> GPIO_DISP_B2_02
- J7 pad 5: unconnected-(J7-Pin_5-Pad5) -> GND
- J7 pad 50: unconnected-(J7-Pin_50-Pad50) -> Net-(J7-Pin_2)
- J7 pad 6: unconnected-(J7-Pin_6-Pad6) -> GPIO_EMC_B1_40
- J7 pad 8: unconnected-(J7-Pin_8-Pad8) -> Net-(J7-Pin_2)
Routing:
- net Net-(J7-Pin_2): track 0.00 -> 67.7 mm
- net GPIO_LPSR_02: track 0.00 -> 55.3 mm, vias 0 -> 1
- net GPIO_LPSR_00: track 0.00 -> 55.3 mm, vias 0 -> 1
- net GPIO_LPSR_01: track 0.00 -> 54.4 mm, vias 0 -> 1
- net GPIO_EMC_B2_19: track 0.00 -> 53.8 mm, vias 0 -> 1
- net GPIO_EMC_B2_18: track 0.00 -> 53.5 mm, vias 0 -> 1
- net GPIO_EMC_B2_17: track 0.00 -> 53.3 mm, vias 0 -> 1
- net GPIO_LPSR_03: track 0.00 -> 52.3 mm, vias 0 -> 1
- net GPIO_EMC_B2_20: track 0.00 -> 52.3 mm, vias 0 -> 1
- net GPIO_DISP_B2_01: track 0.00 -> 51.0 mm, vias 0 -> 1
- net GPIO_LPSR_04: track 0.00 -> 50.9 mm, vias 0 -> 1
- net GPIO_LPSR_05: track 0.00 -> 50.6 mm, vias 0 -> 1
- net GPIO_EMC_B2_05: track 0.00 -> 50.6 mm
- net GPIO_EMC_B2_15: track 0.00 -> 50.1 mm
- net GPIO_EMC_B2_06: track 0.00 -> 49.7 mm
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- added copper zone on B.Cu, net GND
- added copper zone on F.Cu, net GND
- added copper zone on In1.Cu, net GND
- added copper zone on F.Cu, net VDD_1V8
- added copper zone on F.Cu, net VDD_3V3
- added copper zone on F.Cu, net VDD_3V3_LP
- added copper zone on F.Cu, net VSYS
- added copper zone on In2.Cu, net VSYS
