File: hardware/sqrt_of_g_temp/sqrt_of_g_temp.kicad_sch (KiCad schematic)
At the start: 17 parts, among them J1 353620650, J1 CLP-105-02-X-D, J10 Thruster Connector, J2 353620650, J2 DF40HC_3.0_-100DS-0.4V_51_, J21 Conn_01x10, J3 353620850, J3 DF40HC_3.0_-100DS-0.4V_51_, J4 353620850

Commit message: pre-autorouter part 2
Other:
- added sheet h-bridge (hbridge.kicad_sch)

Commit message: ads board 1.0.1
Parts:
- removed J1, J2: 353620650, mainboard:MOLEX_35362-0650, symbol mainboard:35362-0650
- removed J10: Thruster Connector, CON_353621050, symbol adcs:353621050
- removed J21: Conn_01x10, Connector_PinHeader_2.54mm:PinHeader_1x10_P2.54mm_Vertical, symbol Connector_Generic:Conn_01x10
- removed J3, J4: 353620850, adcs:SHDR8W50P0X200_1X8_1830X550X850P, symbol Connector_Generic:Conn_01x08
- added J1, J11, J2, J3: 5055680431, adcs:CON_5055680431, symbol adcs:5055680431
- added J12, J4: 5055680631, adcs:CON_5055680631, symbol adcs:5055680631
- H2, H3, H4, H5, H6, H7, H8: now left out of the parts list
- renumbered J1 to J5, J2 to J6, J3 to J7
Connections:
- net GPIO_LPSR_05 is gone; now on net RX_FROM_GPS: J6.13
- net GPIO_LPSR_08 is gone; now on net TX_TO_GPS: J6.21
- net VDD_3V3 is gone; now on net +3V3: J6.2, J6.4, J6.6, J6.8, J7.1, J7.2, J7.3, J7.4, J7.5, J7.6, J7.7, J7.8
- net 3V3_PD1: now also J1.1, J3.1, J4.1
- net 3V3_PD2: now also J11.1, J12.1, J2.1
- net GND: now also J1.2, J1.5 (Shield), J1.6 (Shield), J11.2, J11.5 (Shield), J11.6 (Shield), J12.2, J12.7 (SHIELD), J12.8 (SHIELD), J2.2, J2.5 (Shield), J2.6 (Shield), J3.2, J3.5 (Shield), J3.6 (Shield), J4.2, J4.7 (SHIELD), J4.8 (SHIELD)
- net GPIO_AD_06: now also J1.3
- net GPIO_AD_07: now also J3.3
- net GPIO_AD_08: now also J4.3
- net GPIO_AD_09: now also J4.4
- net GPIO_AD_10: now also J4.5
- net GPIO_AD_11: now also J4.6
- net GPIO_AD_12: now also J2.3
- net GPIO_AD_14: now also J11.3
- net GPIO_AD_15: now also J12.3
- net GPIO_AD_16: now also J12.4
- net GPIO_AD_17: now also J12.5
- net GPIO_AD_18: now also J12.6
- net GPIO_AD_00 renamed CS_MAG1
- net GPIO_AD_01 renamed CS_MAG2
- net GPIO_AD_02 renamed EN_PD1
- net GPIO_AD_03 renamed EN_PD2
- net GPIO_DISP_B1_06: no longer names the net of J7.34
- net GPIO_DISP_B1_07: no longer names the net of J7.36
- net GPIO_DISP_B1_08: no longer names the net of J7.38
- net GPIO_DISP_B1_09: no longer names the net of J7.40
- net GPIO_DISP_B1_10: no longer names the net of J7.42
- net GPIO_DISP_B1_11: no longer names the net of J7.44
- net GPIO_DISP_B2_00: no longer names the net of J7.48
- net GPIO_DISP_B2_01: no longer names the net of J7.50
- net GPIO_DISP_B2_02: no longer names the net of J7.52
- net GPIO_DISP_B2_03: no longer names the net of J7.54
- net GPIO_DISP_B2_04: no longer names the net of J7.56
- net GPIO_DISP_B2_05: no longer names the net of J7.58
- net GPIO_DISP_B2_06 renamed RF_BUSY
- net GPIO_DISP_B2_07 renamed EN_RF
- net GPIO_DISP_B2_08 renamed RF_IO1
- net GPIO_DISP_B2_09 renamed RF_IO2
- net GPIO_DISP_B2_10 renamed RF_IO3
- net GPIO_DISP_B2_11 renamed RF_RX_EN
- net GPIO_DISP_B2_12 renamed SCK
- net GPIO_DISP_B2_13 renamed SDI
- net GPIO_DISP_B2_14 renamed SDO
- net GPIO_DISP_B2_15 renamed RF_TX_EN
- net GPIO_EMC_B2_10 renamed CS_RF
- net GPIO_EMC_B2_13 renamed RF_RST
- net GPIO_LPSR_00 renamed EN_MAG1
- net GPIO_LPSR_01 renamed DRDY_MAG1
- net GPIO_LPSR_02: no longer names the net of J6.5
- net GPIO_LPSR_03: no longer names the net of J6.7
- net GPIO_LPSR_07 renamed EN_MAG2
- net GPIO_LPSR_09 renamed DRDY_MAG2
- net VDD_1V8 renamed +1V8
- no-connect marks 15 -> 33
Other:
- sheet IMU1_and_MAG1 renamed MAG1
- sheet IMU2_and_MAG2 renamed MAG2
- removed sheet Magnetorquer Controller 1
- removed sheet Magnetorquer Controller 2
- removed sheet Motor Controller 1
- removed sheet Motor Controller 2
- removed sheet Motor Controller 3
- removed sheet Motor Controller 4
- removed sheet h-bridge
- added sheet 2.4 Ghz modem (lora_2400.kicad_sch)
- sheet GPS ports: added V_BCKP; removed none
- sheet MAG1 ports: added CS_SENSOR, SCK_SENSOR, SDI_SENSOR, SDO_SENSOR; removed SCL_SENSE, SDA_SENSE
- sheet MAG2 ports: added CS_SENSOR, SCK_SENSOR, SDI_SENSOR, SDO_SENSOR; removed SCL_SENSE, SDA_SENSE
- note added: "ADC1"
- note added: "ADC2"
- note added: "GPIO_AD_00"
- note added: "GPIO_AD_01"
- note added: "GPIO_DISP_B1_06"
- note added: "GPIO_DISP_B1_07"
- note added: "GPIO_DISP_B1_08"
- note added: "GPIO_DISP_B1_09"
- note added: "GPIO_DISP_B1_10"
- note added: "GPIO_DISP_B1_11"
- note added: "GPIO_DISP_B2_00"
- note added: "GPIO_DISP_B2_01"
- note added: "GPIO_DISP_B2_02"
- note added: "GPIO_DISP_B2_03"
- note added: "GPIO_DISP_B2_04"
- note added: "GPIO_DISP_B2_05"
- note added: "GPIO_DISP_B2_06"
- note added: "GPIO_DISP_B2_07"
- note added: "GPIO_DISP_B2_08"
- note added: "GPIO_DISP_B2_09"
- note added: "GPIO_DISP_B2_10"
- note added: "GPIO_DISP_B2_11"
- note added: "GPIO_DISP_B2_12"
- note added: "GPIO_DISP_B2_13"
- note added: "GPIO_DISP_B2_14"
- note added: "GPIO_DISP_B2_15"
- note added: "GPIO_EMC_B2_10"
- note added: "GPIO_EMC_B2_13"
- note added: "GPIO_LPSR_00"
- note added: "GPIO_LPSR_01"
- note added: "GPIO_LPSR_05"
- note added: "GPIO_LPSR_07"
- note added: "GPIO_LPSR_08"
- note added: "GPIO_LPSR_09"
- note added: "LPISPI2"
- note added: "LPUART11"
- note removed: "Coils"
- note removed: "GPIO"
- note removed: "LDO for analog 3V3 supply? add inductor, caps to filter things out? Should I make an analog GND plane? I feel like I am fine."
- note removed: "LPI2C1"
- note removed: "LPI2C2"
- note removed: "LPI2C4"
- note removed: "LPUART4"
- note removed: "PWM"
- note removed: "These are set up to either run the current coils, or run new coils that just have h-bridges on them (i.e. by PWM-ing them). The jumpers are to protect the GNC board from Vsolar (which is on the current side panel harnesses)"
- note removed: "Thruster"
- note removed: "Wheels"
- note removed: "X+"
- note removed: "X-"
- note removed: "Y+"
- note removed: "Y-"
- note removed: "Z+"
- note removed: "Z-"
- company: (none) -> Stanford Student Space Initiative
- title: (none) -> √g
- moved on the sheet: J5, J6, J7
Changed lines of the file:
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@@
-(kicad_sch (version 20230121) (generator eeschema)
-  (paper "A2")
+(kicad_sch
+	(version 20231120)
+	(generator "eeschema")
+	(generator_version "8.0")
+	(paper "A2")
+	(title_block
+		(title "√g")
+		(date "2024-08-05")
+		(rev "1.0.1")
+		(company "Stanford Student Space Initiative")
+		(comment 1 "RE: Flynn Dreilinger")
+	)
