File: hardware/PCBranch/PCBranch.kicad_pcb (KiCad board)
At the start: 4 copper layers, 90.2 x 95.9 mm, 15 parts, among them J1 CLP-105-02-X-D, J2 DF40HC_3.0_-100DS-0.4V_51_, J3 DF40HC_3.0_-100DS-0.4V_51_, J4 Conn_02x25_Odd_Even, J5 Conn_02x25_Odd_Even, J6 Conn_02x25_Odd_Even, J7 Conn_02x25_Odd_Even

Commit message: 1.0.1
Other:
- board text added: "Flynn Dreilinger • July 2024"
- board text added: "GND AD_10 AD_11 AD_12 AD_13 GND AD_14 AD_15 AD_16 AD_17 GND AD_18 AD_19 AD_20 AD_21 GND AD_30 AD_29 AD_28 AD_27 GND VDD_3V3_LP VDD_3V3_LP VDD_3V3_LP VDD_3V3_LP"
- board text added: "GND EMC_B2_05 EMC_B2_06 EMC_B2_07 EMC_B2_08 EMC_B2_09 GND EMC_B2_10 EMC_B2_11 EMC_B2_12 EMC_B2_13 EMC_B2_14 GND EMC_B2_15 EMC_B2_16 EMC_B2_17 EMC_B2_18 EMC_B2_19 EMC_B2_20 VSYS VSYS VSYS VSYS VSYS VSYS"
- board text added: "GND GND VSYS VSYS VSYS VSYS GND VSYS VSYS VSYS VSYS VSYS VSYS GND GND AD_31 AD_32 AD_33 AD_34 AD_35 GND AD_26 LPUART1_RX_BOOT AD_22 AD_23"
- board text added: "LPSR_00 LPSR_01 LPSR_02 LPSR_03 GND LPSR_04 LPSR_05 LPSR_06 LPSR_07 GND LPSR_08 LPSR_09 AD_00 AD_01 GND AD_02 AD_03 AD_04 BT_CFG_IO_EN GND AD_06 AD_07 AD_08 AD_09 GND"
- board text added: "NC NC GND NC NC GND NC NC GND DISP_B2_15 DISP_B2_14 DISP_B2_13 DISP_B2_12 DISP_B2_11 GND DISP_B2_10 DISP_B2_09 DISP_B2_08 DISP_B2_07 DISP_B2_06 GND DISP_B2_05 DISP_B2_04 DISP_B2_03 DISP_B2_02"
- board text added: "Net-(J7-Pin_2) EMC_B1_41 EMC_B1_40 Net-(J7-Pin_2) USDHC2_CMD USDHC2_CLK USDHC2_DATA0 USDHC2_DATA1 USDHC2_DATA2 USDHC2_DATA3 Net-(J7-Pin_2) SD_B1_05 SD_B1_04 SD_B1_03 SD_B1_01 SD_B1_00 Net-(J7-Pin_2) EN_ADCS DAC_OUT PMIC_ON_REQ WAKEUP PMIC_STBY_REQ ONOFF Net-(J7-Pin_2) Net-(J7-Pin_2)"
- board text added: "PCBranch 1.0.1"
- board text added: "VDD_1V8 VDD_1V8 VDD_1V8 VDD_1V8 VDD_3V3 VDD_3V3 VDD_3V3 VDD_3V3 GND DISP_B1_00 DISP_B1_01 DISP_B1_02 DISP_B1_03 DISP_B1_04 DISP_B1_05 GND DISP_B1_06 DISP_B1_07 DISP_B1_08 DISP_B1_09 DISP_B1_10 DISP_B1_11 GND DISP_B2_00 DISP_B2_01"
- board text added: "VDD_1V8 VDD_1V8 VDD_1V8 VDD_3V3 VDD_3V3 VDD_3V3 VDD_3V3 SNVS_00 SNVS_01 SNVS_02 SNVS_03 SNVS_04 GND SNVS_05 SNVS_06 SNVS_07 SNVS_08 SNVS_09 GND EMC_B2_00 EMC_B2_01 EMC_B2_02 EMC_B2_03 EMC_B2_04"
