File: hardware/PCBranch/PCBranch.kicad_sch (KiCad schematic)
At the start: 15 parts, among them J1 CLP-105-02-X-D, J2 DF40HC_3.0_-100DS-0.4V_51_, J3 DF40HC_3.0_-100DS-0.4V_51_, J4 Conn_02x25_Odd_Even, J5 Conn_02x25_Odd_Even, J6 Conn_02x25_Odd_Even, J7 Conn_02x25_Odd_Even

Commit message: PrintedCoralBoard
Parts:
- H2, H3, H4, H5, H6, H7, H8: now left out of the parts list
- J1: MANUFACTURER SAMTEC -> (none); Manufacturer_Name (none) -> SAMTEC; Manufacturer_Part_Number (none) -> CLP-105-02-L-D
- J4, J5, J6, J7: LCSC Part Number (none) -> C350296
Other:
- moved on the sheet: J3
Changed lines of the file:
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@@
-(kicad_sch (version 20230121) (generator eeschema)
-  (paper "A2")
+(kicad_sch
+	(version 20231120)
+	(generator "eeschema")
+	(generator_version "8.0")
+	(paper "A2")
