File: hardware/Soldermander/board_to_board.kicad_sch (KiCad schematic)
At the start: 3 parts, among them J8 SAMTEC-FTS-105-03-X-DV

Commit message: pre-autorouter part 2
Connections:
- net GPIO_DISP_B1_06: no longer names the net of J?.34
- net GPIO_DISP_B1_07: no longer names the net of J?.36
- net GPIO_DISP_B1_08: no longer names the net of J?.38
- net GPIO_DISP_B1_09: no longer names the net of J?.40
- net GPIO_DISP_B1_10: no longer names the net of J?.42
- net GPIO_DISP_B1_11: no longer names the net of J?.44
- net GPIO_DISP_B2_00: no longer names the net of J?.48
- net GPIO_DISP_B2_01: no longer names the net of J?.50
- net GPIO_DISP_B2_02: no longer names the net of J?.52
- net GPIO_DISP_B2_03: no longer names the net of J?.54
- net GPIO_DISP_B2_04: no longer names the net of J?.56
- net GPIO_DISP_B2_05: no longer names the net of J?.58
- net GPIO_LPSR_02: no longer names the net of J?.5
- net GPIO_LPSR_03: no longer names the net of J?.7
- net LPUART1_RX_BOOT: no longer names the net of J?.85
- no-connect marks 15 -> 31
Other:
- note added: "GPIO_DISP_B1_06"
- note added: "GPIO_DISP_B1_07"
- note added: "GPIO_DISP_B1_08"
- note added: "GPIO_DISP_B1_09"
- note added: "GPIO_DISP_B1_10"
- note added: "GPIO_DISP_B1_11"
- note added: "GPIO_DISP_B2_00"
- note added: "GPIO_DISP_B2_01"
- note added: "GPIO_DISP_B2_02"
- note added: "GPIO_DISP_B2_03"
- note added: "GPIO_DISP_B2_04"
- note added: "GPIO_DISP_B2_05"
- note added: "GPIO_LPSR_02"
- note added: "GPIO_LPSR_03"
- note added: "LPUART1_RX_BOOT"
- moved on the sheet: J?
