File: hardware/Soldermander/boot_config.kicad_sch (KiCad schematic)
At the start: 30 parts, among them SW2 SW_DIP_x10, SW3 SW_DIP_x04

Commit message: pre-autorouter part 2
Parts:
- R37, R38, R39, R40, R41, R42, R43, R44, R45, R46, R47, R48, R49, R50, R51, R52, R53, R54, R55, R56, R57, R58, R59, R60, R61, R62, R63, R64: renamed from R?; footprint adcs:Perfect_0402 -> Resistor_SMD:R_0402_1005Metric
