File: hardware/Soldermander/power.kicad_sch (KiCad schematic)
At the start: 42 parts, among them U1 TPS16630PWPR, U10 CD40109BQNSRQ1, U7 TPS54226PWPRPWP14_2P31X2P46-L, U8 TPS54226PWPRPWP14_2P31X2P46-L, U9 LT3014IS5-TRMPBF

Commit message: update 3.3uH inductor
Parts:
- L3, L4: footprint mainboard:L_2141 -> Inductor_SMD:L_1210_3225Metric; Flight HPC5040NF-3R3MTH -> SRP3212-3R3M; JLCPCB P/N C304367 -> (none); Manufacturer_Name TAI-TECH -> Bourns; Power Rating (none) -> 3.1A, 3.4A Saturation; Proto HPC5040NF-3R3MTH -> SRP3212-3R3M; Supplier 1 (none) -> Digi-Key

Commit message: pre-autorouter part 2
Parts:
- C84, C85, C86, C87, C88, C89, C? (x3): footprint adcs:Perfect_0402 -> Capacitor_SMD:C_0402_1005Metric
- R14, R2, R21, R34, R35: renamed from R5; footprint adcs:Perfect_0402 -> Resistor_SMD:R_0402_1005Metric
- R15, R19: renamed from R6; footprint adcs:Perfect_0402 -> Resistor_SMD:R_0402_1005Metric
- R27, R28, R29, R30, R31, R32, R5, R6: footprint adcs:Perfect_0402 -> Resistor_SMD:R_0402_1005Metric
- gave numbers to parts that had none: 1
Other:
- note removed: "Could also use EN_ADCS here, in case the E-fuse shorts on"

Commit message: PrintedCoralBoard
Parts:
- C79, C81, C82, C83: JLCPCB P/N (none) -> C191180
- C84, C85: Footprint (for JLCPCB) 0402 -> (none)
