File: hardware/Soldermander/rt1176_1.kicad_sch (KiCad schematic)
At the start: 41 parts, among them SW1 SWITCH_SMT4.6X2.8, U2 MIMXRT1176

Commit message: pre-autorouter part 2
Parts:
- removed C12, C13: 1uF, adcs:Perfect_0201, symbol Device:C_Small
- removed C15, C17, C22: 4.7uF, adcs:Perfect_0201, symbol Device:C_Small
- removed C26: 2.2uF, adcs:Perfect_0201, symbol Device:C_Small
- removed C42: 0.1uF, adcs:Perfect_0201, symbol Device:C_Small
- added C16: 22uF, Capacitor_SMD:C_0603_1608Metric, symbol Device:C_Small
- added C24, C7: 4.7uF, Capacitor_SMD:C_0402_1005Metric, symbol Device:C_Small
- added C28: 0.1uF, Capacitor_SMD:C_0402_1005Metric, symbol Device:C_Small
- added C29: 0.22uF, Capacitor_SMD:C_0402_1005Metric, symbol Device:C_Small
- added L5: 4.7µH, adcs:IND_4x4mm, symbol Device:L
- added R11: 30kΩ, Resistor_SMD:R_0402_1005Metric, symbol Device:R_Small_US
- added R9: 4.7kΩ, Resistor_SMD:R_0402_1005Metric, symbol Device:R_Small_US
- C10, C14, C23, C34, C38, C40, C41, C43, C6, C8, C9, C? (x2): footprint adcs:Perfect_0201 -> Capacitor_SMD:C_0402_1005Metric
- C31, C? (x4): footprint adcs:Perfect_0402 -> Capacitor_SMD:C_0402_1005Metric
- FB1, FB2: footprint adcs:Perfect_0402 -> Fuse:Fuse_0402_1005Metric
- R7, R8: footprint adcs:Perfect_0402 -> Resistor_SMD:R_0402_1005Metric
- gave numbers to parts that had none: 1
Connections:
- net ADC_1V8_IN: now also C34.1, U2.M11 (VDDA_1P8_IN)
- net GND: now also C16.2, C24.2, C28.2, C29.2, C7.2, R9.1; no longer U2.N4 (DCDC_MODE), U2.P3 (DCDC_PSWITCH)
- net VDD_3V3: now also U2.L5 (DCDC_IN_Q), U2.M5 (DCDC_IN_1), U2.N5 (DCDC_IN_2), C16.1, C24.1, C28.1, R11.2
- net VDD_SOC_IN: now also U2.K8 (DCDC_DIG_1), U2.K9 (DCDC_DIG_2), U2.L8 (DCDC_DIG_3)
- net DCDC_1V8_OUT: now reaches U2.M7 (DCDC_ANA_1)
- net DCDC_1V8_OUT: now also U2.M8 (DCDC_ANA_2)
- net at U2.T3 (DCDC_LP_1): now also U2.U3 (DCDC_LP_2), L5.1
- net at U2.T4 (DCDC_LN_1): now also U2.U4 (DCDC_LN_2), L5.2
- net VDD_1P0 renamed VDDA_1P0
- new net DCDC_MODE: C7.1, R9.2, U2.N4 (DCDC_MODE)
- new net DCDC_PSWITCH: C29.1, R11.1, U2.P3 (DCDC_PSWITCH)
- no-connect marks 14 -> 2
Other:
- note added: "Changed from Coral schematic, based on HDUG note 2 on pAge 3 "Avoid using the internal DCDC/LDO output for the ADC reference. Use an external voltage reference, which is more accurate.""
- note added: "Deleted 4.7uF cap here"
- note added: "Deleted Caps here, since we are not using this output."
- note added: "Deleted Caps here, since we are only using this to power the micro (and there are a lot of caps in U2A above)"
- note added: "Deleted some caps here"
- note added: "Removed cap since we aren't using this"
- note removed: "Not using internal regulators. HDUG page 6."
- moved on the sheet: C10, C38, C4, C40, C43, C6, FB2, R8, TP3

Commit message: PrintedCoralBoard
Parts:
- C10, C28, C34, C?: Footprint (for JLCPCB) 0201 -> (none)
- C14, C23, C24, C29, C38, C40, C41, C43, C6, C7, C8, C9, C?: Footprint (for JLCPCB) 0201 -> 0402
- C16: Footprint (for JLCPCB) 0402 -> 0603
- C31: Footprint (for JLCPCB) 0402 -> (none)
