File: hardware/Soldermander/rt1176_2.kicad_sch (KiCad schematic)
At the start: 9 parts, among them U2 MIMXRT1176

Commit message: pre-autorouter part 2
Parts:
- C44, C45, C46, C47, C48, C49, C50: renamed from C?; footprint adcs:Perfect_0201 -> Capacitor_SMD:C_0402_1005Metric
- R10: renamed from R?; footprint adcs:Perfect_0402 -> Resistor_SMD:R_0402_1005Metric

Commit message: PrintedCoralBoard
Parts:
- C44, C45, C46, C47, C48, C49, C50: Footprint (for JLCPCB) 0201 -> 0402
Changed lines of the file:
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@@
 			)
 		)
-		(property "Footprint (for JLCPCB)" "0201"
+		(property "Footprint (for JLCPCB)" "0402"
 			(at 217.805 79.375 0)
 			(effects
@@
 			)
 		)
+		(property "LCSC P/N" ""
+			(at 217.805 79.375 0)
+			(effects
+				(font
+					(size 1.27 1.27)
+				)
+				(hide yes)
+			)
+		)
+		(property "LCSC P/N Flight" ""
+			(at 217.805 79.375 0)
+			(effects
+				(font
+					(size 1.27 1.27)
+				)
+				(hide yes)
+			)
+		)
 		(pin "1"
 		)
@@
 			)
 		)
-		(property "Footprint (for JLCPCB)" "0201"
+		(property "Footprint (for JLCPCB)" "0402"
 			(at 217.805 104.775 0)
 			(effects
@@
 			)
 		)
+		(property "LCSC P/N" ""
+			(at 217.805 104.775 0)
+			(effects
+				(font
+					(size 1.27 1.27)
+				)
+				(hide yes)
+			)
+		)
+		(property "LCSC P/N Flight" ""
+			(at 217.805 104.775 0)
+			(effects
+				(font
+					(size 1.27 1.27)
+				)
+				(hide yes)
+			)
+		)
 		(pin "1"
 		)
@@
 			)
 		)
-		(property "Footprint (for JLCPCB)" "0201"
+		(property "Footprint (for JLCPCB)" "0402"
 			(at 62.23 170.815 0)
 			(effects
@@
 			)
 		)
+		(property "LCSC P/N" ""
+			(at 62.23 170.815 0)
+			(effects
+				(font
+					(size 1.27 1.27)
+				)
+				(hide yes)
+			)
+		)
+		(property "LCSC P/N Flight" ""
+			(at 62.23 170.815 0)
+			(effects
+				(font
+					(size 1.27 1.27)
+				)
+				(hide yes)
+			)
+		)
 		(pin "1"
 		)
@@
 			)
 		)
+		(property "LCSC P/N" ""
+			(at 97.79 180.975 0)
+			(effects
+				(font
+					(size 1.27 1.27)
+				)
+				(hide yes)
+			)
+		)
+		(property "LCSC P/N Flight" ""
+			(at 97.79 180.975 0)
+			(effects
+				(font
+					(size 1.27 1.27)
+				)
+				(hide yes)
+			)
+		)
 		(pin "L9"
 		)
@@
 			)
 		)
-		(property "Footprint (for JLCPCB)" "0201"
+		(property "Footprint (for JLCPCB)" "0402"
 			(at 69.215 90.805 0)
 			(effects
@@
 			)
 		)
+		(property "LCSC P/N" ""
+			(at 69.215 90.805 0)
+			(effects
+				(font
+					(size 1.27 1.27)
+				)
+				(hide yes)
+			)
+		)
+		(property "LCSC P/N Flight" ""
+			(at 69.215 90.805 0)
+			(effects
+				(font
+					(size 1.27 1.27)
+				)
+				(hide yes)
+			)
+		)
 		(pin "1"
 		)
@@
 			)
 		)
+		(property "LCSC P/N" ""
+			(at 99.695 90.805 0)
+			(effects
+				(font
+					(size 1.27 1.27)
+				)
+				(hide yes)
+			)
+		)
+		(property "LCSC P/N Flight" ""
+			(at 99.695 90.805 0)
+			(effects
+				(font
+					(size 1.27 1.27)
+				)
+				(hide yes)
+			)
+		)
 		(pin "L9"
 		)
@@
 			)
 		)
+		(property "LCSC P/N" ""
+			(at 257.81 191.77 0)
+			(effects
+				(font
+					(size 1.27 1.27)
+				)
+				(hide yes)
+			)
+		)
+		(property "LCSC P/N Flight" ""
+			(at 257.81 191.77 0)
+			(effects
+				(font
+					(size 1.27 1.27)
+				)
+				(hide yes)
+			)
+		)
 		(pin "L9"
 		)
@@
 			)
 		)
+		(property "LCSC P/N" ""
+			(at 259.08 95.885 0)
+			(effects
+				(font
+					(size 1.27 1.27)
+				)
+				(hide yes)
+			)
+		)
+		(property "LCSC P/N Flight" ""
+			(at 259.08 95.885 0)
+			(effects
+				(font
+					(size 1.27 1.27)
+				)
+				(hide yes)
+			)
+		)
 		(pin "L9"
 		)
@@
 			)
 		)
-		(property "Footprint (for JLCPCB)" "0201"
+		(property "Footprint (for JLCPCB)" "0402"
 			(at 72.39 170.815 0)
 			(effects
@@
 			)
 		)
+		(property "LCSC P/N" ""
+			(at 72.39 170.815 0)
+			(effects
+				(font
+					(size 1.27 1.27)
+				)
+				(hide yes)
+			)
+		)
+		(property "LCSC P/N Flight" ""
+			(at 72.39 170.815 0)
+			(effects
+				(font
+					(size 1.27 1.27)
+				)
+				(hide yes)
+			)
+		)
 		(pin "1"
 		)
@@
 			)
 		)
+		(property "LCSC P/N" ""
+			(at 144.145 106.045 0)
+			(effects
+				(font
+					(size 1.27 1.27)
+				)
+				(hide yes)
+			)
+		)
+		(property "LCSC P/N Flight" ""
+			(at 144.145 106.045 0)
+			(effects
+				(font
+					(size 1.27 1.27)
+				)
+				(hide yes)
+			)
+		)
 		(pin "1"
 		)
@@
 			)
 		)
-		(property "Footprint (for JLCPCB)" "0201"
+		(property "Footprint (for JLCPCB)" "0402"
 			(at 215.265 172.72 0)
 			(effects
@@
 			)
 		)
+		(property "LCSC P/N" ""
+			(at 215.265 172.72 0)
+			(effects
+				(font
+					(size 1.27 1.27)
+				)
+				(hide yes)
+			)
+		)
+		(property "LCSC P/N Flight" ""
+			(at 215.265 172.72 0)
+			(effects
+				(font
+					(size 1.27 1.27)
+				)
+				(hide yes)
+			)
+		)
 		(pin "1"
 		)
@@
 			)
 		)
-		(property "Footprint (for JLCPCB)" "0201"
+		(property "Footprint (for JLCPCB)" "0402"
 			(at 215.265 205.74 0)
 			(effects
@@
 			(at 215.265 205.74 0)
 			(effects
+				(font
+					(size 1.27 1.27)
+				)
+				(hide yes)
+			)
+		)
+		(property "LCSC P/N" ""
+			(at 215.265 205.74 0)
+			(effects
+				(font
+					(size 1.27 1.27)
+				)
+				(hide yes)
+			)
+		)
+		(property "LCSC P/N Flight" ""
+			(at 215.265 205.74 0)
+			(effects
