File: hardware/Soldermander/sdram.kicad_sch (KiCad schematic)
At the start: 14 parts

Commit message: pre-autorouter part 2
Parts:
- C68, C69: renamed from C?; footprint adcs:Perfect_0402 -> Capacitor_SMD:C_0402_1005Metric
- C70, C71, C72, C73, C74, C75: renamed from C?; footprint adcs:Perfect_0201 -> Capacitor_SMD:C_0402_1005Metric
- FB6: renamed from FB?; footprint adcs:Perfect_0402 -> Fuse:Fuse_0402_1005Metric
- R24, R25, R26: renamed from R?; footprint adcs:Perfect_0402 -> Resistor_SMD:R_0402_1005Metric
- gave numbers to parts that had none: 1

Commit message: PrintedCoralBoard
Parts:
- C69: Footprint (for JLCPCB) 0402 -> (none)
- C70, C71, C72, C73, C74, C75: Footprint (for JLCPCB) 0201 -> (none)
