File: hardware/Soldermander/usbc.kicad_sch (KiCad schematic)
At the start: 8 parts, among them J1 USB_C_pycubed, U5 USBLC6-2SC6

Commit message: pre-autorouter part 2
Parts:
- C66: footprint adcs:Perfect_0402 -> Capacitor_SMD:C_0402_1005Metric
- R22, R23: footprint adcs:Perfect_0402 -> Resistor_SMD:R_0402_1005Metric
Connections:
- net OTG1_D_N: now also L2.3, TP9.1; no longer L2.2, TP8.1
- net OTG1_D_P: now also L2.2, TP8.1; no longer L2.3, TP9.1
