File: hardware/sqrt_of_g/adcs-hardware.kicad_sch (KiCad schematic)
At the start: 16 parts, among them J1 353620650, J10 Thruster Connector, J2 353620650, J21 Conn_01x10, J3 353620850, J4 353620850, J5 353620650, J6 353620650, J8 Control Debug Header, J9 353620850

Commit message: fix landing pattern
Other:
- sheet MCU: file microcontroller.kicad_sch -> rt1176.kicad_sch
Changed lines of the file:
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@@
       (effects (font (size 1.27 1.27)) (justify left bottom))
     )
-    (property "Sheetfile" "microcontroller.kicad_sch" (at 53.34 292.1 0)
+    (property "Sheetfile" "rt1176.kicad_sch" (at 53.34 292.1 0)
       (effects (font (size 1.27 1.27)) (justify left top) hide)
     )
