File: hardware/sun_sensor_pyramid/PCBassProShop.kicad_sch (KiCad schematic)
At the start: 6 parts, among them J1 5055670631, U1 LTC2052IS_PBF

Commit message: update names
Other:
- company: (none) -> Stanford Student Space Initiative
- title: (none) -> PCBassProShop
Changed lines of the file:
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@@
 	(generator_version "8.0")
 	(paper "A4")
+	(title_block
+		(title "PCBassProShop")
+		(date "2024-08-08")
+		(rev "3.0.0")
+		(company "Stanford Student Space Initiative")
+		(comment 1 "RE: Flynn Dreilinger")
+	)
 	(junction
 		(at 186.69 99.06)
@@
 		)
 		(instances
-			(project "ProBassCircuitboard"
+			(project "PCBassProShop"
 				(path "/1410c7f8-e2b9-4be8-9c91-5e92ba002382"
 					(page "2")
@@
 		)
 		(instances
-			(project "ProBassCircuitboard"
+			(project "PCBassProShop"
 				(path "/1410c7f8-e2b9-4be8-9c91-5e92ba002382"
 					(page "5")
@@
 		)
 		(instances
-			(project "ProBassCircuitboard"
+			(project "PCBassProShop"
 				(path "/1410c7f8-e2b9-4be8-9c91-5e92ba002382"
 					(page "3")
@@
 		)
 		(instances
-			(project "ProBassCircuitboard"
+			(project "PCBassProShop"
 				(path "/1410c7f8-e2b9-4be8-9c91-5e92ba002382"
 					(page "4")
