File: hardware/sun_sensor_pyramid/smol.kicad_sch (KiCad schematic)
At the start: 4 parts

Commit message: update names
Other:
- company: (none) -> Stanford Student Space Initiative
- title: (none) -> PCBassProShop
Changed lines of the file:
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@@
 	(generator_version "8.0")
 	(paper "A4")
+	(title_block
+		(title "PCBassProShop")
+		(date "2024-08-08")
+		(rev "3.0.0")
+		(company "Stanford Student Space Initiative")
+		(comment 1 "RE: Flynn Dreilinger")
+	)
 	(junction
 		(at 165.5318 94.3864)
